File: PIRT1280A1-12-carrier/PIRT1280A1-12-breakout.sch (EAGLE design)
At the start: 39 parts, among them U1 PIRT1280A1-12

Commit message: Prototype of PIRT sensor and an example LT3042 power supply layout for one of the supplies.
Parts:
- removed JP10, JP5, JP6, JP7, JP8, JP9: (no value), pinhead:PINHD-1X2
- removed TP15, TP16, TP17, TP18, TP19, TP20, TP21, TP22, TP23: TEST-POINT-LARGE-SQUARE, oresat-misc:TEST-POINT-LARGE-SQUARE
- added R1, R2: 10k, oresat-rcl:R-US_0603-C-NOSILK
- added R3, R4, R5, R6: (no value), oresat-rcl:R-US_0603-C-NOSILK
- added R7: 0, oresat-rcl:R-US_0603-C-NOSILK
- added U2, U3, U4, U5: LT3042IMSE#TRPBF, U-Analog-LT3042-ultralow-noise-ldo:LT3042IMSE#TRPBF
- C1, C2, C3: value 100n -> 4.7u
- U1: value PIRT1280A1-12 -> LT3042IMSE#TRPBF; device PIRT1280A1-12:PIRT1280A1-12 -> U-Analog-LT3042-ultralow-noise-ldo:LT3042IMSE#TRPBF
Connections:
- removed net ABITOUT: TP1.1, U1G$1.ABITOUT
- new net 5V: C1.1, R1.2, R2.2, TP12.1, U1.IN
- new net N$10: C2.1, R3.2, TP1.1, U1.SET
- new net N$11: R2.1, TP10.1, U1.PG
- new net N$12: R5.2, TP14.1, U1.ILIM
- new net N$15: R4.1, R6.2, U1.PGFB
- new net N$9: R1.1, TP11.1, U1.EN/UV
- new net VPOUT: C3.1, R4.2, R7.2, TP13.1, U1.OUT, U1.OUTS
- net GND: now also R3.1, R5.1, R6.1, U1.GND, U2.GND, U3.GND, U4.GND, U5.GND; no longer C4.2, C5.2, JP10.1, JP10.2, JP5.1, JP5.2, JP6.1, JP6.2, JP7.1, JP7.2, JP8.1, JP8.2, JP9.1, JP9.2, U1G$1.VGND, U1G$1.VN, U1G$1.VNOUT
- net JAMSYNC: no longer TP19.1, U1G$1.JAMSYNC
- net OUT1_N: no longer U1G$1.OUT1N
- net OUT1_P: no longer U1G$1.OUT1P
- net OUT2_N: no longer U1G$1.OUT2N
- net OUT2_P: no longer U1G$1.OUT2P
- net OUT3_N: no longer U1G$1.OUT3N
- net OUT3_P: no longer U1G$1.OUT3P
- net OUT4_N: no longer U1G$1.OUT4N
- net OUT4_P: no longer U1G$1.OUT4P
- net REFCLK: no longer TP20.1, U1G$1.REFCLK
- net SDCLK: no longer TP10.1, U1G$1.SDCLK
- net SDIN: no longer TP11.1, U1G$1.SDIN
- net SDOUT: no longer TP12.1, U1G$1.SDOUT
- net TEC+: no longer TP14.1, U1G$1.TEC+
- net TEC-: no longer TP13.1, U1G$1.TEC-
- net THERM+: no longer TP15.1, U1G$1.THERM+
- net THERM-: no longer TP16.1, U1G$1.THERM-
- net TXCLK_N: no longer U1G$1.TXCLKN
- net TXCLK_P: no longer U1G$1.TXCLKP
- net VEDETCOM-2.9V: no longer C2.1, TP17.1, U1G$1.VDETCOM
- net VPH-3.3V: no longer C5.1, TP21.1, U1G$1.VPH
- net VPL-1.6V: no longer C4.1, TP22.1, U1G$1.VPL
- net VPOS-3.3V: no longer C1.1, TP18.1, U1G$1.VPOS
- net VPOUT-0.9V: now also R7.1; no longer C3.1, TP23.1, U1G$1.VPOUT
Other:
- note added: "VPOUT = 0.9 +/- 0.05 V (5%) @ < 40 mA VPL = 1.6 +/- 0.05 V (3%) @ < 40 mA VDETCOM = 2.9 +/-0.05 V (1%) @ 0.6 mA VPH = 3.3 +/- 0.05 V (1%) @ < 40 mA VOPS = 3.3 +/- 0.05 V (1%) @ < 75 mA"
