File: PIRT1280A1-12-carrier/PIRT1280A1-12-carrier.brd (EAGLE design)
At the start: 156.8 x 68.6 mm, 124 parts, among them J1 5-1734592-0, U1 LT3042IMSE#TRPBF, U2 LT3042IMSE#TRPBF, U3 LT3042IMSE#TRPBF, U4 LT3042IMSE#TRPBF, U5 LT3042IMSE#TRPBF, U6 DS90CR218AMTD/NOPBMTD48_TEX-L

Commit message: mostly finished with PIRT1280 carrier
Parts:
- removed C38: 10u, oresat-rcl:.0603-C-NOSILK
- removed SJ11, SJ12, SJ13, SJ14, SJ15, SJ22: SOLDERJUMPERNC, SparkFun-Passives:SJ_2S
- removed TEC+, TEC-, VDETCOM, VPH, VPL, VPOS, VPOUT: TEST-POINT_SMD-SMD-10SN, oresat-misc:TESTPOINT_SMD-10SN
- removed TP39, TP40, TP41, TP42, TP43: TEST-POINT-LARGE-SQUARE, oresat-misc:1X01
- added C16: 1u, oresat-rcl:.0603-A
- added C17: 0.1u, oresat-rcl:.0603-A
- added C18: 1n, oresat-rcl:.0402-C-NOSILK
- added D1: GREEN, SparkFun-LED:LED-0603
- added J10, J3, J4, J5, J6: 455-1750-1-ND, SparkFun-Connectors:1X03
- added J11: USB_A_SMT_FEMALE, SparkFun-Connectors:USB-A-S-SILK-FEMALE
- added J12: (no value), SparkFun-Connectors:SCREWTERMINAL-5MM-2
- added J13: POWER_JACK, SparkFun-Connectors:POWER_JACK_PTH
- added J2: (no value), SparkFun-Connectors:1X02
- added J7: (no value), SparkFun-Connectors:1X05
- added J8: (no value), SparkFun-Connectors:1X13
- added J9: 5-1734592-0, J-TEConnectivity-X-1734592-X:TE_5-1734592-0
- added JP1, JP100, JP101: JUMPER-SMT_2_NC_TRACE_NO-SILK, SparkFun-Jumpers:SMT-JUMPER_2_NC_TRACE_NO-SILK
- added Q1: 35A/25V/8.5mΩ, Q-Fairchild-FDD8780-MOSFET-NCH:DPAK
- added R100, R101, R21, R22, R23, R24, R25, R26: 100, oresat-rcl:.0402-C-NOSILK
- added R12: NP, oresat-rcl:.0603-A
- added R19: 10k, R-Panasonic-EXB_A10PXXXJ:ARRAY_EXBA-M
- added R20: TBD, oresat-rcl:.0603-A
- added REFCLK, THERM+, THERM-, TP9: TEST-POINT-LARGE-SQUARE, oresat-misc:1X01
- added TP100, TP101, TP102, TP103, TP104, TP105, TP106, TP107: TEST-POINT-SMD-0.5MM, oresat-misc:TESTPOINT_SMD-0.5MM
- added U$2: POCKETBEAGLE, PocketBeagle:POCKETBEAGLE
- added U$3: (no value), Oliver_Custom:POLARITY_SYMBOL_SMALL
- added U7: DS90CR218AMTD/NOPBMTD48_TEX-L, U-TI-DS90CR218-LVDSReceiver:MTD48_TEX-L
- added X1: 16MHz, X-OSCILLATOR-GENERIC:OSC_2.5X2.0
- C1, C10, C2, C3, C4, C5, C6, C7, C8, C9: device oresat-rcl:.0402-A-NOSILK -> oresat-rcl:.0603-A
- C11, C12, C13, C14, C15: value 4.7u -> 0.47u; device oresat-rcl:.0402-A-NOSILK -> oresat-rcl:.0603-A
- C19, C22: value 1n -> 10n
- C20, C23: value 1n -> 100n
- C24: value 1n -> 10u; device oresat-rcl:.0402-C-NOSILK -> oresat-rcl:.0603-C-NOSILK
- C25, C30: value 10n -> 100n
- C27, C28: value 10n -> 1n
- C31, C36: value 100n -> 1n
- C32, C35: value 100n -> 10n
- J1: value 5-1734592-0 -> 455-1750-1-ND; device J-TEConnectivity-X-1734592-X:TE_5-1734592-0 -> SparkFun-Connectors:1X03
- R1: value (none) -> 1k; device oresat-rcl:.0603-A-NOSILK -> oresat-rcl:.0603-A
- R10, R11, R8, R9: value 100 -> NP; device oresat-rcl:.0402-C-NOSILK -> oresat-rcl:.0603-A
- R13, R14: value 100 -> 0; device oresat-rcl:.0402-C-NOSILK -> oresat-rcl:.0603-A
- R15, R17: device oresat-rcl:.0603-A-NOSILK -> oresat-rcl:.0603-A
- R16: value (none) -> 0; device oresat-rcl:.0603-A-NOSILK -> oresat-rcl:.0603-A
- R18: value 100 -> 20k; device oresat-rcl:.0402-C-NOSILK -> oresat-rcl:.0805-A
- R2: value 0 -> 10k; device oresat-rcl:.0603-A-NOSILK -> R-Panasonic-EXB-2HV103JV:RES_EXB2HV
- R3: value (none) -> 29.4k; device oresat-rcl:.0603-A-NOSILK -> oresat-rcl:.0603-A
- R4: value (none) -> 9.09k; device oresat-rcl:.0603-A-NOSILK -> oresat-rcl:.0603-A
- R5: value 0 -> 16.2k; device oresat-rcl:.0603-A-NOSILK -> oresat-rcl:.0603-A
- R6: value (none) -> 33.2k; device oresat-rcl:.0603-A-NOSILK -> oresat-rcl:.0603-A
- R7: value 0 -> 33.2k; device oresat-rcl:.0603-A-NOSILK -> oresat-rcl:.0603-A
- SJ1, SJ10, SJ2, SJ3, SJ4, SJ5, SJ6, SJ7, SJ8, SJ9: value SOLDERJUMPERNC -> JUMPER-SMT_2_NC_TRACE_NO-SILK; device SparkFun-Passives:SJ_2S -> SparkFun-Jumpers:SMT-JUMPER_2_NC_TRACE_NO-SILK
- U$1: value POCKETBEAGLE -> (none); device PocketBeagle:POCKETBEAGLE -> PIRT1280-BREAKOUT-FOOTPRINT:PIRT1280_BREAKOUT
- U6: value DS90CR218AMTD/NOPBMTD48_TEX-L -> LM2901QPWRQ1PW14-M; device U-TI-DS90CR218-LVDSReceiver:MTD48_TEX-L -> U-TI-LM2901:PW14-M
- moved R14 265.4 mm to (89.2, 77.5), turned to 90 degrees
- moved TP8 261.4 mm to (95.0, 94.0), turned to 270 degrees
- moved R13 258.3 mm to (80.2, 77.5), turned to 90 degrees
- moved R18 253.0 mm to (56.0, 75.0), turned to 90 degrees
- moved TP4 249.6 mm to (84.0, 94.0), turned to 90 degrees
- moved TP2 249.4 mm to (77.0, 94.0), turned to 270 degrees
- moved TP7 249.2 mm to (93.0, 94.0), turned to 270 degrees
- moved TP5 249.0 mm to (86.0, 94.0), turned to 90 degrees
- moved TP3 248.8 mm to (79.0, 94.0), turned to 270 degrees
- moved TP6 248.5 mm to (88.0, 94.0), turned to 90 degrees
- moved C15 247.8 mm to (111.5, 84.0), turned to 180 degrees
- moved R17 243.6 mm to (116.2, 77.5), turned to 90 degrees
- moved J1 237.3 mm to (14.0, 88.0), turned to 180 degrees
- moved R16 236.8 mm to (107.2, 77.5), turned to 90 degrees
- moved C14 234.0 mm to (102.5, 84.0), turned to 180 degrees
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Connections:
- removed net CLK: U$1.P1_20, U6.23
- removed net D0: U$1.P1_36, U6.24
- removed net D1: U$1.P1_33, U6.26
- removed net D2: U$1.P2_32, U6.27
- removed net D3: U$1.P2_30, U6.29
- removed net D4: U$1.P1_31, U6.30
- removed net D5: U$1.P2_34, U6.31
- removed net D6: U$1.P2_28, U6.33
- removed net D7: U$1.P1_29, U6.34
- removed net N$30: SJ11.1, TP32.1, U4.3
- removed net N$34: U6.22
- removed net SDCLK: J1.49, TP4.1
- removed net SDIN: J1.50, TP5.1
- removed net SDOUT: J1.48, TP6.1
- removed net USB_D+: U$1.P1_11
- removed net USB_D-: U$1.P1_9
- new net !PWR_DWN: J3.2, R19.1, U7.22
- new net 1.8V-A: R20.2, U$2.P1_18
- new net N$1: R2.1, R2.2
- new net N$2: R2.15, R2.3, U6.10
- new net N$270: D1.A, R1.1
- new net N$3: R2.14, R2.4, U6.8
- new net N$4: R2.13, R2.5, U6.4
- new net N$41: J13.PWR, U$2.P1_1
- new net N$44: R2.11, R2.12, U6.6
- new net N$47: TP100.TP, U7.34
- new net N$48: TP101.TP, U7.35
- new net N$49: TP102.TP, U7.37
- new net N$5: C16.1, R18.2, U6.11, U6.5, U6.7, U6.9
- new net N$50: TP103.TP, U7.39
- new net N$51: TP104.TP, U7.40
- new net N$52: TP105.TP, U7.41
- new net N$53: TP106.TP, U7.43
- new net N$54: TP107.TP, U7.45
- new net N$55: J2.2, U$2.P1_34
- new net N$56: J10.1, Q1.4
- new net N$58: J3.1, U$2.P2_20
- new net N$6: R2.6, R2.7
- new net N$8: JP100.1, U$2.P1_5
- new net PRU0: J8.2, U$2.P1_36, U7.24
- new net PRU1: J8.3, U$2.P1_33, U7.26
- new net PRU14_OUT: J8.11, U$2.P2_24
- new net PRU15_OUT: J8.12, U$2.P2_33
- new net PRU16_CLK: J8.9, U$2.P1_20, U7.23
- new net PRU2: J8.4, U$2.P2_32, U7.27
- new net PRU3: J8.5, U$2.P2_30, U7.29
- new net PRU4: J8.6, U$2.P1_31, U7.30
- new net PRU5: J8.7, U$2.P2_34, U7.31
- new net PRU6: J8.8, U$2.P2_28, U7.33
- new net PRU7: J8.10, U$2.P1_29
- new net PRU_UART_RX: J6.2, U$2.P1_12
- new net PRU_UART_TX: J6.1, U$2.P1_6
- new net REFCLK_ENABLE: R19.3, TP27.1, TP28.1, U6.13, X1.1
- new net SENSOR_ENABLE: J4.1, U$2.P1_28
- new net TEC_ENABLE: Q1.1, R19.2, U$2.P1_35
- new net TEC_GND: J10.3, J12.1, Q1.3
- new net UART0_RX: J5.2, U$2.P1_32
- new net UART0_TX: J5.1, U$2.P1_30
- new net USB_N: J11.D-, U$2.P1_9
- new net USB_P: J11.D+, U$2.P1_11
- net 3.3V: now also C18.1, J3.3, J4.3, R2.16, U$2.P1_14, U$2.P2_23, U6.3, U7.12, U7.20, U7.28, U7.36, U7.42, U7.48, X1.4; no longer C38.1, U$1.P1_14, U$1.P2_23, U6.12, U6.20, U6.28, U6.36, U6.42, U6.48
- net 5V: now also C2.1, C3.1, C5.1, J11.VBUS, JP100.2, SJ10.2, SJ7.2, TP15.1, TP3.1, TP6.1, TP9.1, U$2.P1_24, U$2.P2_13; no longer C10.1, C13.1, C7.1, SJ11.2, SJ12.2, SJ14.2, SJ15.2, SJ2.2, SJ3.2, SJ5.2, TP19.1, TP26.1, TP33.1, TP40.1, U$1.P1_7
- net CAN_RX: now also J1.2, U$2.P2_9; no longer U$1.P2_9
- net CAN_TX: now also J1.1, U$2.P2_11; no longer U$1.P2_11
- net GND: now also C16.2, C17.2, C18.2, D1.C, J11.GND, J11.SHLD1, J11.SHLD2, J13.GND, J13.GNDBREAK, J5.3, J6.3, J7.5, J8.1, J8.13, J9.1, J9.10, J9.13, J9.16, J9.19, J9.2, J9.22, J9.25, J9.28, J9.3, J9.31, J9.34, J9.37, J9.40, J9.44, J9.48, J9.7, J9.S1, J9.S2, JP1.1, JP101.2, R10.1, R11.1, R12.1, R19.10, R19.5, R2.10, R5.1, R7.1, R8.1, R9.1, SJ2.1, SJ3.1, SJ5.1, U$2.P1_15, U$2.P1_16, U$2.P1_22, U$2.P2_15, U$2.P2_21, U6.12, U7.13, U7.18, U7.19, U7.21, U7.25, U7.3, U7.32, U7.38, U7.44, U7.7, X1.2; no longer C38.2, J1.12, J1.15, J1.19, J1.23, J1.27, J1.31, J1.35, J1.39, J1.43, J1.6, J1.9, J1.S1, J1.S2, R1.1, R16.1, SJ10.1, SJ13.1, SJ7.1, U$1.P1_15, U$1.P1_22, U$1.P2_15, U$1.P2_21, U6.13, U6.18, U6.19, U6.21, U6.25, U6.3, U6.32, U6.38, U6.44, U6.7
- net JAMSYNC: now also J2.1, J9.49; no longer J1.47, TP7.1
- net N$10: now also R19.7, TP20.1, TP21.1, U1.3, U6.14; no longer SJ5.1, TP18.1, U2.3
- net N$11: now also SJ7.1, TP31.1, U5.6; no longer SJ3.1, TP15.1, U1.6
- net N$12: now also SJ2.2, TP4.1, U5.5; no longer SJ1.2, TP14.1, U1.5
- net N$13: now also R100.2, U7.14; no longer R9.2, U6.14
- net N$14: now also R100.1, U7.15; no longer R9.1, U6.15
- net N$15: now also TP5.1, U5.4; no longer TP10.1, U1.4
- net N$16: now also JP101.1, U$2.P1_13; no longer U$1.P1_16
- net N$17: now also J4.2, R18.1; no longer U$1.P1_3, U$1.P1_5
- net N$18: now also R101.2, U7.10; no longer R10.2, U6.10
- net N$19: now also R101.1, U7.11; no longer R10.1, U6.11
- net N$20: now also C12.1, R4.2, R9.2, TP32.1, U5.7; no longer C2.1, R3.2, TP1.1, U1.7
- net N$21: now also SJ1.2, TP1.1, U1.5; no longer SJ4.2, TP21.1, U2.5
- net N$22: now also TP29.1, U1.6; no longer TP22.1, U2.6
- net N$23: now also TP2.1, U1.4; no longer TP17.1, U2.4
- net N$24: now also C11.1, R3.2, R8.2, TP30.1, U1.7; no longer C5.1, R1.2, TP16.1, U2.7
- net N$25: now also R1.2, R19.6, TP16.1, TP17.1, U3.3, U4.3, U6.1; no longer SJ8.1, TP25.1, U5.3
- net N$26: now also SJ5.2, TP13.1, U4.5; no longer SJ7.2, TP28.1, U5.5
- net N$27: now also SJ10.1, TP37.1, U4.6; no longer SJ9.1, TP29.1, U5.6
- net N$28: now also TP14.1, U4.4; no longer TP24.1, U5.4
- net N$29: now also C15.1, R12.2, R7.2, TP38.1, U4.7; no longer C8.1, R4.2, TP23.1, U5.7
- net N$31: now also SJ4.2, TP10.1, U3.5; no longer SJ10.2, TP35.1, U4.5
- net N$32: now also SJ9.1, TP35.1, U3.6; no longer SJ12.1, TP36.1, U4.6
- net N$33: now also TP11.1, U3.4; no longer TP31.1, U4.4
- net N$35: now also C14.1, R11.2, TP36.1, U3.7; no longer C11.1, TP30.1, U4.7
- net N$36: now also R19.4, TP18.1, TP19.1, U2.3, U5.3, U6.2; no longer SJ14.1, TP39.1, U3.3
- net N$37: now also SJ3.2, TP7.1, U2.5; no longer SJ13.2, TP42.1, U3.5
- net N$38: now also SJ8.1, TP33.1, U2.6; no longer SJ15.1, TP43.1, U3.6
- net N$39: now also TP8.1, U2.4; no longer TP38.1, U3.4
- net N$40: now also C13.1, R10.2, R5.2, TP34.1, U2.7; no longer C14.1, R16.2, TP37.1, U3.7
- net N$9: now also R26.1, X1.3; no longer SJ2.1, TP11.1, U1.3
- net OUT1_N: now also J9.27, R24.2, U7.8; no longer J1.11, R8.2, U6.8
- net OUT1_P: now also J9.26, R24.1, U7.9; no longer J1.10, R8.1, U6.9
- net OUT2_N: now also J9.24, R23.1; no longer J1.8, R13.2
- net OUT2_P: now also J9.23, R23.2; no longer J1.7, R13.1
- net OUT3_N: now also J9.21, R22.1; no longer J1.5, R14.2
- net OUT3_P: now also J9.20, R22.2; no longer J1.4, R14.1
- net OUT4_N: now also J9.18, R21.1; no longer J1.2, R18.2
- net OUT4_P: now also J9.17, R21.2; no longer J1.1, R18.1
- net REFCLK: now also J9.50, R26.2, REFCLK.1; no longer J1.46, TP8.1
- net SPI1_CLK: now also J7.2, J9.5, U$2.P2_29; no longer U$1.P2_29
- net SPI1_CS1: now also J7.4, U$2.P2_31; no longer U$1.P2_31
- net SPI1_MISO: now also J7.3, J9.6, U$2.P2_27; no longer U$1.P2_27
- net SPI1_MOSI: now also J7.1, J9.4, U$2.P2_25; no longer U$1.P2_25
- net TEC+: now also J12.2, J9.45, J9.46, J9.47; no longer J1.40, J1.41, J1.42, TEC+.TP
- net TEC-: now also J10.2, J9.41, J9.42, J9.43; no longer J1.36, J1.37, J1.38, TEC-.TP
- net THERM+: now also C17.1, J9.9, R20.1, THERM+.1, U$2.P1_17; no longer J1.45, TP2.1
- net THERM-: now also J9.8, JP1.2, THERM-.1; no longer J1.44, TP3.1
- net TXCLK_N: now also J9.30, R25.1, U7.16; no longer J1.14, R11.1, U6.16
- net TXCLK_P: now also J9.29, R25.2, U7.17; no longer J1.13, R11.2, U6.17
- net VDETCOM: now also R13.2, TP22.1, U1.10, U1.9; no longer J1.28, J1.29, J1.30, R2.2, TP20.1, U2.10, U2.9, VDETCOM.TP
- net VDETCOM-2.9V: now also J9.11, J9.12, R13.1; no longer R2.1
- net VPH: now also C9.1, R16.2, TP25.1, U3.10, U3.9; no longer C12.1, J1.24, J1.25, J1.26, R15.2, TP34.1, U4.10, U4.9, VPH.TP
- net VPH-3.3V: now also J9.35, J9.36, R16.1; no longer R15.1
- net VPL: now also C8.1, R15.2, TP24.1, U2.10, U2.9; no longer C15.1, J1.20, J1.21, J1.22, R17.2, TP41.1, U3.10, U3.9, VPL.TP
- net VPL-1.6V: now also J9.32, J9.33, R15.1; no longer R17.1
- net VPOS: now also C10.1, R17.2, TP26.1, U4.10, U4.9; no longer C9.1, J1.32, J1.33, J1.34, R5.2, TP27.1, U5.10, U5.9, VPOS.TP
- net VPOS-3.3V: now also J9.38, J9.39, R17.1; no longer R5.1
- net VPOUT: now also C7.1, R14.2, TP23.1, U5.10, U5.9; no longer C3.1, J1.16, J1.17, J1.18, R7.2, TP13.1, U1.10, U1.9, VPOUT.TP
- net VPOUT-0.9V: now also J9.14, J9.15, R14.1; no longer R7.1
Routing:
- net SPI1_MOSI: track 0.00 -> 152.2 mm
- net SPI1_MISO: track 0.00 -> 145.9 mm
- net SPI1_CLK: track 0.00 -> 143.0 mm
- net SENSOR_ENABLE: track 0.00 -> 137.0 mm, vias 0 -> 1
- net PRU16_CLK: track 0.00 -> 122.6 mm, vias 0 -> 2
- net PRU6: track 0.00 -> 114.8 mm, vias 0 -> 1
- net PRU4: track 0.00 -> 110.8 mm, vias 0 -> 1
- net PRU2: track 0.00 -> 107.9 mm, vias 0 -> 1
- net PRU3: track 0.00 -> 107.4 mm, vias 0 -> 1
- net JAMSYNC: track 0.00 -> 106.6 mm, vias 0 -> 2
- net TEC_ENABLE: track 0.00 -> 106.5 mm, vias 0 -> 4
- net PRU5: track 0.00 -> 106.4 mm, vias 0 -> 1
- net GND: track 2.16 -> 105.2 mm, vias 25 -> 208
- net PRU1: track 0.00 -> 95.3 mm, vias 0 -> 1
- net N$58: track 0.00 -> 89.2 mm
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- added copper zone on layer 1, net 3.3V
- added copper zone on layer 15, net 3.3V
- added copper zone on layer 16, net 3.3V
- added copper zone on layer 16, net 3.3V3
- added copper zone on layer 15, net 5V
- added copper zone on layer 16, net 5V
- added copper zone on layer 1, net N$56
- added copper zone on layer 1, net TEC+
- added copper zone on layer 1, net TEC-
- added copper zone on layer 1, net TEC_GND
- added copper zone on layer 1, net VDETCOM
- added copper zone on layer 1, net VDETCOM-2.9V
- added copper zone on layer 1, net VPH
- added copper zone on layer 1, net VPH-3.3V
- added copper zone on layer 1, net VPL
- added copper zone on layer 1, net VPL-1.6V
- added copper zone on layer 1, net VPOS
- added copper zone on layer 1, net VPOS-3.3V
- added copper zone on layer 1, net VPOUT-0.9V
- removed copper zone on layer 15, net GND
Other:
- board size 156.8 x 68.6 mm -> 204 x 100 mm
- board text added: "+"
- board text added: "-"
- board text added: "5V"
- board text added: "5V MAX"
- board text added: "8.2VDC @ 27C 9.2VDC @ 50C"
- board text added: "CAMERA/PRU"
- board text added: "CAN0"
- board text added: "CLK"
- board text added: "CS"
- board text added: "D0"
- board text added: "D1"
- board text added: "D2"
- board text added: "D3"
- board text added: "D4"
- board text added: "D5"
- board text added: "D6"
- board text added: "DISABLE"
- board text added: "ENABLE"
- board text added: "GND"
- board text added: "GPIO"
- board text added: "MANUAL"
- board text added: "MISO"
- board text added: "MOSI"
- board text added: "OFF"
- board text added: "OLIVER REW"
- board text added: "OreSat PIRT1280A1-12 Carrier Board v1.0"
- board text added: "PIRT1280 ENABLE"
- board text added: "PRU UART"
- board text added: "R30_14"
- board text added: "R30_15"
- board text added: "R30_7"
- board text added: "RX"
- board text added: "SENSOR ENABLE"
- board text added: "SERDES ENABLE"
- board text added: "SPI"
- board text added: "TEC"
- board text added: "TODO RENUMBER"
- board text added: "TX"
- board text added: "UART0"
- board text added: "copper plate thickness = 9.5mm ribbon cable length = 30mm 9.5mm^2 + x^2 = 30mm^2 x = ~28.4mm **Distance between connectors should be less than 28mm, lets say 20mm?***"
- board text removed: "OUT1_N"
- board text removed: "OUT1_P"
- board text removed: "OUT2_N"
- board text removed: "OUT2_P"
- board text removed: "OUT3_N"
- board text removed: "OUT3_P"
- board text removed: "OUT4_N"
- board text removed: "OUT4_P"
- board text removed: "OreSat PIRT1280A1-12 Carrier Board"
- board text removed: "REFCLK"
- board text removed: "SDCLK"
- board text removed: "SDIN"
- board text removed: "SDOUT"
- board text removed: "TEC+"
- board text removed: "TEC-"
- board text removed: "THERM+"
- board text removed: "THERM-"
- board text removed: "TXCLK_N"
- board text removed: "TXCLK_P"
- board text removed: "VDETCOM"
- board text removed: "VPH"
- board text removed: "VPL"
- board text removed: "VPOS"
- board text removed: "VPOUT"
- board text removed: "v1"

Commit message: touch ups
Other:
- outline, holes or cut-outs redrawn
- board text removed: "TODO RENUMBER"
Changed lines of the file:
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@@
 <text x="137" y="94" size="1.778" layer="21" font="vector" ratio="15">2021-01-21</text>
 <text x="18.25" y="92.75" size="1.778" layer="48">TODOimage sensor test board with test points and load resistors</text>
-<wire x1="0" y1="0" x2="0" y2="100" width="0" layer="20"/>
-<wire x1="0" y1="100" x2="204" y2="100" width="0" layer="20"/>
-<wire x1="204" y1="100" x2="204" y2="0" width="0" layer="20"/>
-<wire x1="204" y1="0" x2="0" y2="0" width="0" layer="20"/>
+<wire x1="0" y1="3" x2="0" y2="97" width="0" layer="20"/>
+<wire x1="3" y1="100" x2="201" y2="100" width="0" layer="20"/>
+<wire x1="204" y1="97" x2="204" y2="3" width="0" layer="20"/>
 <text x="128" y="60" size="1.016" layer="51">copper plate thickness = 9.5mm
 ribbon cable length = 30mm
@@
 <hole x="200" y="96" drill="3"/>
 <hole x="200" y="4" drill="3"/>
-<text x="67" y="119.5" size="6.4516" layer="51">TODO RENUMBER</text>
 <text x="54.25" y="94" size="1.016" layer="21" font="vector" ratio="20">PIRT1280 ENABLE</text>
 <text x="173" y="94" size="1.778" layer="21" font="vector" ratio="15">OLIVER REW</text>
@@
 <text x="76.7525" y="19.333" size="1" layer="21" font="vector" ratio="15" distance="240" rot="R180" align="center-left">5V</text>
 <text x="81.27875" y="19.333" size="1" layer="21" font="vector" ratio="15" distance="240" rot="R180" align="center-right">GND</text>
+<wire x1="201" y1="0" x2="3" y2="0" width="0" layer="20"/>
 <wire x1="88" y1="0" x2="88" y2="29" width="0.508" layer="21"/>
 <wire x1="88" y1="29" x2="70" y2="29" width="0.508" layer="21"/>
@@
 <wire x1="17.0875" y1="91.9" x2="17.0875" y2="90.4" width="0.127" layer="21"/>
 <wire x1="17.0875" y1="90.4" x2="20.0875" y2="90.4" width="0.127" layer="21"/>
+<wire x1="3" y1="0" x2="0" y2="3" width="0" layer="20" curve="-90"/>
+<wire x1="3" y1="100" x2="0" y2="97" width="0" layer="20" curve="90"/>
+<wire x1="201" y1="100" x2="204" y2="97" width="0" layer="20" curve="-90"/>
+<wire x1="201" y1="0" x2="204" y2="3" width="0" layer="20" curve="90"/>
 </plain>
 <attributes>

Commit message: pre-review cleanup
Changed lines of the file:
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@@
 <drawing>
 <settings>
-<setting alwaysvectorfont="yes"/>
+<setting alwaysvectorfont="no"/>
 <setting verticaltext="up"/>
 </settings>
@@
 <contactref element="TP31" pad="1"/>
 <contactref element="SJ7" pad="1"/>
-<wire x1="85.999996875" y1="85.84" x2="85.16" y2="85.84" width="0.3048" layer="1"/>
 <wire x1="85.16" y1="85.84" x2="85" y2="86" width="0.3048" layer="1"/>
 <wire x1="85" y1="86" x2="84.008" y2="86" width="0.3048" layer="1"/>
@@
 <wire x1="82.5" y1="79" x2="84" y2="77.5" width="0.3048" layer="1"/>
 <wire x1="84" y1="85.992" x2="82.5" y2="84.492" width="0.3048" layer="1"/>
+<wire x1="86" y1="85.84" x2="85.16" y2="85.84" width="0.3048" layer="1"/>
 </signal>
 <signal name="N$15">

Commit message: address review comments
Parts:
- added C37: 1n, oresat-rcl:.0402-C-NOSILK
- added C38, C39: NP, oresat-rcl:C1210
- added C40: 0.1u, oresat-rcl:.0603-A
- added D2: GREEN, SparkFun-LED:LED-0603
- added FB1: (no value), oresat-rcl:.0805-B
- added J14: POWER_JACK, SparkFun-Connectors:POWER_JACK_PTH
- added R27: 100, oresat-rcl:.0402-C-NOSILK
- added R28: 1k, oresat-rcl:.0603-A
- C11: value 0.47u -> 0.1u
- C16: value 1u -> 0.47u
- C17: value 0.1u -> 1u
- C18: value 1n -> 0.1u; device oresat-rcl:.0402-C-NOSILK -> oresat-rcl:.0603-A
- C19, C22, C29, C32: value 10n -> 1n
- C20, C23, C30, C33: value 100n -> 10n
- C21, C31: value 1n -> 100n
- C24: value 10u -> 100n; device oresat-rcl:.0603-C-NOSILK -> oresat-rcl:.0402-C-NOSILK
- C25: value 100n -> 10u; device oresat-rcl:.0402-C-NOSILK -> oresat-rcl:.0603-C-NOSILK
- C26, C35: value 10n -> 100n
- C27, C36: value 1n -> 10n
- J11: value USB_A_SMT_FEMALE -> (none); device SparkFun-Connectors:USB-A-S-SILK-FEMALE -> SparkFun-Connectors:1X02
- J12: value (none) -> USB_A_SMT_FEMALE; device SparkFun-Connectors:SCREWTERMINAL-5MM-2 -> SparkFun-Connectors:USB-A-S-SILK-FEMALE
- J13: value POWER_JACK -> (none); device SparkFun-Connectors:POWER_JACK_PTH -> SparkFun-Connectors:SCREWTERMINAL-5MM-2
- J5: value 455-1750-1-ND -> (none); device SparkFun-Connectors:1X03 -> SparkFun-Connectors:1X04
- R18: value 20k -> 200k
- R19: value 10k -> 20k; device R-Panasonic-EXB_A10PXXXJ:ARRAY_EXBA-M -> oresat-rcl:.0805-A
- R20: value TBD -> 10k; device oresat-rcl:.0603-A -> R-Panasonic-EXB_A10PXXXJ:ARRAY_EXBA-M
- R21: value 100 -> TBD; device oresat-rcl:.0402-C-NOSILK -> oresat-rcl:.0603-A
- R22, R23, R24, R29, R30: value 100 -> NP
- moved C16 53.3 mm to (111.5, 84.0), turned to 180 degrees
- moved J12 41.1 mm to (59.0, 7.00), turned to 90 degrees
- moved C17 28.2 mm to (59.0, 75.0), turned to 270 degrees
- moved U5 27.0 mm to (114.0, 88.0)
- moved J13 21.4 mm to (100.0, 4.00)
- moved C11 21.1 mm to (54.4, 85.8), turned to 90 degrees
- moved R20 20.2 mm to (67.0, 75.0), turned to 90 degrees
- moved R24 19.8 mm to (99.8, 51.2)
- moved R21 19.2 mm to (83.0, 64.0), turned to 180 degrees
- moved C24 19.0 mm to (94.5, 52.2), turned to 90 degrees
- moved J11 18.1 mm to (53.2, 24.2), turned to 0 degrees
- moved C34 17.5 mm to (94.5, 45.2), turned to 90 degrees
- moved C28 11.5 mm to (80.0, 49.0)
- moved C18 11.5 mm to (83.0, 62.0), turned to 180 degrees
- moved R26 11.2 mm to (80.0, 47.0), turned to 270 degrees
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- renumbered JP100 to JP2, JP101 to JP3, R100 to R29, R101 to R30, TP100 to TP39, TP101 to TP40, TP102 to TP41, TP103 to TP42, TP104 to TP43, TP105 to TP44, TP106 to TP45, TP107 to TP46
Connections:
- net N$58 renamed SERDES_PWR_DOWN
- removed net N$41: J13.PWR, U$2.P1_1
- new net N$30: J11.1, U$2.P1_1
- new net N$34: D2.A, R28.1
- new net N$7: FB1.1, J11.2, J14.PWR, R28.2
- new net VDD: J12.VBUS, JP2.2, U$2.P1_24, U$2.P2_13
- net !PWR_DWN: now also R20.1; no longer R19.1
- net 1.8V-A: now also R21.2; no longer R20.2
- net 3.3V: now also C11.1, C37.1, C40.1, J5.1; no longer C18.1
- net 5V: now also C38.1, C39.1, FB1.2; no longer J11.VBUS, JP2.2, U$2.P1_24, U$2.P2_13
- net GND: now also C37.2, C38.2, C39.2, C40.2, D2.C, J12.GND, J12.SHLD1, J12.SHLD2, J14.GND, J14.GNDBREAK, J5.4, R18.1, R20.10, R20.5; no longer J11.GND, J11.SHLD1, J11.SHLD2, J13.GND, J13.GNDBREAK, J5.3, R19.10, R19.5
- net N$10: now also R20.7; no longer R19.7
- net N$11: now also U2.6; no longer U5.6
- net N$12: now also U2.5; no longer U5.5
- net N$15: now also U2.4; no longer U5.4
- net N$17: now also R19.1; no longer R18.1
- net N$20: now also C13.1, U2.7; no longer C12.1, U5.7
- net N$24: now also C12.1; no longer C11.1
- net N$25: now also R20.6, U5.3; no longer R19.6, U3.3
- net N$26: now also U5.5; no longer U4.5
- net N$27: now also U5.6; no longer U4.6
- net N$28: now also U5.4; no longer U4.4
- net N$29: now also C16.1, U5.7; no longer C15.1, U4.7
- net N$31: now also U4.5; no longer U3.5
- net N$32: now also U4.6; no longer U3.6
- net N$33: now also U4.4; no longer U3.4
- net N$35: now also C15.1, U4.7; no longer C14.1, U3.7
- net N$36: now also R20.4, U3.3; no longer R19.4, U5.3
- net N$37: now also U3.5; no longer U2.5
- net N$38: now also U3.6; no longer U2.6
- net N$39: now also U3.4; no longer U2.4
- net N$40: now also C14.1, U3.7; no longer C13.1, U2.7
- net N$5: now also C17.1, R19.2; no longer C16.1
- net N$9: now also R27.1; no longer R26.1
- net OUT1_N: now also R25.2; no longer R24.2
- net OUT1_P: now also R25.1; no longer R24.1
- net OUT2_N: now also R24.1; no longer R23.1
- net OUT2_P: now also R24.2; no longer R23.2
- net OUT3_N: now also R23.1; no longer R22.1
- net OUT3_P: now also R23.2; no longer R22.2
- net OUT4_N: now also R22.1; no longer R21.1
- net OUT4_P: now also R22.2; no longer R21.2
- net REFCLK: now also R27.2; no longer R26.2
- net REFCLK_ENABLE: now also R20.3; no longer R19.3
- net TEC+: now also J13.2; no longer J12.2
- net TEC_ENABLE: now also R20.2; no longer R19.2
- net TEC_GND: now also J13.1; no longer J12.1
- net THERM+: now also C18.1, R21.1; no longer C17.1, R20.1
- net TXCLK_N: now also R26.1; no longer R25.1
- net TXCLK_P: now also R26.2; no longer R25.2
- net UART0_RX: now also J5.3; no longer J5.2
- net UART0_TX: now also J5.2; no longer J5.1
- net USB_N: now also J12.D-; no longer J11.D-
- net USB_P: now also J12.D+; no longer J11.D+
- net VPH: now also U4.10, U4.9; no longer U3.10, U3.9
- net VPL: now also U3.10, U3.9; no longer U2.10, U2.9
- net VPOS: now also U5.10, U5.9; no longer U4.10, U4.9
- net VPOUT: now also U2.10, U2.9; no longer U5.10, U5.9
Routing:
- net VDD: track 0.00 -> 85.8 mm, vias 0 -> 1
- net 5V: track 66.5 -> 4.96 mm, vias 32 -> 28
- net N$7: track 0.00 -> 44.0 mm
- net N$41: track 43.7 -> 0.00 mm
- net N$30: track 0.00 -> 23.7 mm
- net 3.3V: track 36.2 -> 41.2 mm
- net VPOUT: track 4.50 -> 0.00 mm, vias 1 -> 0
- net VPOS: track 4.50 -> 0.00 mm, vias 1 -> 0
- net UART0_TX: track 60.9 -> 65.0 mm
- net VPL: track 4.00 -> 0.00 mm, vias 1 -> 0
- net VPH: track 4.00 -> 0.00 mm, vias 1 -> 0
- net VDETCOM: track 4.00 -> 0.00 mm, vias 1 -> 0
- net UART0_RX: track 60.3 -> 64.1 mm
- net N$17: track 22.0 -> 25.1 mm
- net N$5: track 25.8 -> 28.8 mm
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- removed copper zone on layer 16, net 5V
Other:
- board text added: "2021-04-12"
- board text added: "3.3V"
- board text added: "5V MAX 2A"
- board text added: "8.2VDC @ 27C 9.2VDC @ 50C 2.5A"
- board text added: "POCKETBEAGLE POWER"
- board text removed: "2021-01-21"
- board text removed: "5V MAX"
- board text removed: "8.2VDC @ 27C 9.2VDC @ 50C"

Commit message: added PIRT1280 BOM, used internal library in carrier, added attributes
Parts:
- J12: device SparkFun-Connectors:USB-A-S-SILK-FEMALE -> J-Generic-USB_A_Female:USB-A-S-SILK-FEMALE
- J13: device SparkFun-Connectors:SCREWTERMINAL-5MM-2 -> J-Generic-5mm-Screw-Terminal:SCREWTERMINAL-5MM-2
- J14: device SparkFun-Connectors:POWER_JACK_PTH -> J-Generic-5.5mm-Barrel-Jack:POWER_JACK

Commit message: rebase: backup work
Parts:
- R21: value TBD -> 10k
- U6: value LM2901QPWRQ1PW14-M -> TLC3704IPWRPW14-M; device U-TI-LM2901:PW14-M -> U-TI-TLC3704:14-TSSOP
Changed lines of the file:
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@@
 <attribute name="VALUE" x="42.27" y="79.032" size="0.6096" layer="27" font="vector" ratio="20" rot="R180"/>
 </element>
-<element name="U6" library="U-TI-LM2901" package="PW14-M" value="LM2901QPWRQ1PW14-M" x="60" y="84" smashed="yes">
+<element name="U6" library="U-TI-TLC3704" package="14-TSSOP" value="TLC3704IPWRPW14-M" x="60" y="84" smashed="yes">
 <attribute name="DATASHEET_URL" value="http://www.ti.com/lit/gpn/LM2901-Q1" x="60" y="84" size="1.778" layer="27" display="off"/>
 <attribute name="DESCRIPTION" value="Automotive Catalog Quad Differential Comparator" x="60" y="84" size="1.778" layer="27" display="off"/>
@@
 <attribute name="VALUE" x="87" y="62.857" size="0.6096" layer="27" font="vector" ratio="20" align="top-center"/>
 </element>
-<element name="R21" library="oresat-rcl" package=".0603-A" value="TBD" x="83" y="64" smashed="yes" rot="R180">
+<element name="R21" library="oresat-rcl" package=".0603-A" value="10k" x="83" y="64" smashed="yes" rot="R180">
 <attribute name="NAME" x="80.9" y="64.3" size="0.635" layer="25" font="vector" ratio="20" rot="R180"/>
 <attribute name="NAME" x="83" y="64" size="0.3" layer="33" ratio="15" rot="R180" align="center"/>

Commit message: mostly finished octavo card
Connections:
- net GND: now also U$2.P1_17
- net THERM+: now also U$2.P1_19; no longer U$2.P1_17
Routing:
- net THERM+: track 81.2 -> 81.8 mm
