File: PIRT1280A1-12-carrier/PIRT1280A1-12-carrier.sch (EAGLE design)
At the start: 159 parts, among them J1 455-1750-1-ND, J10 455-1750-1-ND, J12 USB_A_SMT_FEMALE, J14 POWER_JACK, J3 455-1750-1-ND, J4 455-1750-1-ND, J6 455-1750-1-ND, J9 5-1734592-0, Q1 35A/25V/8.5mΩ, U1 LT3042IMSE#TRPBF, U2 LT3042IMSE#TRPBF, U3 LT3042IMSE#TRPBF, U4 LT3042IMSE#TRPBF, U5 LT3042IMSE#TRPBF, U6 TLC3704IPWRPW14-M, U7 DS90CR218AMTD/NOPBMTD48_TEX-L, X1 16MHz

Commit message: mostly finished octavo card
Connections:
- net GND: now also U$2G$1.P1_17
- net THERM+: now also U$2G$1.P1_19; no longer U$2G$1.P1_17
Changed lines of the file:
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@@
 <segment>
 <pinref part="GND21" gate="1" pin="GND"/>
-<wire x1="129.54" y1="-5.08" x2="142.24" y2="-5.08" width="0.1524" layer="91"/>
+<wire x1="129.54" y1="-5.08" x2="137.16" y2="-5.08" width="0.1524" layer="91"/>
 <pinref part="U$2" gate="G$1" pin="P1_15"/>
 <pinref part="JP3" gate="G$1" pin="2"/>
+<wire x1="137.16" y1="-5.08" x2="142.24" y2="-5.08" width="0.1524" layer="91"/>
 <wire x1="129.54" y1="-2.54" x2="129.54" y2="-5.08" width="0.1524" layer="91"/>
 <junction x="129.54" y="-5.08"/>
+<pinref part="U$2" gate="G$1" pin="P1_17"/>
+<wire x1="142.24" y1="-7.62" x2="137.16" y2="-7.62" width="0.1524" layer="91"/>
+<wire x1="137.16" y1="-7.62" x2="137.16" y2="-5.08" width="0.1524" layer="91"/>
+<junction x="137.16" y="-5.08"/>
 </segment>
 <segment>
@@
 <pinref part="R21" gate="R" pin="1"/>
 <wire x1="101.6" y1="-33.02" x2="109.22" y2="-33.02" width="0.1524" layer="91"/>
-<pinref part="U$2" gate="G$1" pin="P1_17"/>
-<wire x1="142.24" y1="-7.62" x2="134.62" y2="-7.62" width="0.1524" layer="91"/>
-<wire x1="134.62" y1="-7.62" x2="134.62" y2="-20.32" width="0.1524" layer="91"/>
-<wire x1="134.62" y1="-20.32" x2="124.46" y2="-20.32" width="0.1524" layer="91"/>
-<wire x1="124.46" y1="-20.32" x2="124.46" y2="-33.02" width="0.1524" layer="91"/>
+<wire x1="124.46" y1="-10.16" x2="124.46" y2="-33.02" width="0.1524" layer="91"/>
 <wire x1="124.46" y1="-33.02" x2="109.22" y2="-33.02" width="0.1524" layer="91"/>
 <junction x="109.22" y="-33.02"/>
 <pinref part="C18" gate="CE" pin="1"/>
-</segment>
-</net>
+<pinref part="U$2" gate="G$1" pin="P1_19"/>
+<wire x1="124.46" y1="-10.16" x2="142.24" y2="-10.16" width="0.1524" layer="91"/>
+</segment>
+</net>
