File: PIRT1280A1-12-breakout/PIRT1280A1-12-breakout.sch (EAGLE design)
At the start: 39 parts, among them U1 PIRT1280A1-12

Commit message: mostly finished PIRT breakout
Parts:
- removed C1, C2, C3, C4, C5: 100n, oresat-rcl:C-EU0603-C-NOSILK
- removed JP10, JP5, JP6, JP7, JP8, JP9: (no value), pinhead:PINHD-1X2
- removed JP3: (no value), pinhead:PINHD-1X7
- removed JP4: (no value), pinhead:PINHD-1X25
- removed TP10, TP11, TP12, TP13, TP14, TP15, TP16, TP17, TP18, TP19, TP2, TP20, TP21, TP22, TP23, TP3, TP4, TP5, TP6, TP7, TP8, TP9: TEST-POINT-LARGE-SQUARE, oresat-misc:TEST-POINT-LARGE-SQUARE
- added C100, C101, C102, C103, C104: 100n, oresat-rcl:C-EU0805-A
- added J1: 5-1734592-0, J-TEConnectivity-X-1734592-X:5-1734592-0
- added JAMSYNC, REFCLK, SDCLK, SDIN, SDOUT, THERM+, THERM-: TEST-POINT-LARGE-SQUARE, oresat-misc:TEST-POINT-LARGE-SQUARE
- added TEC+, TEC-, VDETCOM, VPH, VPL, VPOS, VPOUT: TEST-POINT_SMD-SMD-10SN, oresat-misc:TEST-POINT_SMD-SMD-10SN
- JP1: device pinhead:PINHD-1X8 -> pinhead:PINHD-1X2
- JP2: device pinhead:PINHD-1X10 -> pinhead:PINHD-1X2
Connections:
- removed net N$1: JP2.1, TP2.1
- removed net N$2: JP3.7, TP9.1
- removed net N$3: JP3.6, TP8.1
- removed net N$4: JP3.5, TP7.1
- removed net N$5: JP3.4, TP6.1
- removed net N$6: JP3.3, TP5.1
- removed net N$7: JP3.2, TP4.1
- removed net N$8: JP3.1, TP3.1
- removed net VEDETCOM-2.9V: C2.1, JP2.3, TP17.1, U1G$1.VDETCOM
- removed net VPH-3.3V: C5.1, JP4.20, TP21.1, U1G$1.VPH
- removed net VPL-1.6V: C4.1, JP4.18, TP22.1, U1G$1.VPL
- removed net VPOS-3.3V: C1.1, JP2.5, TP18.1, U1G$1.VPOS
- removed net VPOUT-0.9V: C3.1, JP4.1, TP23.1, U1G$1.VPOUT
- new net VDETCOM: C102.1, J1.39, J1.40, U1G$1.VDETCOM~2.9V, VDETCOM.TP
- new net VPH: C100.1, J1.15, J1.16, U1G$1.VPH-3.3V, VPH.TP
- new net VPL: C101.1, J1.18, J1.19, U1G$1.VPL-1.6V, VPL.TP
- new net VPOS: C103.1, J1.12, J1.13, U1G$1.VPOS-3.3V, VPOS.TP
- new net VPOUT: C104.1, J1.36, J1.37, U1G$1.VPOUT-0.9V, VPOUT.TP
- net GND: now also C100.2, C101.2, C102.2, C103.2, C104.2, J1.11, J1.14, J1.17, J1.20, J1.23, J1.26, J1.29, J1.3, J1.32, J1.35, J1.38, J1.41, J1.44, J1.48, J1.49, J1.50, J1.7, J1.PAD, JP1.1, JP1.2, JP2.1; no longer C1.2, C2.2, C3.2, C4.2, C5.2, JP1.3, JP1.6, JP10.1, JP10.2, JP2.10, JP2.4, JP2.6, JP4.11, JP4.14, JP4.17, JP4.19, JP4.2, JP4.21, JP4.23, JP4.25, JP4.5, JP4.8, JP5.1, JP5.2, JP6.1, JP6.2, JP7.1, JP7.2, JP8.1, JP8.2, JP9.1, JP9.2
- net JAMSYNC: now also J1.2, JAMSYNC.1; no longer JP4.24, TP19.1
- net OUT1_N: now also J1.24; no longer JP4.13
- net OUT1_P: now also J1.25; no longer JP4.12
- net OUT2_N: now also J1.27; no longer JP4.10
- net OUT2_P: now also J1.28; no longer JP4.9
- net OUT3_N: now also J1.30; no longer JP4.7
- net OUT3_P: now also J1.31; no longer JP4.6
- net OUT4_N: now also J1.33; no longer JP4.4
- net OUT4_P: now also J1.34; no longer JP4.3
- net REFCLK: now also J1.1, REFCLK.1; no longer JP4.22, TP20.1
- net SDCLK: now also J1.46, SDCLK.1; no longer JP2.8, TP10.1
- net SDIN: now also J1.47, SDIN.1; no longer JP2.9, TP11.1
- net SDOUT: now also J1.45, SDOUT.1; no longer JP2.7, TP12.1
- net TEC+: now also J1.4, J1.5, J1.6, TEC+.TP; no longer JP1.1, JP1.2, TP14.1
- net TEC-: now also J1.10, J1.8, J1.9, TEC-.TP; no longer JP1.7, JP1.8, TP13.1
- net THERM+: now also J1.42, THERM+.1; no longer JP1.5, TP15.1
- net THERM-: now also J1.43, THERM-.1; no longer JP1.4, TP16.1
- net TXCLK_N: now also J1.21; no longer JP4.16
- net TXCLK_P: now also J1.22; no longer JP4.15
Other:
- note added: "TODO RENUMBER!!!"
- note added: "TODO TEST POINTS?"
- moved on the sheet: U1G$1, U1G$2

Commit message: mostly finished with PIRT1280 carrier
Other:
- note removed: "TODO RENUMBER!!!"
- moved on the sheet: C100, C101, C102, C103, C104, J1, JP1, JP2, U1G$1, U1G$2

Commit message: address review comments
Other:
- note removed: "TODO TEST POINTS?"
- moved on the sheet: U1G$2
Changed lines of the file:
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@@
 <?xml version="1.0" encoding="utf-8"?>
 <!DOCTYPE eagle SYSTEM "eagle.dtd">
-<eagle version="9.5.2">
+<eagle version="9.6.2">
 <drawing>
 <settings>
@@
 <sheet>
 <plain>
-<text x="303.53" y="119.38" size="3.81" layer="97">TODO TEST POINTS?</text>
 </plain>
 <instances>
@@
 <attribute name="VALUE" x="91.44" y="106.68" size="1.778" layer="96" ratio="20"/>
 </instance>
-<instance part="U1" gate="G$2" x="283.21" y="121.92" smashed="yes">
-<attribute name="NAME" x="283.21" y="93.98" size="1.778" layer="95" ratio="20"/>
-<attribute name="VALUE" x="283.21" y="91.44" size="1.778" layer="96" ratio="20"/>
+<instance part="U1" gate="G$2" x="13.97" y="33.02" smashed="yes">
+<attribute name="NAME" x="13.97" y="5.08" size="1.778" layer="95" ratio="20"/>
+<attribute name="VALUE" x="13.97" y="2.54" size="1.778" layer="96" ratio="20"/>
 </instance>
 <instance part="FRAME1" gate="G$1" x="1.27" y="0" smashed="yes"/>

Commit message: rebase: backup work
Changed lines of the file:
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@@
 <wire x1="48.26" y1="139.7" x2="35.56" y2="139.7" width="0.1524" layer="91"/>
 <label x="38.1" y="139.7" size="1.27" layer="95"/>
-<label x="203.2" y="55.88" size="1.778" layer="95"/>
+<label x="203.2" y="58.42" size="1.778" layer="95"/>
 <wire x1="35.56" y1="139.7" x2="35.56" y2="58.42" width="0.1524" layer="91"/>
 <pinref part="J1" gate="G$1" pin="46"/>
@@
 <pinref part="U1" gate="G$1" pin="SDIN"/>
 <label x="38.1" y="137.16" size="1.27" layer="95"/>
-<label x="203.2" y="58.42" size="1.778" layer="95"/>
+<label x="203.2" y="55.88" size="1.778" layer="95"/>
 <pinref part="J1" gate="G$1" pin="47"/>
 <wire x1="33.02" y1="137.16" x2="48.26" y2="137.16" width="0.1524" layer="91"/>
