File: cfc-sensor-card/cfc-sensor-card.brd (EAGLE design)
At the start: 99.8 x 94.6 mm, 139 parts, among them J2 J-SAMTEC-TFM-110-X1-XXX-D-RA, J4 TFM-120-01-L-D-RA, Q1 35A/25V/8.5mΩ, Q2 PMV45EN, Q3 DMP2240UDM, Q4 PMV45EN, Q5 MOSFET-PCH-SOT23-6, Q6 MOSFET-PCH-SOT23-6, U1 PIRT1280A1-12, U12 MIC842LYC5, U13 MIC842LYC5, U14 MAX4211FETE, U16 MAX7310ATE, U2 LT3042IMSE#TRPBF, U3 LT3042IMSE#TRPBF, U4 LT3042IMSE#TRPBF, U5 LT3042IMSE#TRPBF, U6 LT3042IMSE#TRPBF, U7 TLC3704IPWRPW14-M, X1 16MHz

Commit message: mostly finished sensor card
Parts:
- removed R21: 1k, oresat-rcl:.0603-A
- removed TP65, TP66: TEST-POINT_SMD-SMD-10SN, oresat-misc:TESTPOINT_SMD-10SN
- added C18: 1uF, oresat-rcl:.0603-B
- added C19: 4.7u, oresat-rcl:.0603-B
- added C20: 0.1u, oresat-rcl:.0603-B
- added D2: GREEN, SparkFun-LED:LED-0603
- added Q7: MOSFET-PCH-SOT23-6, Q-MOSFET-PCH-SOT23-6:SOT23-6
- added Q8: PMV45EN, Tova:SOT23
- added R10, R8, R9: 10k, oresat-rcl:.0603-B
- added R11: 1k, oresat-rcl:.0603-B
- added U8: LP2985AIM5-3.3_NOPB, U-TI-LP2985AIM5-3.3_NOPB-3.3V-Fixed-LDO:SOT-23
- C1, C10, C11, C12, C13, C14, C15, C16, C17, C2, C3, C4, C5, C6, C7, C8, C9, R1, R3, R4, R5, R6, R7: device oresat-rcl:.0603-A -> oresat-rcl:.0603-B
- C40: value 0.1u -> 1u; device oresat-rcl:.0603-A -> oresat-rcl:.0603-B
- Q1: value 35A/25V/8.5mΩ -> MOSFET-PCH-SOT23-6; device Q-Fairchild-FDD8780-MOSFET-NCH:DPAK -> Q-MOSFET-PCH-SOT23-6:SOT23-6
- R18: device oresat-rcl:.0805-A -> oresat-rcl:.0603-B
- R19: value 20k -> 10k; device oresat-rcl:.0805-A -> oresat-rcl:.0603-B
- R27: device oresat-rcl:.0402-C-NOSILK -> oresat-rcl:.0402-A
- TP40: value TEST-POINT-LARGE-SQUARE -> TEST-POINT_SMD-SMD-10SN; device oresat-misc:1X01 -> oresat-misc:TESTPOINT_SMD-10SN
- moved TP40 223.4 mm to (59.1, 75.8)
- moved R27 205.6 mm to (15.5, 69.0), flipped to the bottom, turned to 90 degrees
- moved C11 201.2 mm to (10.0, 69.0), flipped to the bottom, turned to 90 degrees
- moved X1 197.4 mm to (13.0, 69.0), flipped to the bottom, turned to 180 degrees
- moved Q1 180.5 mm to (69.5, 20.6), flipped to the bottom
- moved C3 124.8 mm to (71.5, 80.5), flipped to the bottom
- moved C4 117.3 mm to (71.5, 74.0), flipped to the bottom
- moved C2 109.6 mm to (32.0, 71.5), flipped to the bottom, turned to 90 degrees
- moved TP39 107.5 mm to (15.5, 34.5), flipped to the bottom, turned to 270 degrees
- moved TP27 96.9 mm to (15.0, 62.5), turned to 90 degrees
- moved TP18 96.6 mm to (11.0, 62.5), turned to 90 degrees
- moved C17 87.8 mm to (16.5, 42.0), flipped to the bottom, turned to 90 degrees
- moved C40 87.7 mm to (6.50, 40.5), flipped to the bottom, turned to 270 degrees
- moved D1 83.7 mm to (41.0, 4.50), flipped to the bottom
- moved R20 75.8 mm to (12.5, 56.5), flipped to the bottom, turned to 90 degrees
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Connections:
- removed net N$19: Q1.4, U1.22
- removed net N$30: Q1.3, R21.2
- new net N$12: D2.A, R11.1
- new net N$18: C20.1, U8.4
- new net N$2: R19.1, R8.2
- new net N$3: Q1.3, Q7.3, Q8.3, R9.1
- new net TEC+: Q1.1, Q1.2, Q1.5, Q1.6, Q7.1, Q7.2, Q7.5, Q7.6, R11.2, U1.23
- net 3.3V: now also C19.1, U8.5
- net GND: now also C18.2, C19.2, C20.2, D2.C, Q8.2, R10.1, U1.22, U8.2
- net N$16: now also TP40.TP; no longer TP40.1
- net OUT1N: now also J2.5, J2.6; no longer J2.1, J2.2
- net OUT1P: now also J2.7, J2.8; no longer J2.3, J2.4
- net PEN-SCL-FILT: no longer TP66.TP
- net PEN-SDA-FILT: no longer TP65.TP
- net SENSOR_ENABLE: now also R8.1; no longer R19.1
- net TEC_ENABLE: now also Q8.1, R10.2; no longer Q1.1, R20.2, R21.1
- net TXCLKN: now also J2.1, J2.2; no longer J2.5, J2.6
- net TXCLKP: now also J2.3, J2.4; no longer J2.7, J2.8
- net VBUSP: now also C18.1, Q1.4, Q7.4, R9.2, U8.1, U8.3; no longer U1.23
Routing:
- net N$1: track 0.00 -> 187.8 mm, vias 0 -> 5
- net N$36: track 0.00 -> 153.0 mm, vias 0 -> 3
- net TEC_ENABLE: track 0.00 -> 146.8 mm, vias 0 -> 2
- net N$10: track 0.00 -> 86.6 mm, vias 0 -> 2
- net VPD: track 0.00 -> 86.6 mm, vias 0 -> 5
- net 3.3V: track 0.00 -> 69.2 mm, vias 0 -> 2
- net N$17: track 0.00 -> 63.3 mm, vias 0 -> 1
- net GND: track 0.00 -> 61.5 mm, vias 15 -> 132
- net SENSOR_ENABLE: track 0.00 -> 60.2 mm, vias 0 -> 1
- net OPD_SDA: track 0.00 -> 47.2 mm, vias 0 -> 1
- net OPD_SCL: track 0.00 -> 45.1 mm, vias 0 -> 1
- net PEN-SCL-FILT: track 0.00 -> 43.9 mm, vias 0 -> 5
- net TXCLKN: track 0.00 -> 41.4 mm
- net OUT1N: track 0.00 -> 41.3 mm
- net REFCLK_ENABLE: track 0.00 -> 40.9 mm, vias 0 -> 3
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- added copper zone on layer 16, net N$98
- added copper zone on layer 16, net N$99
- added copper zone on layer 1, net TEC+
- added copper zone on layer 16, net TEC+
- added copper zone on layer 16, net VBUS
- added copper zone on layer 15, net VBUSP
- added copper zone on layer 16, net VBUSP
- added copper zone on layer 16, net VDETCOM-2.9V
- added copper zone on layer 16, net VPH-3.3V
- added copper zone on layer 16, net VPL-1.6V
- added copper zone on layer 16, net VPOS-3.3V
- added copper zone on layer 16, net VPOUT-0.9V
Other:
- board text added: "2021/07/27"
- board text added: "Inner pin signal should be 3.15mm longer that outer pin signal for the pair to be balanced because of the pin row offset"
- board text added: "ON/OFF"
- board text added: "OreSat CFC Sensor Card v1.0"
- board text added: "SENSOR ENABLE"
- board text added: "TEC PWR"
- board text removed: "2020/12/08"
- board text removed: "BOOT SELECT"
- board text removed: "DEFAULT : 0b11x00"
- board text removed: "NOTE: SYSBOOT[2] is not set by default. It must be set with J3 or JP107, BUT NOT BOTH. See AM335x TRM Table 26-7 for details."
- board text removed: "ON/ OFF"
- board text removed: "OreSat Star Tracker v1.2"
- board text removed: "SYSBOOT [4:0]"
- board text removed: "eMMC"
- board text removed: "eMMC : 0b11100"
- board text removed: "uSD"
- board text removed: "uSD : 0b11000"

Commit message: mostly finished octavo card
Parts:
- removed Q1: MOSFET-PCH-SOT23-6, Q-MOSFET-PCH-SOT23-6:SOT23-6
- moved Q7 2.50 mm to (69.5, 19.0)
- moved Q8 2.50 mm to (69.5, 15.0)
- moved R10 2.50 mm to (72.5, 15.0)
- moved R9 2.50 mm to (66.5, 15.0)
Connections:
- net N$3: no longer Q1.3
- net TEC+: no longer Q1.1, Q1.2, Q1.5, Q1.6
- net VBUSP: no longer Q1.4
Routing:
- net N$3: track 10.6 -> 5.41 mm, vias 2 -> 0
- net TEC+: track 19.0 -> 21.2 mm
- net VBUSP: track 32.5 -> 34.3 mm
- net TEC_ENABLE: track 146.8 -> 145.8 mm

Commit message: oh god almost done
Parts:
- added U$2: (no value), oresat-misc:ORESAT_ORIENTATION_COPPER
Routing:
- net N$3: track 5.41 -> 4.70 mm
