File: cfc-sensor-card/cfc-sensor-card.brd (EAGLE design)
At the start: 99.8 x 94.6 mm, 147 parts, among them J2 J-SAMTEC-TFM-110-X1-XXX-D-RA, J4 TFM-120-01-L-D-RA, Q2 PMV45EN, Q3 DMP2240UDM, Q4 PMV45EN, Q5 MOSFET-PCH-SOT23-6, Q6 MOSFET-PCH-SOT23-6, Q7 MOSFET-PCH-SOT23-6, Q8 PMV45EN, U1 PIRT1280A1-12, U12 MIC842LYC5, U13 MIC842LYC5, U14 MAX4211FETE, U16 MAX7310ATE, U2 LT3042IMSE#TRPBF, U3 LT3042IMSE#TRPBF, U4 LT3042IMSE#TRPBF, U5 LT3042IMSE#TRPBF, U6 LT3042IMSE#TRPBF, U7 TLC3704IPWRPW14-M, U8 LP2985AIM5-3.3_NOPB, X1 16MHz

Commit message: boards finished
Parts:
- added C21: NP, oresat-rcl:.0603-B
- added R12, R13, R14: NP, oresat-rcl:.0402-C-NOSILK
- added R15: 0, oresat-rcl:.0603-B
- C100, C101, C102, C103, C104: device oresat-rcl:.0805-A -> oresat-rcl:.0603-B
- moved TP40 3.77 mm to (56.7, 78.6)
- moved Q8 3.00 mm to (72.5, 15.0)
- moved R10 3.00 mm to (75.5, 15.0)
- moved C103 1.00 mm to (54.7, 22.2)
- moved C100 0.75 mm to (60.0, 76.8)
- moved C101 0.75 mm to (58.0, 76.8)
- moved C104 0.56 mm to (41.6, 76.8)
- moved U$1 0.50 mm to (5.70, 10.4)
Connections:
- new net N$11: R12.2, U1.11
- new net N$19: R12.1, U1.12
- new net N$21: R13.2, U1.9
- new net N$22: R13.1, U1.10
- new net N$26: R14.2, U1.7
- new net N$30: R14.1, U1.8
- new net N$31: Q8.3, R15.1
- net N$3: now also C21.2, R15.2; no longer Q8.3
- net VBUSP: now also C21.1
Routing:
- net GND: track 61.5 -> 92.6 mm, vias 132 -> 194
- net N$19: track 0.00 -> 6.17 mm
- net N$22: track 0.00 -> 6.15 mm
- net N$30: track 0.00 -> 6.14 mm
- net N$31: track 0.00 -> 3.80 mm
- net N$16: track 4.18 -> 7.81 mm
- net N$26: track 0.00 -> 3.11 mm
- net N$21: track 0.00 -> 3.09 mm
- net N$11: track 0.00 -> 3.08 mm
- net TEC_ENABLE: track 145.8 -> 148.8 mm
- net N$36: track 153.0 -> 151.5 mm
- net N$17: track 63.3 -> 64.6 mm
- net VBUSP: track 34.3 -> 35.5 mm
- net N$1: track 187.8 -> 187.0 mm
- net VPOS-3.3V: track 10.9 -> 11.6 mm
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Other:
- board text added: "2021/08/01"
- board text added: "GND"
- board text added: "VDETCOM-2.9V"
- board text added: "VPH-3.3V"
- board text added: "VPL-1.6V"
- board text added: "VPOS-3.3V"
- board text added: "VPOUT-0.9V"
- board text removed: "10.5mm Solar Card Opening"
- board text removed: "2021/07/27"
- board text removed: "MAKE SURE CAMERA BOARD CONNECTOR IS CORRECT ORIENTATION"
- board text removed: "Min. Cable Length: 28.625mm FFC Cable: Molex 0151660381 29.97mm"

Commit message: update attrs
Parts:
- C100, C101, C102, C103, C104: value 100n -> 0.1u
- C18, C32, C33, C34, C35: value 1uF -> 1u
- C39: value 0.1uF -> 0.1u

Commit message: Updated OPD address resistors, LED resistors (AAAAAUGH MY EYES), and OPD shunt resistor to give the CFC sensor card addrss 0x1E and a 2.95 A current limit.
Parts:
- R1: value 1k -> 2.7k
- R11: value 1k -> 10k
- R53, R55, R58: value NP -> 10k
- R61: value 2.7k -> 10k
- R63: value 100m -> 10m
