File: cfc-card/cfc-card.brd (EAGLE design)
At the start: 99.8 x 94.6 mm, 273 parts, among them J1 ORESAT-DEBUG-CONNECTOR-CARD, J100 DM3BT-DSF-PEJS, J2 J-SAMTEC-TFM-110-X1-XXX-D-RA, J4 TFM-120-01-L-D-RA, Q1 MMBT2907, Q2 PMV45EN, Q3 DMP2240UDM, Q4 PMV45EN, Q5 MOSFET-PCH-SOT23-6, Q6 MOSFET-PCH-SOT23-6, U1 RCLAMP0504FB, U10 TLVH431, U11 TCAN330, U12 MIC842LYC5, U13 MIC842LYC5, U14 MAX4211FETE, U15 TPS62112, U16 MAX7310ATE, U17 25AAXX, U18 RCLAMP0504FB, U3 THGBMJG7C2LBAU8, U4 SN74LVC1G07DCK, U7 OSD3358-512M-BSM, Y1 24MHz, Y2 ABS07-32.768KHZ-T

Commit message: rebase: backup work
Parts:
- removed JP100, JP101, JP104: JUMPER-SMT_2_NC_TRACE_SILK, SparkFun-Jumpers:SMT-JUMPER_2_NC_TRACE_SILK
- removed TP1, TP100, TP101, TP103, TP104, TP105, TP106, TP107, TP108, TP111, TP114, TP115, TP117, TP118, TP120, TP122, TP123, TP124, TP125, TP126, TP127, TP128, TP131, TP134, TP135, TP137, TP143, TP145, TP147, TP148, TP149, TP150, TP152, TP153, TP158, TP159, TP162, TP169, TP170, TP172, TP174, TP175, TP176, TP179, TP180, TP181, TP30, TP38: TEST-POINT3X4, SparkFun-Connectors:PAD.03X.04
- added C1, C16, C17, C20, C28, C7: 1n, oresat-rcl:.0402-C-NOSILK
- added C21, C23, C24, C25, C26, C27: 10n, oresat-rcl:.0402-C-NOSILK
- added C42, C43, C45, C46, C47, C48: 100n, oresat-rcl:.0402-C-NOSILK
- added C49: 10u, oresat-rcl:.0603-C-NOSILK
- added R6, R7: 100, oresat-rcl:.0402-C-NOSILK
- added TP13, TP15, TP16, TP17: TEST-POINT3X4, SparkFun-Connectors:PAD.03X.04
- added U2: DS90CR218AMTD/NOPBMTD48_TEX-L, U-TI-DS90CR218-LVDSReceiver:MTD48_TEX-L
- C40: value 0.1uF -> DNP
- J5: value (none) -> 455-1750-1-ND; device SparkFun-Connectors:1X02 -> SparkFun-Connectors:1X03
- R29, R30: value 4.7k -> NP; device oresat-rcl:.0603-A -> oresat-rcl:.0402-C-NOSILK
- moved TP112 153.5 mm to (-70.6, 36.3)
- moved TP142 153.5 mm to (-73.6, 39.3)
- moved TP146 153.5 mm to (-74.6, 40.3)
- moved TP151 153.5 mm to (-71.6, 37.3)
- moved TP155 153.5 mm to (-72.6, 38.3)
- moved TP164 153.5 mm to (-74.1, 42.6)
- moved TP165 153.5 mm to (-76.2, 42.6)
- moved TP4 143.6 mm to (-76.0, -15.0), turned to 0 degrees
- moved J5 118.1 mm to (-39.0, 81.0)
- moved TP102 106.7 mm to (-41.1, 31.7)
- moved TP109 106.7 mm to (-58.0, 32.3)
- moved TP110 106.7 mm to (-59.1, 33.2)
- moved TP121 106.7 mm to (-45.5, 35.5)
- moved TP129 106.7 mm to (-48.2, 37.5)
- moved TP130 106.7 mm to (-46.0, 37.5)
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Connections:
- net AUX-5 renamed TEC_ENABLE
- net AUX-6 renamed THERM+
- net AUX-7 renamed SENSOR_ENABLE
- net AUX-8 renamed SPI_MISO
- net AUX-9 renamed SPI_CLK
- net AUX_!SHUTDOWN renamed SPI_MOSI
- removed net AUX-1: J2.1, J2.2
- removed net AUX-2: J2.3, J2.4
- removed net AUX-3: J2.5, J2.6
- removed net AUX-4: J2.7, J2.8
- removed net BUS_OE: U7.F14
- removed net CAM_OE: U7.F15
- removed net CLK_EN: U7.E16
- removed net FLASH: U7.G15
- removed net INPUT_EN: U7.E14
- removed net N$36: TP123.P$1, U7.P5
- removed net N$37: TP115.P$1, U7.R5
- removed net N$38: TP105.P$1, U7.T5
- removed net N$39: TP124.P$1, U7.P6
- removed net N$40: TP120.P$1, U7.R6
- removed net N$407: JP104.2, Q1.C, R31.1, U10.3
- removed net N$41: TP125.P$1, U7.N14
- removed net N$42: TP114.P$1, U7.P15
- removed net N$43: TP111.P$1, U7.R16
- removed net N$46: TP162.P$1, U7.F1
- removed net N$47: TP153.P$1, U7.F3
- removed net N$48: TP152.P$1, U7.F2
- removed net N$49: TP159.P$1, U7.E1
- removed net N$50: TP143.P$1, U7.J14
- removed net N$51: TP174.P$1, U7.D13
- removed net N$52: TP158.P$1, U7.E13
- removed net N$53: TP147.P$1, U7.H16
- removed net N$54: TP137.P$1, U7.H15
- removed net N$55: TP149.P$1, U7.H14
- removed net N$56: TP135.P$1, U7.G16
- removed net N$57: TP172.P$1, U7.D12
- removed net N$58: TP150.P$1, U7.J6
- removed net N$59: TP145.P$1, U7.K4
- removed net N$66: TP179.P$1, U7.C9
- removed net N$67: TP169.P$1, U7.C8
- removed net N$68: TP176.P$1, U7.C7
- removed net N$69: TP175.P$1, U7.C6
- removed net N$70: TP181.P$1, U7.B6
- removed net N$71: TP38.P$1, U7.B8
- removed net N$75: TP106.P$1, U7.T7
- removed net N$76: TP100.P$1, U7.T12
- removed net N$77: TP118.P$1, U7.R12
- removed net N$78: TP126.P$1, U7.P12
- removed net N$79: TP101.P$1, U7.T13
- removed net N$82: TP108.P$1, U7.T15
- removed net N$83: TP117.P$1, U7.R15
- removed net N$84: TP103.P$1, U7.T16
- removed net N$85: TP122.P$1, U7.P3
- removed net N$86: TP107.P$1, U7.R7
- removed net N$93: TP134.P$1, U7.M1
- removed net N$94: TP131.P$1, U7.N3
- removed net N$95: TP127.P$1, U7.N2
- removed net N$96: TP128.P$1, U7.N1
- removed net N$97: TP148.P$1, U7.G14
- removed net RESET: U7.D16
- removed net SADDR: U7.D15
- removed net SCL_2: R30.2, U7.A10
- removed net SDA_2: R29.2, U7.B10
- removed net STANDBY: U7.D14
- removed net TRIGGER: U7.E15
- removed net VREG_EN: U7.F16
- new net !PWR_DWN: J5.2, U2.22
- new net N$112: TP13.P$1, U7.A10
- new net N$119: TP16.P$1, U7.L16
- new net N$120: TP17.P$1, U7.M15
- new net OUT1N: J2.5, J2.6, R6.2, U2.8
- new net OUT1P: J2.7, J2.8, R6.1, U2.9
- new net PRU0: U2.24
- new net PRU1: U2.26
- new net PRU16_CLK: U2.23
- new net PRU2: U2.27
- new net PRU3: U2.29
- new net PRU4: U2.30
- new net PRU5: U2.31
- new net PRU6: U2.33
- new net SERDES_PWR_DOWN: J5.1
- new net TXCLKN: J2.1, J2.2, R7.1, U2.16
- new net TXCLKP: J2.3, J2.4, R7.2, U2.17
- net 3.3V: now also C1.1, C16.1, C17.1, C20.1, C21.1, C23.1, C24.1, C25.1, C26.1, C27.1, C28.1, C42.1, C43.1, C45.1, C46.1, C47.1, C48.1, C49.1, C7.1, J5.3, U2.12, U2.20, U2.28, U2.36, U2.42, U2.48; no longer R29.1, R30.1
- net 3.3VA: now also Q1.E, R23.2, R28.2; no longer JP101.1
- net GND: now also C1.2, C16.2, C17.2, C20.2, C21.2, C23.2, C24.2, C25.2, C26.2, C27.2, C28.2, C42.2, C43.2, C45.2, C46.2, C47.2, C48.2, C49.2, C7.2, U2.13, U2.18, U2.19, U2.21, U2.25, U2.3, U2.32, U2.38, U2.44, U2.7, U3.A6, U7.L14; no longer JP100.2
- net N$102: now also TP15.P$1, U7.L15; no longer JP100.1, U7.L14
- net N$118: now also Q1.C, R31.1, U10.3; no longer JP104.1
- net N$20: now also TP4.P$1, U7.B10; no longer JP101.2, Q1.E, R23.2, R28.2
- net N$3: now also R29.2, U2.14; no longer TP170.P$1, U7.D7
- net N$33: now also R29.1, U2.15; no longer TP30.P$1, U7.A4
- net N$34: now also R30.2, U2.10; no longer TP180.P$1, U7.C5
- net N$35: now also R30.1, U2.11; no longer TP104.P$1, U7.T4
- net N$401: no longer TP4.P$1
- net USB_HO_N: no longer U1.6, U7.L16
- net USB_HO_PX: no longer U1.4, U7.L15
- net USB_HO_VBUS: no longer J5.1, TP1.P$1, U7.M15
- net VDD: no longer J5.2
Routing:
- net 3.3V: track 166.2 -> 3.13 mm, vias 40 -> 1
- net EEPROM_WP: track 92.5 -> 0.00 mm, vias 2 -> 0
- net I2C0_SCL: track 89.7 -> 0.00 mm, vias 2 -> 0
- net I2C0_SDA: track 87.9 -> 0.00 mm, vias 2 -> 0
- net TRIGGER: track 85.7 -> 0.00 mm, vias 2 -> 0
- net SADDR: track 85.6 -> 0.00 mm, vias 2 -> 0
- net VREG_EN: track 84.1 -> 0.00 mm, vias 2 -> 0
- net STANDBY: track 84.0 -> 0.00 mm, vias 2 -> 0
- net UART0_TX: track 81.8 -> 0.00 mm, vias 2 -> 0
- net RESET: track 81.4 -> 0.00 mm, vias 2 -> 0
- net CAM_OE: track 80.8 -> 0.00 mm, vias 2 -> 0
- net N$582: track 79.5 -> 0.00 mm, vias 3 -> 0
- net USB_HO_VBUS: track 79.1 -> 0.00 mm, vias 2 -> 0
- net UART0_RX: track 78.5 -> 0.00 mm, vias 2 -> 0
- net CLK_EN: track 77.6 -> 0.00 mm, vias 2 -> 0
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- added copper zone on layer 16, net GND1
- added copper zone on layer 15, net OPD_PWR
- added copper zone on layer 16, net OPD_PWR
- removed copper zone on layer 16, net 3.3V
- removed copper zone on layer 15, net VIN_USB
Other:
- board text added: "ON/ OFF"
- board text removed: "CAMERA"
- board text removed: "Camera Lens Center Line"
- board text removed: "FFC Cable Center Line"
- board text removed: "JTAG"
- board text removed: "ON/OFF"

Commit message: mostly finished sensor card
Parts:
- moved D6 63.2 mm to (91.9, 82.0), turned to 0 degrees
- moved R49 61.0 mm to (91.9, 80.2), turned to 0 degrees
- moved R53 40.0 mm to (68.9, 84.4)
- moved R54 40.0 mm to (70.8, 84.4)
- moved R55 40.0 mm to (72.6, 84.4)
- moved R56 40.0 mm to (74.4, 84.4)
- moved R57 40.0 mm to (76.2, 84.4)
- moved R58 40.0 mm to (78.0, 84.4)
- moved R65 40.0 mm to (68.9, 88.0)
- moved R66 40.0 mm to (70.8, 88.0)
- moved R67 40.0 mm to (72.6, 88.0)
- moved R68 40.0 mm to (74.4, 88.0)
- moved R69 40.0 mm to (76.2, 88.0)
- moved R70 40.0 mm to (78.0, 88.0)
- moved C31 10.3 mm to (38.5, 53.6)
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Routing:
- net CAN2_L: track 47.0 -> 18.7 mm, vias 1 -> 0
- net CAN2_H: track 46.2 -> 20.1 mm, vias 1 -> 0
- net ON/!OFF: track 46.4 -> 30.4 mm
- net AD2: track 24.3 -> 9.47 mm, vias 2 -> 1
- net AD1: track 18.5 -> 7.28 mm, vias 2 -> 1
- net AD0: track 14.9 -> 7.28 mm, vias 2 -> 0
- net PEN-SCL-FILT: track 52.4 -> 48.8 mm
- net VPD: track 52.8 -> 49.9 mm, vias 12 -> 9
- net PEN-SDA-FILT: track 49.2 -> 46.4 mm
- net GND: vias 112 -> 110

Commit message: mostly finished octavo card
Parts:
- removed C15: 22uF, oresat-rcl:C1210
- removed C41: 0.1uF, oresat-rcl:.0603-A
- removed J5: 455-1750-1-ND, SparkFun-Connectors:1X03
- removed JP105, JP106, JP108, JP109: JUMPER-SMT_3_1-NC_TRACE_SILK, SparkFun-Jumpers:SMT-JUMPER_3_1-NC_TRACE_SILK
- removed R24, R25, R26: 100K, R-Panasonic-EXB_A10PXXXJ:ARRAY_EXBA-M
- removed TP112, TP142, TP146, TP151, TP155, TP171, TP177, TP178, TP182, TP25, TP58, TP59, TP60, TP61, TP62: TEST-POINT3X4, SparkFun-Connectors:PAD.03X.04
- removed U18: RCLAMP0504FB, U-Semtec-RCLAMP0504FB:SC70-6
- added C50: 0.1uF, oresat-rcl:.0603-A
- added C51: 0.1u, oresat-rcl:.0603-A
- added JP1: JUMPER-SMT_2_NC_TRACE_NO-SILK, SparkFun-Jumpers:SMT-JUMPER_2_NC_TRACE_NO-SILK
- added JP3: JUMPER-SMT_2_NO_SILK, SparkFun-Jumpers:SMT-JUMPER_2_NO_SILK
- added R11, R14: DNP, oresat-rcl:.0603-A
- added R16, R17: EXB-2HV103JV, R-Panasonic-EXB-2HV103JV:RES_EXB2HV
- added R21: 10k, oresat-rcl:.0603-A
- added SB0, SB1, SB10, SB11, SB12, SB13, SB14, SB15, SB2, SB3, SB4, SB5, SB6, SB7, SB8, SB9: TEST-POINT-SMALL, oresat-misc:TEST-POINT-SMALL
- added TP1, TP18, TP19, TP20, TP21, TP23, TP24, TP26, TP27, TP28, TP29, TP30, TP31, TP32, TP33, TP34, TP70, TP71, TP72, TP74, TP75, TP77, TP78: TEST-POINT, Tova:2MM-TEST-POINT
- added TP36, TP37, TP38: TEST-POINT3X4, SparkFun-Connectors:PAD.03X.04
- TP2, TP39: value TEST-POINT3X4 -> TEST-POINT; device SparkFun-Connectors:PAD.03X.04 -> Tova:2MM-TEST-POINT
- moved TP17 157.5 mm to (67.0, 40.5)
- moved TP16 155.1 mm to (65.5, 40.5)
- moved TP13 154.6 mm to (59.5, 56.5), turned to 180 degrees
- moved TP15 152.7 mm to (64.0, 40.5)
- moved TP4 152.5 mm to (59.5, 55.0), turned to 180 degrees
- moved TP165 144.4 mm to (68.0, 50.0), flipped to the top, turned to 180 degrees
- moved TP164 140.3 mm to (66.0, 50.0), flipped to the top, turned to 180 degrees
- moved TP110 124.7 mm to (65.5, 26.5), flipped to the top
- moved TP109 120.6 mm to (62.5, 26.5), flipped to the top
- moved TP161 107.6 mm to (64.0, 42.0), flipped to the top
- moved TP166 106.7 mm to (65.5, 42.0), flipped to the top, turned to 270 degrees
- moved TP163 106.2 mm to (60.0, 40.5), turned to 0 degrees
- moved J3 105.2 mm to (12.0, 43.4)
- moved TP144 103.2 mm to (60.0, 36.0)
- moved TP160 101.8 mm to (62.5, 42.0), flipped to the top, turned to 270 degrees
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Connections:
- net N$641 renamed EMMC_DAT0
- net N$642 renamed EMMC_DAT1
- net N$643 renamed EMMC_DAT2
- net N$647 renamed EMMC_DAT6
- net N$648 renamed EMMC_DAT7
- net N$649 renamed EMMC_CMD
- net OUT1N renamed OUT1_N
- net OUT1P renamed OUT1_P
- net TXCLKN renamed TXCLK_N
- net TXCLKP renamed TXCLK_P
- removed net D10_I: U7.C3
- removed net D11_I: U7.C4
- removed net D4_I: U7.A1
- removed net D5_I: U7.A2
- removed net D6_I: U7.B2
- removed net D7_I: U7.B1
- removed net D8_I: U7.A3
- removed net D9_I: U7.B3
- removed net HSYNC_I: U7.P7
- removed net N$105: JP105.1, R24.9
- removed net N$106: JP106.1, R24.2
- removed net N$107: JP108.3, R24.3
- removed net N$108: JP109.3, R24.6
- removed net N$21: JP2.1, R25.8
- removed net N$44: TP177.P$1, U7.C12
- removed net N$45: TP178.P$1, U7.C13
- removed net N$535: JP105.2, U7.G3
- removed net N$578: JP106.2, U7.G2
- removed net N$582: J3.2, JP2.2, U7.G1
- removed net N$583: JP108.2, U7.H3
- removed net N$584: JP109.2, U7.H2
- removed net N$585: R25.4, U7.H1
- removed net N$586: R25.7, U7.J3
- removed net N$587: R26.4, U7.J1
- removed net N$588: R26.7, U7.K3
- removed net N$591: R26.3, U7.K2
- removed net N$592: R26.8, U7.K1
- removed net N$594: R26.2, U7.L3
- removed net N$595: R26.9, U7.L2
- removed net N$601: R24.4, U7.L1
- removed net N$602: R26.1, U7.M3
- removed net N$629: R26.6, U7.J2
- removed net N$630: JP109.1, R25.6
- removed net N$632: JP108.1, R25.9
- removed net N$633: JP106.3, R25.2
- removed net N$634: JP105.3, R25.3
- removed net N$644: R9.7, U3.B2, U7.T3
- removed net N$645: R9.4, U3.B3, U7.T2
- removed net N$646: R9.3, U3.B4, U7.T1
- removed net N$651: R9.8, U3.M6, U7.P2
- removed net N$652: R10.3, U3.K5, U7.R13
- removed net N$72: TP39.P$1, U7.A8
- removed net N$89: TP182.P$1, U7.A7
- removed net PIXCLK_I: U7.B4
- removed net PRU0: U2.24
- removed net PRU1: U2.26
- removed net PRU16_CLK: U2.23
- removed net PRU2: U2.27
- removed net PRU3: U2.29
- removed net PRU4: U2.30
- removed net PRU5: U2.31
- removed net PRU6: U2.33
- removed net SERDES_PWR_DOWN: J5.1
- removed net SPI_CLK: J2.17, J2.18
- removed net SPI_MISO: J2.15, J2.16
- removed net SPI_MOSI: J2.19, J2.20
- removed net VSYNC_I: U7.T6
- new net !EMMC_RST: R9.3, U3.K5, U7.R13
- new net 1.8V-A: C50.1, R21.2, U7.A7, U7.B7
- new net EMMC_CLK: R9.9, U3.M6, U7.P2
- new net EMMC_DAT3: R9.4, U3.B2, U7.T3
- new net EMMC_DAT4: R9.7, U3.B3, U7.T2
- new net EMMC_DAT5: R9.8, U3.B4, U7.T1
- new net N$37: TP36.P$1, U7.B8
- new net N$38: TP37.P$1, U7.B6
- new net N$39: TP38.P$1, U7.C6
- new net PRU0_0: TP30.1, U2.24, U7.A1
- new net PRU0_1: TP29.1, U2.26, U7.A2
- new net PRU0_14: TP33.1, U7.P6
- new net PRU0_15: TP34.1, U7.R6
- new net PRU0_16_CLK: TP20.1, U2.23, U7.B4
- new net PRU0_2: TP28.1, U2.27, U7.B2
- new net PRU0_3: TP27.1, U2.29, U7.B1
- new net PRU0_4: TP26.1, U2.30, U7.A3
- new net PRU0_5: TP24.1, U2.31, U7.B3
- new net PRU0_6: TP23.1, U2.33, U7.C3
- new net PRU0_7: R11.2, TP21.1, U7.C4
- new net SPI1_CLK: J2.17, J2.18, TP19.1, U7.C5
- new net SPI1_MISO: J2.15, J2.16, TP1.1, U7.C12
- new net SPI1_MOSI: J2.19, J2.20, TP18.1, U7.C13
- new net SYSBOOT0: R17.14, SB0.TP, U7.G3
- new net SYSBOOT1: R17.13, SB1.TP, U7.G2
- new net SYSBOOT10: R16.13, SB10.TP, U7.K2
- new net SYSBOOT11: R16.12, SB11.TP, U7.K1
- new net SYSBOOT12: R16.11, SB12.TP, U7.L3
- new net SYSBOOT13: R16.10, SB13.TP, U7.L2
- new net SYSBOOT14: R17.9, SB14.TP, U7.L1
- new net SYSBOOT15: R16.9, SB15.TP, U7.M3
- new net SYSBOOT2: J3.2, JP2.2, JP3.2, SB2.TP, U7.G1
- new net SYSBOOT3: R17.11, SB3.TP, U7.H3
- new net SYSBOOT4: R17.10, SB4.TP, U7.H2
- new net SYSBOOT5: R17.15, SB5.TP, U7.H1
- new net SYSBOOT6: R17.16, SB6.TP, U7.J3
- new net SYSBOOT7: R16.16, SB7.TP, U7.J2
- new net SYSBOOT8: R16.15, SB8.TP, U7.J1
- new net SYSBOOT9: R16.14, SB9.TP, U7.K3
- net !PWR_DWN: now also JP1.2; no longer J5.2
- net 3.3V: now also JP1.1, R17.5, R17.6, R17.7, R17.8, TP2.1; no longer J5.3, R24.10, R24.5, TP25.P$1
- net 3.3VA: no longer C41.1, U18.5
- net BOOT0: now also JP3.1
- net EEPROM_WP: now also TP71.1; no longer TP112.P$1, U18.6
- net GND: now also C50.2, C51.2, R11.1, R14.1, R16.1, R16.2, R16.3, R16.4, R16.5, R16.6, R16.7, R16.8, R17.1, R17.2, R17.3, R17.4, TP72.1, TP74.1, TP75.1, TP77.1, TP78.1, U7.A9, U7.B9; no longer C15.2, C41.2, R25.10, R25.5, R26.10, R26.5, U18.2
- net I2C0_SCL: now also TP39.1, U1.6; no longer TP155.P$1, U18.3
- net I2C0_SDA: now also TP70.1, U1.4; no longer TP151.P$1, U18.1
- net N$1: now also JP2.1, R14.2; no longer TP171.P$1, U7.A9, U7.B7, U7.B9
- net N$103: no longer TP62.P$1
- net N$19: now also R17.12; no longer R24.7
- net SENSOR_ENABLE: now also U7.F3
- net SPARE1: no longer TP58.P$1
- net SPARE2: no longer TP59.P$1
- net SPARE3: no longer TP60.P$1
- net SPARE4: no longer TP61.P$1
- net TEC_ENABLE: now also U7.F1
- net THERM+: now also C51.1, R21.1, U7.A8
- net UART0_RX: now also TP31.1; no longer TP146.P$1
- net UART0_TX: now also TP32.1; no longer TP142.P$1
- net USB_CLI_N: now also U1.3; no longer U1.1
- net USB_CLI_P: now also U1.1; no longer U1.3
- net VDD: now also C4.1, U1.5; no longer C15.1
- net VIN_USB: no longer C4.1, TP2.P$1, U1.5
Routing:
- net UART0_TX: track 0.00 -> 112.5 mm, vias 0 -> 2
- net UART0_RX: track 0.00 -> 109.5 mm, vias 0 -> 2
- net SPI1_MOSI: track 0.00 -> 92.2 mm
- net SPI1_MISO: track 0.00 -> 84.5 mm
- net 3.3V: track 3.13 -> 87.1 mm, vias 1 -> 32
- net SPI1_CLK: track 0.00 -> 75.2 mm, vias 0 -> 2
- net SENSOR_ENABLE: track 0.00 -> 71.9 mm, vias 0 -> 2
- net SYSBOOT2: track 0.00 -> 70.3 mm, vias 0 -> 3
- net TEC_ENABLE: track 0.00 -> 69.2 mm, vias 0 -> 2
- net THERM+: track 0.00 -> 65.6 mm, vias 0 -> 1
- net N$118: track 0.00 -> 63.9 mm, vias 0 -> 3
- net N$114: track 0.00 -> 63.1 mm, vias 0 -> 2
- net N$116: track 0.00 -> 59.4 mm, vias 0 -> 2
- net PRU0_15: track 0.00 -> 49.6 mm
- net PRU0_14: track 0.00 -> 47.7 mm
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- added copper zone on layer 1, net OPD_PWR
- added copper zone on layer 15, net USB_CLI_VBUS
- removed copper zone on layer 1, net N$26
- removed copper zone on layer 15, net OPD_PWR
- removed copper zone on layer 15, net VDD
Other:
- board text added: "3.3V"
- board text added: "CLK"
- board text added: "CONNECTOR THIS SIDE"
- board text added: "EEPROM_WP"
- board text added: "GND"
- board text added: "I2C0_SCL"
- board text added: "I2C0_SDA"
- board text added: "ON/OFF"
- board text added: "PRU0"
- board text added: "PRU1"
- board text added: "PRU14"
- board text added: "PRU15"
- board text added: "PRU2"
- board text added: "PRU3"
- board text added: "PRU4"
- board text added: "PRU5"
- board text added: "PRU6"
- board text added: "PRU7"
- board text added: "SPI_CLK"
- board text added: "SPI_MISO"
- board text added: "SPI_MOSI"
- board text added: "UART0_RX"
- board text added: "UART0_TX"
- board text added: "uSD/USB"
- board text removed: "0"
- board text removed: "1"
- board text removed: "2"
- board text removed: "3"
- board text removed: "4"
- board text removed: "NOTE: SYSBOOT[2] UNSET"
- board text removed: "ON/ OFF"
- board text removed: "uSD"

Commit message: oh god almost done
Parts:
- added U$4: (no value), oresat-misc:ORESAT_ORIENTATION_COPPER
- J1: value ORESAT-DEBUG-CONNECTOR-CARD -> ORESAT-DEBUG-CONNECTOR-ALL
- JP1: value JUMPER-SMT_2_NC_TRACE_NO-SILK -> JUMPER-SMT_2_NC_TRACE_SILK; device SparkFun-Jumpers:SMT-JUMPER_2_NC_TRACE_NO-SILK -> SparkFun-Jumpers:SMT-JUMPER_2_NC_TRACE_SILK
- moved U$3 51.3 mm to (88.0, 29.9)
- moved JP1 1.52 mm to (35.8, 74.0), flipped to the top
Connections:
- removed net USB_HO_N: J1.8
- removed net USB_HO_PX: J1.7
- removed net USB_HO_VBUS: J1.17
Routing:
- net !PWR_DWN: track 7.14 -> 8.73 mm, vias 1 -> 2
- net GND: vias 175 -> 213
Other:
- board text added: "2021/08/01"
- board text added: "OreSat CFC Card v1.0"
- board text removed: "2020/12/08"
- board text removed: "DEFAULT : 0b11x00"
- board text removed: "NOTE: SYSBOOT[2] is not set by default. It must be set with J3 or JP107, BUT NOT BOTH. See AM335x TRM Table 26-7 for details."
- board text removed: "OreSat Star Tracker v1.2"
- board text removed: "SYSBOOT [4:0]"
- board text removed: "eMMC : 0b11100"
- board text removed: "uSD : 0b11000"

Commit message: couple more changes
Parts:
- moved U$1 65.8 mm to (7.10, 59.7), turned to 90 degrees
Changed lines of the file:
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@@
 <attribute name="VALUE" x="62.7" y="75" size="0.8" layer="27" font="vector" ratio="15" rot="R270"/>
 </element>
-<element name="U$1" library="oresat-flight-marker" package="FLIGHTMARKER_NEW_BOARDS" value="FLIGHMARKERNEW" x="6.2" y="-6.1" smashed="yes"/>
+<element name="U$1" library="oresat-flight-marker" package="FLIGHTMARKER_NEW_BOARDS" value="FLIGHMARKERNEW" x="7.1" y="59.7" smashed="yes" rot="R90"/>
 <element name="J2" library="J-Samtec-TFM-110-X1-XXX-D-RA" package="J-SAMTEC-TFM-110-X1-XXX-D-RA" value="J-SAMTEC-TFM-110-X1-XXX-D-RA" x="21.9" y="87.9" locked="yes" smashed="yes">
 <attribute name="DIS" value="Digikey" x="21.9" y="87.9" locked="yes" size="1.778" layer="27" display="off"/>

Commit message: boards finished
Parts:
- R50: value 0 -> 10k
- R51: value NP -> 4.7k
- moved JP1 1.25 mm to (37.0, 74.0)
Routing:
- net PRU0_0: track 28.7 -> 32.0 mm
- net PRU0_16_CLK: track 44.3 -> 47.1 mm
- net !PWR_DWN: track 8.73 -> 10.7 mm
- net TEC_ENABLE: track 69.2 -> 69.7 mm
- net GND: vias 213 -> 260
Other:
- board text added: "OreSat CFC Processor Card v1.0"
- board text removed: "OreSat CFC Card v1.0"
