File: cfc-card/cfc-card.brd (EAGLE design)
At the start: 99.8 x 94.6 mm, 274 parts, among them J1 ORESAT-DEBUG-CONNECTOR-ALL, J100 DM3BT-DSF-PEJS, J2 J-SAMTEC-TFM-110-X1-XXX-D-RA, J4 TFM-120-01-L-D-RA, Q1 MMBT2907, Q2 PMV45EN, Q3 DMP2240UDM, Q4 PMV45EN, Q5 MOSFET-PCH-SOT23-6, Q6 MOSFET-PCH-SOT23-6, U1 RCLAMP0504FB, U10 TLVH431, U11 TCAN330, U12 MIC842LYC5, U13 MIC842LYC5, U14 MAX4211FETE, U15 TPS62112, U16 MAX7310ATE, U17 25AAXX, U2 DS90CR218AMTD/NOPBMTD48_TEX-L, U3 THGBMJG7C2LBAU8, U4 SN74LVC1G07DCK, U7 OSD3358-512M-BSM, Y1 24MHz, Y2 ABS07-32.768KHZ-T

Commit message: fixed resistor array value
Parts:
- R16, R17: value EXB-2HV103JV -> 100k
Changed lines of the file:
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@@
 <attribute name="DPN" value="THGBMJG7C2LBAU8-ND" x="19.9" y="20" size="1.778" layer="27" rot="R270" display="off"/>
 <attribute name="MPN" value="THGBMJG7C2LBAU8" x="19.9" y="20" size="1.778" layer="27" rot="R270" display="off"/>
+<attribute name="NAME" x="27.0125" y="15.575" size="0.635" layer="25" font="vector" ratio="20" rot="R270"/>
 <attribute name="NAME" x="19.9" y="20" size="1.5" layer="33" ratio="15" rot="R270" align="center"/>
-<attribute name="NAME" x="27.0125" y="15.575" size="0.635" layer="25" font="vector" ratio="20" rot="R270"/>
 <attribute name="VALUE" x="12.3" y="25.6" size="0.8" layer="27" font="vector" ratio="15" rot="R270"/>
 </element>
@@
 <attribute name="VALUE" x="25.75" y="37.6" size="0.8" layer="27" font="vector" ratio="15" rot="R90"/>
 </element>
-<element name="R16" library="R-Panasonic-EXB-2HV103JV" package="RES_EXB2HV" value="EXB-2HV103JV" x="28.5" y="37.25" smashed="yes">
+<element name="R16" library="R-Panasonic-EXB-2HV103JV" package="RES_EXB2HV" value="100k" x="28.5" y="37.25" smashed="yes">
 <attribute name="BUILT_BY" value="EMA_UL_Team" x="24" y="46.25" size="1.778" layer="27" display="off"/>
 <attribute name="DPN" value="Y1103CT-ND" x="24" y="46.25" size="1.778" layer="27" display="off"/>
@@
 <attribute name="VENDOR" value="Panasonic" x="24" y="46.25" size="1.778" layer="27" display="off"/>
 </element>
-<element name="R17" library="R-Panasonic-EXB-2HV103JV" package="RES_EXB2HV" value="EXB-2HV103JV" x="28.5" y="43.5" smashed="yes">
+<element name="R17" library="R-Panasonic-EXB-2HV103JV" package="RES_EXB2HV" value="100k" x="28.5" y="43.5" smashed="yes">
 <attribute name="BUILT_BY" value="EMA_UL_Team" x="24" y="52.5" size="1.778" layer="27" display="off"/>
 <attribute name="DPN" value="Y1103CT-ND" x="24" y="52.5" size="1.778" layer="27" display="off"/>
