File: cfc-card/cfc-card.sch (EAGLE design)
At the start: 271 parts, among them J1 ORESAT-DEBUG-CONNECTOR-CARD, J100 DM3BT-DSF-PEJS, J2 J-SAMTEC-TFM-110-X1-XXX-D-RA, J4 TFM-120-01-L-D-RA, Q1 MMBT2907, Q2 PMV45EN, Q3 DMP2240UDM, Q4 PMV45EN, Q5 MOSFET-PCH-SOT23-6, Q6 MOSFET-PCH-SOT23-6, U1 RCLAMP0504FB, U10 TLVH431, U11 TCAN330, U12 MIC842LYC5, U13 MIC842LYC5, U14 MAX4211FETE, U15 TPS62112, U16 MAX7310ATE, U17 25AAXX, U18 RCLAMP0504FB, U3 THGBMJG7C2LBAU8, U4 SN74LVC1G07DCK, U7 OSD3358-512M-BSM, Y1 24MHz, Y2 ABS07-32.768KHZ-T

Commit message: rebase: backup work
Parts:
- removed JP100, JP101, JP104: JUMPER-SMT_2_NC_TRACE_SILK, SparkFun-Jumpers:JUMPER-SMT_2_NC_TRACE_SILK
- removed TP1, TP100, TP101, TP103, TP104, TP105, TP106, TP107, TP108, TP111, TP114, TP115, TP117, TP118, TP120, TP122, TP123, TP124, TP125, TP126, TP127, TP128, TP131, TP134, TP135, TP137, TP143, TP145, TP147, TP148, TP149, TP150, TP152, TP153, TP158, TP159, TP162, TP169, TP170, TP172, TP174, TP175, TP176, TP179, TP180, TP181, TP30, TP38: TEST-POINT3X4, SparkFun-Connectors:TEST-POINT3X4
- added C1, C16, C17, C20, C28, C7: 1n, oresat-rcl:C-EU0402-C-NOSILK
- added C21, C23, C24, C25, C26, C27: 10n, oresat-rcl:C-EU0402-C-NOSILK
- added C42, C43, C45, C46, C47, C48: 100n, oresat-rcl:C-EU0402-C-NOSILK
- added C49: 10u, oresat-rcl:C-EU0603-C-NOSILK
- added R6, R7: 100, oresat-rcl:R-US_0402-C-NOSILK
- added TP13, TP15, TP16, TP17: TEST-POINT3X4, SparkFun-Connectors:TEST-POINT3X4
- added U2: DS90CR218AMTD/NOPBMTD48_TEX-L, U-TI-DS90CR218-LVDSReceiver:DS90CR218AMTD/NOPBMTD48_TEX-L
- C40: value 0.1uF -> DNP
- J5: value (none) -> 455-1750-1-ND; device SparkFun-Connectors:CONN_02 -> SparkFun-Connectors:CONN_03
- R10, R8, R9: MPN EXB-A10P103J -> (none)
- R24, R25, R26: MPN EXB-A10P104J -> (none)
- R29, R30: value 4.7k -> NP; device oresat-rcl:R-US_0603-A -> oresat-rcl:R-US_0402-C-NOSILK; DIS (none) -> Dgi-Key; DPN (none) -> 311-100MCT-ND; MFR (none) -> Yageo; MPN (none) -> RC0201FR-07100RL
Connections:
- net AUX-5 renamed TEC_ENABLE
- net AUX-6 renamed THERM+
- net AUX-7 renamed SENSOR_ENABLE
- net AUX-8 renamed SPI_MISO
- net AUX-9 renamed SPI_CLK
- net AUX_!SHUTDOWN renamed SPI_MOSI
- removed net AUX-1: J2.1, J2.2
- removed net AUX-2: J2.3, J2.4
- removed net AUX-3: J2.5, J2.6
- removed net AUX-4: J2.7, J2.8
- removed net BUS_OE: U7D.MII1_CRS
- removed net CAM_OE: U7D.MII1_COL
- removed net CLK_EN: U7D.MII1_RX_CLK
- removed net FLASH: U7D.MII1_TXD3
- removed net INPUT_EN: U7D.MII1_RXD0
- removed net N$36: TP123.1, U7C.GPMC_AD9
- removed net N$37: TP115.1, U7C.GPMC_AD10
- removed net N$38: TP105.1, U7C.GPMC_AD11
- removed net N$39: TP124.1, U7C.GPMC_AD12
- removed net N$40: TP120.1, U7C.GPMC_AD13
- removed net N$407: JP104.2, Q1.C, R31.1, U10.ANODE
- removed net N$41: TP125.1, U7C.GPMC_BEN1
- removed net N$42: TP114.1, U7C.GPMC_WAIT0
- removed net N$43: TP111.1, U7C.GPMC_WPN
- removed net N$46: TP162.1, U7D.LCD_PCLK
- removed net N$47: TP153.1, U7D.LCD_VSYNC
- removed net N$48: TP152.1, U7D.LCD_HSYNC
- removed net N$49: TP159.1, U7D.LCD_AC_BIAS_EN
- removed net N$50: TP143.1, U7D.RMII1_REF_CLK
- removed net N$51: TP174.1, U7D.MDC
- removed net N$52: TP158.1, U7D.MDIO
- removed net N$53: TP147.1, U7D.MII1_TX_CLK
- removed net N$54: TP137.1, U7D.MII1_TXD0
- removed net N$55: TP149.1, U7D.MII1_TXD1
- removed net N$56: TP135.1, U7D.MII1_TXD2
- removed net N$57: TP172.1, U7F.NC@1
- removed net N$58: TP150.1, U7F.NC@2
- removed net N$59: TP145.1, U7F.NC@3
- removed net N$66: TP179.1, U7B.AIN6
- removed net N$67: TP169.1, U7B.AIN5
- removed net N$68: TP176.1, U7B.AIN4
- removed net N$69: TP175.1, U7B.AIN3
- removed net N$70: TP181.1, U7B.AIN2
- removed net N$71: TP38.1, U7B.AIN1
- removed net N$75: TP106.1, U7C.GPMC_CLK
- removed net N$76: TP100.1, U7C.GPMC_A0
- removed net N$77: TP118.1, U7C.GPMC_A1
- removed net N$78: TP126.1, U7C.GPMC_A2
- removed net N$79: TP101.1, U7C.GPMC_A3
- removed net N$82: TP108.1, U7C.GPMC_A9
- removed net N$83: TP117.1, U7C.GPMC_A10
- removed net N$84: TP103.1, U7C.GPMC_A11
- removed net N$85: TP122.1, U7C.GPMC_CSN0
- removed net N$86: TP107.1, U7C.GPMC_CSN3
- removed net N$93: TP134.1, U7C.GPMC_ADVN_ALE
- removed net N$94: TP131.1, U7C.GPMC_BEN0_CLE
- removed net N$95: TP127.1, U7C.GPMC_WEN
- removed net N$96: TP128.1, U7C.GPMC_OEN_REN
- removed net N$97: TP148.1, U7D.MII1_TX_EN
- removed net RESET: U7D.MII1_RXD1
- removed net SADDR: U7D.MII1_RXD2
- removed net SCL_2: R30.2, U7C.UART1_RTSN
- removed net SDA_2: R29.2, U7C.UART1_CTSN
- removed net STANDBY: U7D.MII1_RXD3
- removed net TRIGGER: U7D.MII1_RX_ER
- removed net VREG_EN: U7D.MII1_RX_DV
- new net !PWR_DWN: J5.2, U2.!PWR_DWN
- new net N$112: TP13.1, U7C.UART1_RTSN
- new net N$119: TP16.1, U7B.USB1_DM
- new net N$120: TP17.1, U7B.USB1_VBUS
- new net OUT1N: J2.5, J2.6, R6.2, U2.RXIN0-
- new net OUT1P: J2.7, J2.8, R6.1, U2.RXIN0+
- new net PRU0: U2.RXOUT0
- new net PRU1: U2.RXOUT1
- new net PRU16_CLK: U2.RXCLKOUT
- new net PRU2: U2.RXOUT2
- new net PRU3: U2.RXOUT3
- new net PRU4: U2.RXOUT4
- new net PRU5: U2.RXOUT5
- new net PRU6: U2.RXOUT6
- new net SERDES_PWR_DOWN: J5.1
- new net TXCLKN: J2.1, J2.2, R7.1, U2.RXCLKIN-
- new net TXCLKP: J2.3, J2.4, R7.2, U2.RXCLKIN+
- net 3.3V: now also C1.1, C16.1, C17.1, C20.1, C21.1, C23.1, C24.1, C25.1, C26.1, C27.1, C28.1, C42.1, C43.1, C45.1, C46.1, C47.1, C48.1, C49.1, C7.1, J5.3, U2.LVDS_VCC, U2.PLL_VCC, U2.VCC, U2.VCC_2, U2.VCC_3, U2.VCC_4; no longer R29.1, R30.1
- net 3.3VA: now also Q1.E, R23.2, R28.2; no longer JP101.1
- net GND: now also C1.2, C16.2, C17.2, C20.2, C21.2, C23.2, C24.2, C25.2, C26.2, C27.2, C28.2, C42.2, C43.2, C45.2, C46.2, C47.2, C48.2, C49.2, C7.2, U2.GND, U7B.USB1_ID; no longer JP100.2
- net N$102: now also TP15.1, U7B.USB1_DP; no longer JP100.1, U7B.USB1_ID
- net N$118: now also Q1.C, R31.1, U10.ANODE; no longer JP104.1
- net N$20: now also TP4.1, U7C.UART1_CTSN; no longer JP101.2, Q1.E, R23.2, R28.2
- net N$3: now also R29.2, U2.RXIN2-; no longer TP170.1, U7B.AIN7
- net N$33: now also R29.1, U2.RXIN2+; no longer TP30.1, U7C.XDMA_EVENT_INTR0
- net N$34: now also R30.2, U2.RXIN1-; no longer TP180.1, U7C.ECAP0_IN_PWM0_OUT
- net N$35: now also R30.1, U2.RXIN1+; no longer TP104.1, U7C.GPMC_AD8
- net N$401: no longer TP4.1
- net USB_HO_N: no longer U1.I4, U7B.USB1_DM
- net USB_HO_PX: no longer U1.I3, U7B.USB1_DP
- net USB_HO_VBUS: no longer J5.1, TP1.1, U7B.USB1_VBUS
- net VDD: no longer J5.2
Other:
- note added: "!PWR_DWN is pulled low by default, but can be pulled high via jumper or via GPIO NOTE: Pull down on other sheet"
- note added: "Aux Connector"
- note added: "DESERIALIZER"
- note added: "Only need to connect 7 bits"
- note added: "TODO - Breakout SPI - Breakout UART0 - Breakout PRU bus? - PRU debug signals - Breakout I2C0 - Breakout EEPROM_WP - Pulldiown on PRU0_7"
- note added: "TODO Delete this cap if VDD unused"
- note added: "To other sheet"
- note added: "USB ID grounded to make host circuit"
- note removed: "I2C2 SCL == UART1_RTSN == A10 I2C2 SDA == UART1_CTSN == B10"
- note removed: "NOTE: All these signals are outputs with the exception of FLASH. Likewise, I put the outputs on GPIO2,3 and inputs on GPIO0. I am not sure if this is better, but it seemed logical"
- note removed: "TODO - Breakout SPI - Breakout UART0 - Breakout PRU bus? - Breakout I2C0 - Breakout EEPROM_WP"
- note removed: "VOUT USB JUMPER"
- moved on the sheet: C40, R29, R30

Commit message: mostly finished sensor card
Changed lines of the file:
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@@
 <?xml version="1.0" encoding="utf-8"?>
 <!DOCTYPE eagle SYSTEM "eagle.dtd">
-<eagle version="9.5.2">
+<eagle version="9.6.2">
 <drawing>
 <settings>
@@
 <instance part="U$1" gate="G$1" x="246.38" y="2.54" smashed="yes"/>
 <instance part="J2" gate="G$1" x="111.76" y="68.58" smashed="yes" rot="MR0">
-<attribute name="NAME" x="118.11" y="94.615" size="1.778" layer="95" rot="MR0"/>
 <attribute name="VALUE" x="105.41" y="36.83" size="1.778" layer="96"/>
 <attribute name="MFR" x="111.76" y="68.58" size="1.778" layer="96" rot="MR0" display="off"/>
@@
 <net name="TXCLKN" class="1">
 <segment>
-<wire x1="114.3" y1="91.44" x2="121.92" y2="91.44" width="0.1524" layer="91"/>
 <wire x1="121.92" y1="91.44" x2="139.7" y2="91.44" width="0.1524" layer="91"/>
-<wire x1="114.3" y1="88.9" x2="121.92" y2="88.9" width="0.1524" layer="91"/>
 <wire x1="121.92" y1="88.9" x2="121.92" y2="91.44" width="0.1524" layer="91"/>
-<junction x="121.92" y="91.44"/>
 <label x="139.7" y="91.44" size="1.27" layer="95" xref="yes"/>
 <pinref part="J2" gate="G$1" pin="1"/>
+<wire x1="114.3" y1="91.44" x2="121.92" y2="91.44" width="0.1524" layer="91"/>
+<junction x="121.92" y="91.44"/>
 <pinref part="J2" gate="G$1" pin="2"/>
+<wire x1="121.92" y1="88.9" x2="114.3" y2="88.9" width="0.1524" layer="91"/>
 </segment>
 </net>
 <net name="TXCLKP" class="1">
 <segment>
-<wire x1="114.3" y1="86.36" x2="121.92" y2="86.36" width="0.1524" layer="91"/>
 <wire x1="121.92" y1="86.36" x2="139.7" y2="86.36" width="0.1524" layer="91"/>
-<wire x1="114.3" y1="83.82" x2="121.92" y2="83.82" width="0.1524" layer="91"/>
 <wire x1="121.92" y1="83.82" x2="121.92" y2="86.36" width="0.1524" layer="91"/>
-<junction x="121.92" y="86.36"/>
 <label x="139.7" y="86.36" size="1.27" layer="95" xref="yes"/>
 <pinref part="J2" gate="G$1" pin="3"/>
+<wire x1="114.3" y1="86.36" x2="121.92" y2="86.36" width="0.1524" layer="91"/>
+<junction x="121.92" y="86.36"/>
 <pinref part="J2" gate="G$1" pin="4"/>
+<wire x1="121.92" y1="83.82" x2="114.3" y2="83.82" width="0.1524" layer="91"/>
 </segment>
 </net>
 <net name="OUT1N" class="1">
 <segment>
-<wire x1="114.3" y1="81.28" x2="121.92" y2="81.28" width="0.1524" layer="91"/>
 <wire x1="121.92" y1="81.28" x2="139.7" y2="81.28" width="0.1524" layer="91"/>
-<wire x1="114.3" y1="78.74" x2="121.92" y2="78.74" width="0.1524" layer="91"/>
 <wire x1="121.92" y1="78.74" x2="121.92" y2="81.28" width="0.1524" layer="91"/>
-<junction x="121.92" y="81.28"/>
 <label x="139.7" y="81.28" size="1.27" layer="95" xref="yes"/>
 <pinref part="J2" gate="G$1" pin="5"/>
+<wire x1="114.3" y1="81.28" x2="121.92" y2="81.28" width="0.1524" layer="91"/>
+<junction x="121.92" y="81.28"/>
 <pinref part="J2" gate="G$1" pin="6"/>
+<wire x1="121.92" y1="78.74" x2="114.3" y2="78.74" width="0.1524" layer="91"/>
 </segment>
 </net>
 <net name="OUT1P" class="1">
 <segment>
-<wire x1="114.3" y1="76.2" x2="121.92" y2="76.2" width="0.1524" layer="91"/>
 <wire x1="121.92" y1="76.2" x2="139.7" y2="76.2" width="0.1524" layer="91"/>
-<wire x1="114.3" y1="73.66" x2="121.92" y2="73.66" width="0.1524" layer="91"/>
 <wire x1="121.92" y1="73.66" x2="121.92" y2="76.2" width="0.1524" layer="91"/>
-<junction x="121.92" y="76.2"/>
 <label x="139.7" y="76.2" size="1.27" layer="95" xref="yes"/>
 <pinref part="J2" gate="G$1" pin="7"/>
+<wire x1="114.3" y1="76.2" x2="121.92" y2="76.2" width="0.1524" layer="91"/>
+<junction x="121.92" y="76.2"/>
 <pinref part="J2" gate="G$1" pin="8"/>
-</segment>
-</net>
+<wire x1="121.92" y1="73.66" x2="114.3" y2="73.66" width="0.1524" layer="91"/>
+</segment>
+</net>

Commit message: mostly finished octavo card
Parts:
- removed C15: 22uF, oresat-rcl:C-EUC1210
- removed C41: 0.1uF, oresat-rcl:C-EU0603-A
- removed J5: 455-1750-1-ND, SparkFun-Connectors:CONN_03
- removed JP105, JP106, JP108, JP109: JUMPER-SMT_3_1-NC_TRACE_SILK, SparkFun-Jumpers:JUMPER-SMT_3_1-NC_TRACE_SILK
- removed R24, R25, R26: 100K, R-Panasonic-EXB_A10PXXXJ:EXB-A10P391JC_ARRAY_EXBA-M
- removed TP112, TP142, TP146, TP151, TP155, TP171, TP177, TP178, TP182, TP25, TP58, TP59, TP60, TP61, TP62: TEST-POINT3X4, SparkFun-Connectors:TEST-POINT3X4
- removed U18: RCLAMP0504FB, U-Semtec-RCLAMP0504FB:RCLAMP0504FB
- added C50: 0.1uF, oresat-rcl:C-EU0603-A
- added C51: 0.1u, oresat-rcl:C-EU0603-A
- added JP1: JUMPER-SMT_2_NC_TRACE_NO-SILK, SparkFun-Jumpers:JUMPER-SMT_2_NC_TRACE_NO-SILK
- added JP3: JUMPER-SMT_2_NO_SILK, SparkFun-Jumpers:JUMPER-SMT_2_NO_SILK
- added R11, R14: DNP, oresat-rcl:R-US_0603-A
- added R16, R17: EXB-2HV103JV, R-Panasonic-EXB-2HV103JV:EXB-2HV103JV
- added R21: 10k, oresat-rcl:R-US_0603-A
- added SB0, SB1, SB10, SB11, SB12, SB13, SB14, SB15, SB2, SB3, SB4, SB5, SB6, SB7, SB8, SB9: TEST-POINT-SMALL, oresat-misc:TEST-POINT-SMALL
- added TP1, TP18, TP19, TP20, TP21, TP23, TP24, TP26, TP27, TP28, TP29, TP30, TP31, TP32, TP33, TP34, TP70, TP71, TP72, TP74, TP75, TP77, TP78: TEST-POINT, Tova:TEST-POINT
- added TP36, TP37, TP38: TEST-POINT3X4, SparkFun-Connectors:TEST-POINT3X4
- TP2, TP39: value TEST-POINT3X4 -> TEST-POINT; device SparkFun-Connectors:TEST-POINT3X4 -> Tova:TEST-POINT
Connections:
- net N$641 renamed EMMC_DAT0
- net N$642 renamed EMMC_DAT1
- net N$643 renamed EMMC_DAT2
- net N$647 renamed EMMC_DAT6
- net N$648 renamed EMMC_DAT7
- net N$649 renamed EMMC_CMD
- net OUT1N renamed OUT1_N
- net OUT1P renamed OUT1_P
- net TXCLKN renamed TXCLK_N
- net TXCLKP renamed TXCLK_P
- removed net D10_I: U7C.MCASP0_AXR1
- removed net D11_I: U7C.MCASP0_AHCLKX
- removed net D4_I: U7C.MCASP0_ACLKX
- removed net D5_I: U7C.MCASP0_FSX
- removed net D6_I: U7C.MCASP0_AXR0
- removed net D7_I: U7C.MCASP0_AHCLKR
- removed net D8_I: U7C.MCASP0_ACLKR
- removed net D9_I: U7C.MCASP0_FSR
- removed net HSYNC_I: U7C.GPMC_AD15
- removed net N$105: JP105.1, R24.99
- removed net N$106: JP106.1, R24.22
- removed net N$107: JP108.3, R24.33
- removed net N$108: JP109.3, R24.66
- removed net N$21: JP2.1, R25.88
- removed net N$44: TP177.1, U7C.UART0_CTSN
- removed net N$45: TP178.1, U7C.UART0_RTSN
- removed net N$535: JP105.2, U7D.LCD_DATA0
- removed net N$578: JP106.2, U7D.LCD_DATA1
- removed net N$582: J3.2, JP2.2, U7D.LCD_DATA2
- removed net N$583: JP108.2, U7D.LCD_DATA3
- removed net N$584: JP109.2, U7D.LCD_DATA4
- removed net N$585: R25.44, U7D.LCD_DATA5
- removed net N$586: R25.77, U7D.LCD_DATA6
- removed net N$587: R26.44, U7D.LCD_DATA8
- removed net N$588: R26.77, U7D.LCD_DATA9
- removed net N$591: R26.33, U7D.LCD_DATA10
- removed net N$592: R26.88, U7D.LCD_DATA11
- removed net N$594: R26.22, U7D.LCD_DATA12
- removed net N$595: R26.99, U7D.LCD_DATA13
- removed net N$601: R24.44, U7D.LCD_DATA14
- removed net N$602: R26.11, U7D.LCD_DATA15
- removed net N$629: R26.66, U7D.LCD_DATA7
- removed net N$630: JP109.1, R25.66
- removed net N$632: JP108.1, R25.99
- removed net N$633: JP106.3, R25.22
- removed net N$634: JP105.3, R25.33
- removed net N$644: R9.77, U3.D3, U7C.GPMC_AD3
- removed net N$645: R9.44, U3.D4, U7C.GPMC_AD4
- removed net N$646: R9.33, U3.D5, U7C.GPMC_AD5
- removed net N$651: R9.88, U3.SCK, U7C.GPMC_CSN1
- removed net N$652: R10.33, U3.!RST!, U7C.GPMC_A4
- removed net N$72: TP39.1, U7B.AIN0
- removed net N$89: TP182.1, U7B.SYS_ADC_1P8V
- removed net PIXCLK_I: U7C.XDMA_EVENT_INTR1
- removed net PRU0: U2.RXOUT0
- removed net PRU1: U2.RXOUT1
- removed net PRU16_CLK: U2.RXCLKOUT
- removed net PRU2: U2.RXOUT2
- removed net PRU3: U2.RXOUT3
- removed net PRU4: U2.RXOUT4
- removed net PRU5: U2.RXOUT5
- removed net PRU6: U2.RXOUT6
- removed net SERDES_PWR_DOWN: J5.1
- removed net SPI_CLK: J2.17, J2.18
- removed net SPI_MISO: J2.15, J2.16
- removed net SPI_MOSI: J2.19, J2.20
- removed net VSYNC_I: U7C.GPMC_AD14
- new net !EMMC_RST: R9.33, U3.!RST!, U7C.GPMC_A4
- new net 1.8V-A: C50.1, R21.2, U7B.SYS_ADC_1P8V, U7B.VREFP
- new net EMMC_CLK: R9.99, U3.SCK, U7C.GPMC_CSN1
- new net EMMC_DAT3: R9.44, U3.D3, U7C.GPMC_AD3
- new net EMMC_DAT4: R9.77, U3.D4, U7C.GPMC_AD4
- new net EMMC_DAT5: R9.88, U3.D5, U7C.GPMC_AD5
- new net N$37: TP36.1, U7B.AIN1
- new net N$38: TP37.1, U7B.AIN2
- new net N$39: TP38.1, U7B.AIN3
- new net PRU0_0: TP30.1, U2.RXOUT0, U7C.MCASP0_ACLKX
- new net PRU0_1: TP29.1, U2.RXOUT1, U7C.MCASP0_FSX
- new net PRU0_14: TP33.1, U7C.GPMC_AD12
- new net PRU0_15: TP34.1, U7C.GPMC_AD13
- new net PRU0_16_CLK: TP20.1, U2.RXCLKOUT, U7C.XDMA_EVENT_INTR1
- new net PRU0_2: TP28.1, U2.RXOUT2, U7C.MCASP0_AXR0
- new net PRU0_3: TP27.1, U2.RXOUT3, U7C.MCASP0_AHCLKR
- new net PRU0_4: TP26.1, U2.RXOUT4, U7C.MCASP0_ACLKR
- new net PRU0_5: TP24.1, U2.RXOUT5, U7C.MCASP0_FSR
- new net PRU0_6: TP23.1, U2.RXOUT6, U7C.MCASP0_AXR1
- new net PRU0_7: R11.2, TP21.1, U7C.MCASP0_AHCLKX
- new net SPI1_CLK: J2.17, J2.18, TP19.1, U7C.ECAP0_IN_PWM0_OUT
- new net SPI1_MISO: J2.15, J2.16, TP1.1, U7C.UART0_CTSN
- new net SPI1_MOSI: J2.19, J2.20, TP18.1, U7C.UART0_RTSN
- new net SYSBOOT0: R17.14, SB0.TP, U7D.LCD_DATA0
- new net SYSBOOT1: R17.13, SB1.TP, U7D.LCD_DATA1
- new net SYSBOOT10: R16.13, SB10.TP, U7D.LCD_DATA10
- new net SYSBOOT11: R16.12, SB11.TP, U7D.LCD_DATA11
- new net SYSBOOT12: R16.11, SB12.TP, U7D.LCD_DATA12
- new net SYSBOOT13: R16.10, SB13.TP, U7D.LCD_DATA13
- new net SYSBOOT14: R17.9, SB14.TP, U7D.LCD_DATA14
- new net SYSBOOT15: R16.9, SB15.TP, U7D.LCD_DATA15
- new net SYSBOOT2: J3.2, JP2.2, JP3.2, SB2.TP, U7D.LCD_DATA2
- new net SYSBOOT3: R17.11, SB3.TP, U7D.LCD_DATA3
- new net SYSBOOT4: R17.10, SB4.TP, U7D.LCD_DATA4
- new net SYSBOOT5: R17.15, SB5.TP, U7D.LCD_DATA5
- new net SYSBOOT6: R17.16, SB6.TP, U7D.LCD_DATA6
- new net SYSBOOT7: R16.16, SB7.TP, U7D.LCD_DATA7
- new net SYSBOOT8: R16.15, SB8.TP, U7D.LCD_DATA8
- new net SYSBOOT9: R16.14, SB9.TP, U7D.LCD_DATA9
- net !PWR_DWN: now also JP1.2; no longer J5.2
- net 3.3V: now also JP1.1, R17.5, R17.6, R17.7, R17.8, TP2.1; no longer J5.3, R24.55, TP25.1
- net 3.3VA: no longer C41.1, U18.VCC
- net BOOT0: now also JP3.1
- net EEPROM_WP: now also TP71.1; no longer TP112.1, U18.I4
- net GND: now also C50.2, C51.2, R11.1, R14.1, R16.1, R16.2, R16.3, R16.4, R16.5, R16.6, R16.7, R16.8, R17.1, R17.2, R17.3, R17.4, TP72.1, TP74.1, TP75.1, TP77.1, TP78.1, U7B.AGND_ADC, U7B.VREFN; no longer C15.2, C41.2, R25.55, R26.55, U18.GND
- net I2C0_SCL: now also TP39.1, U1.I4; no longer TP155.1, U18.I2
- net I2C0_SDA: now also TP70.1, U1.I3; no longer TP151.1, U18.I1
- net N$1: now also JP2.1, R14.2; no longer TP171.1, U7B.AGND_ADC, U7B.VREFN, U7B.VREFP
- net N$103: no longer TP62.1
- net N$19: now also R17.12; no longer R24.77
- net SENSOR_ENABLE: now also U7D.LCD_VSYNC
- net SPARE1: no longer TP58.1
- net SPARE2: no longer TP59.1
- net SPARE3: no longer TP60.1
- net SPARE4: no longer TP61.1
- net TEC_ENABLE: now also U7D.LCD_PCLK
- net THERM+: now also C51.1, R21.1, U7B.AIN0
- net UART0_RX: now also TP31.1; no longer TP146.1
- net UART0_TX: now also TP32.1; no longer TP142.1
- net USB_CLI_N: now also U1.I2; no longer U1.I1
- net USB_CLI_P: now also U1.I1; no longer U1.I2
- net VDD: now also C4.1, U1.VCC; no longer C15.1
- net VIN_USB: no longer C4.1, TP2.1, U1.VCC
Other:
- note added: "10k resistor is upper resistor of divider and the PIRT1280 10k thermistor is the lower resistor of the divider"
- note added: "ADC VREFP tied to 1.8V and VREFN tied to GND. Analog inputs must be between 0V-1.8V"
- note added: "ESD Protection"
- note added: "ESD Protection for I2C0 and USB lines"
- note added: "Only need to connect 7 bits + clock"
- note added: "PIRT1280 Enable and TEC enable GPIO. We are using these pins because they are free and are the ones we used on pocketbeagle board"
- note added: "PIRT1280 Thermistor"
- note added: "PWR from OPD 5V"
- note added: "SYSBOOT2 pulled high by default to boot eMMC. Manual jumper here to override"
- note added: "Sensor only uses 7 bits. Optional pulldown so this bit is always read as 0"
- note added: "TODO - DONE Breakout SPI1 - DONE Breakout UART0 - DONE Breakout PRU bus? - PRU debug signals labels - DONE Breakout I2C0 - DONE Breakout EEPROM_WP - DONE Pulldown on PRU0_7 - DONE OPD boot pin"
- note added: "To Octavo Boot Select -->"
- note added: "To PIRT1280 Thermistor -->"
- note added: "USB Device Circuit"
- note removed: "!PWR_DWN is pulled low by default, but can be pulled high via jumper or via GPIO NOTE: Pull down on other sheet"
- note removed: "ESD protection clamping diodes for I2C0 lines. This is required because these lines are routed externally so the internal EEPROM can be programmed."
- note removed: "Jumper to disconnect octavo from OPD power"
- note removed: "Only need to connect 7 bits"
- note removed: "TODO - Breakout SPI - Breakout UART0 - Breakout PRU bus? - PRU debug signals - Breakout I2C0 - Breakout EEPROM_WP - Pulldiown on PRU0_7"
- note removed: "TODO Delete this cap if VDD unused"
- note removed: "TODO add optional resistors from AM335X datasheet?"
- note removed: "TODO connect sysboot 2 to opd GPIO"
- note removed: "To other sheet"
- note removed: "USB Client Circuit"
- note removed: "USB ESD protection"
- moved on the sheet: C1, C10, C11, C12, C16, C17, C2, C20, C21, C23, C24, C25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

Commit message: oh god almost done
Parts:
- J1: value ORESAT-DEBUG-CONNECTOR-CARD -> ORESAT-DEBUG-CONNECTOR-ALL; device oresat-debug-connector:ORESAT-DEBUG-CONNECTOR-CARD -> oresat-debug-connector:ORESAT-DEBUG-CONNECTOR-ALL
- JP1: value JUMPER-SMT_2_NC_TRACE_NO-SILK -> JUMPER-SMT_2_NC_TRACE_SILK; device SparkFun-Jumpers:JUMPER-SMT_2_NC_TRACE_NO-SILK -> SparkFun-Jumpers:JUMPER-SMT_2_NC_TRACE_SILK
Connections:
- removed net USB_HO_N: J1.HOST-D-
- removed net USB_HO_PX: J1.HOST-D+
- removed net USB_HO_VBUS: J1.DEBUG-0
Other:
- note added: "24MHz XO"
- note added: "32.768 KHz RTC XO"
- note added: "<-- To Connectors Sheet"
- note removed: "24MHz RTC XO"
- note removed: "GPIO -> PIN map gpio3_9 == mii1_tx_clk gpio0_28 == mii1_txd0 gpio0_21 == mii1_txd1 gpio0_17 == mii1_txd2 gpio0_16 == mii1_txd3 gpio3_3 == mii1_tx_en gpio3_1 == mii1_crs gpio3_0 == mii1_col gpio3_10 == mii1_rx_clk gpio2_21 == mii1_rxd0 gpio2_20 == mii1_rxd1 gpio2_19 == mii1_rxd2 gpio2_18 == mii1_rxd3 gpio3_2 == mii1_rx_er gpio3_4 == mii1_rx_dv gpio0_0 == mdio"
- note removed: "See Connectors Sheet"
- note removed: "TODO - DONE Breakout SPI1 - DONE Breakout UART0 - DONE Breakout PRU bus? - PRU debug signals labels - DONE Breakout I2C0 - DONE Breakout EEPROM_WP - DONE Pulldown on PRU0_7 - DONE OPD boot pin"
- note removed: "taken verbatim from PB,"
- moved on the sheet: C1, C11, C16, C17, C20, C21, C23, C24, C25, C26, C27, C28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

Commit message: boards finished
Parts:
- R50: value 0 -> 10k
- R51: value NP -> 4.7k
Other:
- moved on the sheet: TP33, TP34
Changed lines of the file:
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@@
 <part name="R39" library="oresat-rcl" deviceset="R-US_" device="0603-A" value="10k"/>
 <part name="GND25" library="supply1" library_urn="urn:adsk.eagle:library:371" deviceset="GND" device=""/>
-<part name="R50" library="oresat-rcl" deviceset="R-US_" device="0603-A" value="0"/>
-<part name="R51" library="oresat-rcl" deviceset="R-US_" device="0603-A" value="NP">
+<part name="R50" library="oresat-rcl" deviceset="R-US_" device="0603-A" value="10k"/>
+<part name="R51" library="oresat-rcl" deviceset="R-US_" device="0603-A" value="4.7k">
 <attribute name="DIS" value="Digi-Key"/>
 <attribute name="DPN" value="1276-4275-1-ND"/>
@@
 <attribute name="NAME" x="283.21" y="387.35" size="1.778" layer="95" font="vector"/>
 </instance>
-<instance part="TP33" gate="G$1" x="353.06" y="281.94" smashed="yes">
-<attribute name="NAME" x="355.346" y="282.194" size="1.778" layer="95" font="vector"/>
+<instance part="TP33" gate="G$1" x="347.98" y="281.94" smashed="yes">
+<attribute name="NAME" x="350.266" y="282.194" size="1.778" layer="95" font="vector"/>
 </instance>
-<instance part="TP34" gate="G$1" x="353.06" y="279.4" smashed="yes">
-<attribute name="NAME" x="355.346" y="279.654" size="1.778" layer="95" font="vector"/>
+<instance part="TP34" gate="G$1" x="347.98" y="279.4" smashed="yes">
+<attribute name="NAME" x="350.266" y="279.654" size="1.778" layer="95" font="vector"/>
 </instance>
 <instance part="JP1" gate="G$1" x="185.42" y="86.36" smashed="yes">
@@
 <wire x1="241.3" y1="248.92" x2="309.88" y2="248.92" width="0.762" layer="92"/>
 <wire x1="309.88" y1="248.92" x2="309.88" y2="111.76" width="0.762" layer="92"/>
-<wire x1="309.88" y1="248.92" x2="365.76" y2="248.92" width="0.762" layer="92"/>
-<wire x1="365.76" y1="248.92" x2="365.76" y2="281.94" width="0.762" layer="92"/>
+<wire x1="309.88" y1="248.92" x2="373.38" y2="248.92" width="0.762" layer="92"/>
+<wire x1="373.38" y1="248.92" x2="373.38" y2="281.94" width="0.762" layer="92"/>
 </segment>
 </bus>
@@
 <segment>
 <pinref part="U7" gate="C" pin="GPMC_AD12"/>
-<wire x1="345.44" y1="281.94" x2="353.06" y2="281.94" width="0.1524" layer="91"/>
+<wire x1="345.44" y1="281.94" x2="347.98" y2="281.94" width="0.1524" layer="91"/>
 <pinref part="TP33" gate="G$1" pin="1"/>
-<wire x1="353.06" y1="281.94" x2="365.76" y2="281.94" width="0.1524" layer="91"/>
-<junction x="353.06" y="281.94"/>
+<wire x1="347.98" y1="281.94" x2="373.38" y2="281.94" width="0.1524" layer="91"/>
+<junction x="347.98" y="281.94"/>
+<label x="358.14" y="281.94" size="1.778" layer="95"/>
 </segment>
 </net>
@@
 <segment>
 <pinref part="U7" gate="C" pin="GPMC_AD13"/>
-<wire x1="345.44" y1="279.4" x2="353.06" y2="279.4" width="0.1524" layer="91"/>
+<wire x1="345.44" y1="279.4" x2="347.98" y2="279.4" width="0.1524" layer="91"/>
 <pinref part="TP34" gate="G$1" pin="1"/>
-<wire x1="353.06" y1="279.4" x2="365.76" y2="279.4" width="0.1524" layer="91"/>
-<junction x="353.06" y="279.4"/>
+<wire x1="347.98" y1="279.4" x2="373.38" y2="279.4" width="0.1524" layer="91"/>
+<junction x="347.98" y="279.4"/>
+<label x="358.14" y="279.4" size="1.778" layer="95"/>
 </segment>
 </net>

Commit message: fixed resistor array value
Parts:
- R16, R17: value EXB-2HV103JV -> 100k
Changed lines of the file:
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@@
 <part name="R14" library="oresat-rcl" deviceset="R-US_" device="0603-A" value="DNP"/>
 <part name="GND45" library="SparkFun-PowerSymbols" deviceset="GND" device=""/>
-<part name="R16" library="R-Panasonic-EXB-2HV103JV" deviceset="EXB-2HV103JV" device=""/>
+<part name="R16" library="R-Panasonic-EXB-2HV103JV" deviceset="EXB-2HV103JV" device="" value="100k"/>
 <part name="GND46" library="SparkFun-PowerSymbols" deviceset="GND" device=""/>
-<part name="R17" library="R-Panasonic-EXB-2HV103JV" deviceset="EXB-2HV103JV" device=""/>
+<part name="R17" library="R-Panasonic-EXB-2HV103JV" deviceset="EXB-2HV103JV" device="" value="100k"/>
 <part name="GND48" library="SparkFun-PowerSymbols" deviceset="GND" device=""/>
 <part name="3V-6" library="oresat-supplies" deviceset="3.3V" device=""/>

Commit message: update attributes
Parts:
- C33: MPN CL05B104KO5NNNC -> (none)
Changed lines of the file:
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@@
 <attribute name="DPN" value="1276-1001-1-ND"/>
 <attribute name="MFR" value="Samsung"/>
-<attribute name="MPN" value="CL05B104KO5NNNC"/>
+<attribute name="MPN" value=""/>
 </part>
 <part name="GND28" library="supply1" library_urn="urn:adsk.eagle:library:371" deviceset="GND" device=""/>
@@
 </instance>
 <instance part="C17" gate="CE" x="241.3" y="187.96" smashed="yes">
-<attribute name="NAME" x="242.824" y="188.341" size="1.778" layer="95"/>
+<attribute name="NAME" x="240.284" y="193.421" size="1.778" layer="95"/>
 <attribute name="VALUE" x="242.824" y="183.261" size="1.778" layer="96"/>
 <attribute name="MPN" x="241.3" y="187.96" size="1.778" layer="96" display="off"/>
