File: cfc-sensor-card-v2/cfc-sensor-card-sch-pirt.kicad_sch (KiCad schematic)
At the start: 75 parts, among them U1 TLC3704IPWR, U10 LT3042IMSE, U11 LT3042IMSE, U12 U-PIRT-PIRT1280A1-12, U13 XO_ISM95-XXXXXX, U6 LP2985-3.3, U7 LT3042IMSE, U8 LT3042IMSE, U9 LT3042IMSE

Commit message: Schematic Changes
Made schematic into hierarchy view. Revised OPD to match modern OPD. Removed connectors page. Separated power sequencing and PIRT sensor into 2 pages.
Parts:
- removed C10, C14, C15, C16, C17, C18, C24, C25, C26, C27, C28: 4.7u, Capacitor_SMD:C_0603_1608Metric_Pad1.08x0.95mm_HandSolder, symbol Device:C_Small
- removed C13, C6, C7: 1u, Capacitor_SMD:C_0603_1608Metric_Pad1.08x0.95mm_HandSolder, symbol Device:C_Small
- removed C19, C20, C21, C22, C23: 470n, Capacitor_SMD:C_0603_1608Metric_Pad1.08x0.95mm_HandSolder, symbol Device:C_Small
- removed C29, C31, C32, C33, C34, C35, C9: 100n, Capacitor_SMD:C_0603_1608Metric_Pad1.08x0.95mm_HandSolder, symbol Device:C_Small
- removed D2: GREEN, LED_SMD:LED_0603_1608Metric, symbol Device:LED_Small
- removed R26, R27, R28, R29, R33, R42, R43, R44, R45, R48, R49, R50, R51: 10K, Resistor_SMD:R_0603_1608Metric_Pad0.98x0.95mm_HandSolder, symbol Device:R_Small_US
- removed R46: 330K, Resistor_SMD:R_0603_1608Metric_Pad0.98x0.95mm_HandSolder, symbol Device:R_Small_US
- removed R47: 4.7K, Resistor_SMD:R_0603_1608Metric_Pad0.98x0.95mm_HandSolder, symbol Device:R_Small_US
- removed R52, R53: 33.2K, Resistor_SMD:R_0603_1608Metric_Pad0.98x0.95mm_HandSolder, symbol Device:R_Small_US
- removed R54: 16.2K, Resistor_SMD:R_0603_1608Metric_Pad0.98x0.95mm_HandSolder, symbol Device:R_Small_US
- removed R55: 9.09K, Resistor_SMD:R_0603_1608Metric_Pad0.98x0.95mm_HandSolder, symbol Device:R_Small_US
- removed R56: 29.4K, Resistor_SMD:R_0603_1608Metric_Pad0.98x0.95mm_HandSolder, symbol Device:R_Small_US
- removed TP16, TP17, TP20, TP23, TP24, TP25, TP26, TP27, TP28, TP29, TP30, TP31, TP32, TP33, TP34, TP35, TP36, TP37, TP38: TestPoint-MinTH, oresat-misc:TestPoint-MinTH, symbol oresat-misc:TestPoint-MinTH
- removed U1: TLC3704IPWR, Package_SO:TSSOP-14_4.4x5mm_P0.65mm, symbol oresat-ics:TLC3704
- removed U10, U11, U7, U8, U9: LT3042IMSE, oresat-ics:MSOP-10-1EP_3x3mm_P0.5mm_EP1.68x1.88mm_0.254_ThermalVias, symbol oresat-ics:LT3042IMSE
- removed U12: U-PIRT-PIRT1280A1-12, U-PIR-PIRT1280A1-12:PIRT1280A1-12, symbol oresat-ics:U-PIRT-PIRT1280A1-12
- removed U13: XO_ISM95-XXXXXX, oresat-ics:XO_ISM95-XXXXXX, symbol oresat-ics:XO_ISM95-XXXXXX
- removed U6: LP2985-3.3, Package_TO_SOT_SMD:SOT-23-5, symbol Regulator_Linear:LP2985-3.3
- added C60, C61, C62, C63, C64, C65: 100n, Capacitor_SMD:C_0603_1608Metric_Pad1.08x0.95mm_HandSolder, symbol Device:C_Small
- added TP55, TP56: TestPoint-MinTH, oresat-misc:TestPoint_Pad_D1.0mm, symbol Oresat Misc:Test-Point-1mm-round
- added U22: U-PIRT-PIRT1280A1-12, U-PIR-PIRT1280A1-12:PIRT1280A1-12, symbol oresat-ics:U-PIRT-PIRT1280A1-12
- added U23: XO_ISM95-XXXXXX, oresat-ics:XO_ISM95-XXXXXX, symbol oresat-ics:XO_ISM95-XXXXXX
Connections:
- net 3.3V: now also C60.1, U23.4 (VCC)
- net GND: now also C60.2, C61.2, C62.2, C63.2, C64.2, C65.2, U22.17 (VN), U22.29 (VGND), U22.44 (THERM-), U22.6 (VNOUT), U23.2 (GND)
- net OUT1_N: now also U22.14 (OUT1N)
- net OUT1_P: now also U22.13 (OUT1P)
- net SPI_CLK: now also U22.26 (SDCLK)
- net SPI_MISO: now also U22.27 (SDOUT)
- net SPI_MOSI: now also U22.25 (SDIN)
- net TEC+: now also U22.23 (TEC+)
- net TEC-: now also U22.22 (TEC-)
- net THERM+: now also U22.1 (THERM+)
- net TXCLK_N: now also U22.16 (TXCLKN)
- net TXCLK_P: now also U22.15 (TXCLKP)
- net VDETCOM-2.9V: now also C63.1, U22.31 (VDETCOM-2.9V)
- net VPH-3.3V: now also C61.1, U22.19 (VPH-3.3V)
- net VPL-1.6V: now also C65.1, U22.18 (VPL-1.6V)
- net VPOS-3.3V: now also C62.1, U22.30 (VPOS-3.3V)
- net VPOUT-0.9V: now also C64.1, U22.5 (VPOUT-0.9V)
- new net: TP55.1, U22.21 (JAMSYNC)
- new net: TP56.1, U22.20 (REFCLK), U23.3 (CLK)
- new net CLK_EN: U23.1 (INH)
Other:
- note removed: "*** NOTE: SET pins need Low Leakage Cap ***"
- note removed: "3.3 LDO"
- note removed: "PIRT1280 Power Supplies"
- note removed: "PIRT1280 Power Supply Sequencer"
- note removed: "Power Up Sequence: (Down is reverse order) 1: ﻿VPOS, VPH 2: VPL, VPOUT 3: VDETCOM 4: REFCLK"
- note removed: "Power Up/Down sequencer: - Neg inputs of comparator are set to consecutive reference values by voltage divider - Pos inputs are all brought up at a fixed rate by the RC circuit - Comparators with lower reference voltage are enabled first"
- note removed: "RC circuit to raise pos inputs of comparator"
- note removed: "Voltage Divider to set sequencer order"

Commit message: Update
Fixed a couple of library issues on testpoints and other misc components. Added Pull up resistors to 8 channel i2c ic
Parts:
- TP55, TP56: symbol Oresat Misc:Test-Point-1mm-round -> oresat-misc:Test-Point-1mm-round
Changed lines of the file:
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@@
 	)
 	(symbol
-		(lib_id "Oresat Misc:Test-Point-1mm-round")
+		(lib_id "oresat-misc:Test-Point-1mm-round")
 		(at 179.07 142.24 0)
 		(unit 1)
@@
 	)
 	(symbol
-		(lib_id "Oresat Misc:Test-Point-1mm-round")
+		(lib_id "oresat-misc:Test-Point-1mm-round")
 		(at 138.43 137.16 0)
 		(unit 1)

Commit message: Update
Changed passive component footprints to 0603 no silk c. Fixed OPD UART termination resistor on cfc processor card. Added low temp co and tolerance resistor for NTC  thermistor tec voltage divider.
Parts:
- C60, C61, C62, C63, C64, C65: footprint Capacitor_SMD:C_0603_1608Metric_Pad1.08x0.95mm_HandSolder -> oresat-passives:0603-C-NOSILK
Changed lines of the file:
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@@
 			)
 		)
-		(property "Footprint" "Capacitor_SMD:C_0603_1608Metric_Pad1.08x0.95mm_HandSolder"
+		(property "Footprint" "oresat-passives:0603-C-NOSILK"
 			(at 186.69 116.84 0)
 			(hide yes)
@@
 			)
 		)
-		(property "Footprint" "Capacitor_SMD:C_0603_1608Metric_Pad1.08x0.95mm_HandSolder"
+		(property "Footprint" "oresat-passives:0603-C-NOSILK"
 			(at 220.98 101.6 0)
 			(hide yes)
@@
 			)
 		)
-		(property "Footprint" "Capacitor_SMD:C_0603_1608Metric_Pad1.08x0.95mm_HandSolder"
+		(property "Footprint" "oresat-passives:0603-C-NOSILK"
 			(at 220.98 85.09 0)
 			(hide yes)
@@
 			)
 		)
-		(property "Footprint" "Capacitor_SMD:C_0603_1608Metric_Pad1.08x0.95mm_HandSolder"
+		(property "Footprint" "oresat-passives:0603-C-NOSILK"
 			(at 193.04 85.09 0)
 			(hide yes)
@@
 			)
 		)
-		(property "Footprint" "Capacitor_SMD:C_0603_1608Metric_Pad1.08x0.95mm_HandSolder"
+		(property "Footprint" "oresat-passives:0603-C-NOSILK"
 			(at 106.68 127 0)
 			(hide yes)
@@
 			)
 		)
-		(property "Footprint" "Capacitor_SMD:C_0603_1608Metric_Pad1.08x0.95mm_HandSolder"
+		(property "Footprint" "oresat-passives:0603-C-NOSILK"
 			(at 187.96 100.33 0)
 			(hide yes)
