File: cfc-sensor-card-v2/cfc-sensor-card-sch-pirt.kicad_sch (KiCad schematic)
At the start: 10 parts, among them U22 U-PIRT-PIRT1280A1-12, U23 XO_ISM95-XXXXXX

Commit message: Processor board routing
Completed rework and routing of processor board. No drc errors or warnings. Ready for design review on processor board. Minor changes to schematic for easier routing on pull down resistors connected to the octavo SIP. Reannotated sensor schematic component designators.
Parts:
- renumbered C60 to C44, C64 to C45, C65 to C46, C63 to C47, C61 to C48, C62 to C49, TP56 to TP28, TP55 to TP29, U23 to U18, U22 to U19
Changed lines of the file:
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@@
 		(dnp no)
 		(fields_autoplaced yes)
-		(property "Reference" "C64"
+		(property "Reference" "C45"
 			(at 189.23 115.5762 0)
 			(show_name no)
@@
 			(project "cfc-sensor-card"
 				(path "/8c53300c-27d6-4efc-b05b-8b907d6da3f5/908db1a6-8c16-4ec7-b1cc-5d68b8eb28f8"
-					(reference "C64")
+					(reference "C45")
 					(unit 1)
 				)
@@
 		(in_pos_files yes)
 		(dnp no)
-		(property "Reference" "TP55"
+		(property "Reference" "TP29"
 			(at 173.99 142.24 0)
 			(show_name no)
@@
 			(project "cfc-sensor-card"
 				(path "/8c53300c-27d6-4efc-b05b-8b907d6da3f5/908db1a6-8c16-4ec7-b1cc-5d68b8eb28f8"
-					(reference "TP55")
+					(reference "TP29")
 					(unit 1)
 				)
@@
 		(dnp no)
 		(fields_autoplaced yes)
-		(property "Reference" "C62"
+		(property "Reference" "C49"
 			(at 223.52 100.3362 0)
 			(show_name no)
@@
 			(project "cfc-sensor-card"
 				(path "/8c53300c-27d6-4efc-b05b-8b907d6da3f5/908db1a6-8c16-4ec7-b1cc-5d68b8eb28f8"
-					(reference "C62")
+					(reference "C49")
 					(unit 1)
 				)
@@
 		(in_pos_files yes)
 		(dnp no)
-		(property "Reference" "TP56"
+		(property "Reference" "TP28"
 			(at 136.2681 135.1039 0)
 			(show_name no)
@@
 			(project "cfc-sensor-card"
 				(path "/8c53300c-27d6-4efc-b05b-8b907d6da3f5/908db1a6-8c16-4ec7-b1cc-5d68b8eb28f8"
-					(reference "TP56")
+					(reference "TP28")
 					(unit 1)
 				)
@@
 		(in_pos_files yes)
 		(dnp no)
-		(property "Reference" "#GND0116"
+		(property "Reference" "#GND091"
 			(at 227.33 179.07 0)
 			(hide yes)
@@
 			(project "cfc-sensor-card"
 				(path "/8c53300c-27d6-4efc-b05b-8b907d6da3f5/908db1a6-8c16-4ec7-b1cc-5d68b8eb28f8"
-					(reference "#GND0116")
+					(reference "#GND091")
 					(unit 1)
 				)
@@
 		(in_pos_files yes)
 		(dnp no)
-		(property "Reference" "#GND0114"
+		(property "Reference" "#GND088"
 			(at 204.47 187.96 0)
 			(hide yes)
@@
 			(project "cfc-sensor-card"
 				(path "/8c53300c-27d6-4efc-b05b-8b907d6da3f5/908db1a6-8c16-4ec7-b1cc-5d68b8eb28f8"
-					(reference "#GND0114")
+					(reference "#GND088")
 					(unit 1)
 				)
@@
 		(dnp no)
 		(fields_autoplaced yes)
-		(property "Reference" "C61"
+		(property "Reference" "C48"
 			(at 223.52 83.8262 0)
 			(show_name no)
@@
 			(project "cfc-sensor-card"
 				(path "/8c53300c-27d6-4efc-b05b-8b907d6da3f5/908db1a6-8c16-4ec7-b1cc-5d68b8eb28f8"
-					(reference "C61")
+					(reference "C48")
 					(unit 1)
 				)
@@
 		(in_pos_files yes)
 		(dnp no)
-		(property "Reference" "#3V012"
+		(property "Reference" "#3V021"
 			(at 208.28 81.28 0)
 			(hide yes)
@@
 			(project "cfc-sensor-card"
 				(path "/8c53300c-27d6-4efc-b05b-8b907d6da3f5/908db1a6-8c16-4ec7-b1cc-5d68b8eb28f8"
-					(reference "#3V012")
+					(reference "#3V021")
 					(unit 1)
 				)
@@
 		(dnp no)
 		(fields_autoplaced yes)
-		(property "Reference" "#GND0117"
+		(property "Reference" "#GND089"
 			(at 220.98 97.79 0)
 			(hide yes)
@@
 			(project "cfc-sensor-card"
 				(path "/8c53300c-27d6-4efc-b05b-8b907d6da3f5/908db1a6-8c16-4ec7-b1cc-5d68b8eb28f8"
-					(reference "#GND0117")
+					(reference "#GND089")
 					(unit 1)
 				)
@@
 		(in_pos_files yes)
 		(dnp no)
-		(property "Reference" "#3V013"
+		(property "Reference" "#3V018"
 			(at 196.85 116.84 0)
 			(hide yes)
@@
 			(project "cfc-sensor-card"
 				(path "/8c53300c-27d6-4efc-b05b-8b907d6da3f5/908db1a6-8c16-4ec7-b1cc-5d68b8eb28f8"
-					(reference "#3V013")
+					(reference "#3V018")
 					(unit 1)
 				)
@@
 		(in_pos_files yes)
 		(dnp no)
-		(property "Reference" "#3V010"
+		(property "Reference" "#3V022"
 			(at 212.09 101.6 0)
 			(hide yes)
@@
 			(project "cfc-sensor-card"
 				(path "/8c53300c-27d6-4efc-b05b-8b907d6da3f5/908db1a6-8c16-4ec7-b1cc-5d68b8eb28f8"
-					(reference "#3V010")
+					(reference "#3V022")
 					(unit 1)
 				)
@@
 		(in_pos_files yes)
 		(dnp no)
-		(property "Reference" "C63"
+		(property "Reference" "C47"
 			(at 190.5 83.8262 0)
 			(show_name no)
@@
 			(project "cfc-sensor-card"
 				(path "/8c53300c-27d6-4efc-b05b-8b907d6da3f5/908db1a6-8c16-4ec7-b1cc-5d68b8eb28f8"
-					(reference "C63")
+					(reference "C47")
 					(unit 1)
 				)
@@
 		(dnp no)
 		(fields_autoplaced yes)
-		(property "Reference" "C60"
+		(property "Reference" "C44"
 			(at 109.22 125.7362 0)
 			(show_name no)
@@
 			(project "cfc-sensor-card"
 				(path "/8c53300c-27d6-4efc-b05b-8b907d6da3f5/908db1a6-8c16-4ec7-b1cc-5d68b8eb28f8"
-					(reference "C60")
+					(reference "C44")
 					(unit 1)
 				)
@@
 		(in_pos_files yes)
 		(dnp no)
-		(property "Reference" "#GND0118"
+		(property "Reference" "#GND090"
 			(at 220.98 113.03 0)
 			(hide yes)
@@
 			(project "cfc-sensor-card"
 				(path "/8c53300c-27d6-4efc-b05b-8b907d6da3f5/908db1a6-8c16-4ec7-b1cc-5d68b8eb28f8"
-					(reference "#GND0118")
+					(reference "#GND090")
 					(unit 1)
 				)
@@
 		(in_pos_files yes)
 		(dnp no)
-		(property "Reference" "#GND0121"
+		(property "Reference" "#GND085"
 			(at 186.69 128.27 0)
 			(hide yes)
@@
 			(project "cfc-sensor-card"
 				(path "/8c53300c-27d6-4efc-b05b-8b907d6da3f5/908db1a6-8c16-4ec7-b1cc-5d68b8eb28f8"
-					(reference "#GND0121")
+					(reference "#GND085")
 					(unit 1)
 				)
@@
 		(in_pos_files yes)
 		(dnp no)
-		(property "Reference" "#GND0120"
+		(property "Reference" "#GND086"
 			(at 187.96 111.76 0)
 			(hide yes)
@@
 			(project "cfc-sensor-card"
 				(path "/8c53300c-27d6-4efc-b05b-8b907d6da3f5/908db1a6-8c16-4ec7-b1cc-5d68b8eb28f8"
-					(reference "#GND0120")
+					(reference "#GND086")
 					(unit 1)
 				)
@@
 		(dnp no)
 		(fields_autoplaced yes)
-		(property "Reference" "#3V08"
+		(property "Reference" "#3V017"
 			(at 120.65 127 0)
 			(hide yes)
@@
 			(project "cfc-sensor-card"
 				(path "/8c53300c-27d6-4efc-b05b-8b907d6da3f5/908db1a6-8c16-4ec7-b1cc-5d68b8eb28f8"
-					(reference "#3V08")
+					(reference "#3V017")
 					(unit 1)
 				)
@@
 		(in_pos_files yes)
 		(dnp no)
-		(property "Reference" "U23"
+		(property "Reference" "U18"
 			(at 135.89 127 0)
 			(show_name no)
@@
 			(project "cfc-sensor-card"
 				(path "/8c53300c-27d6-4efc-b05b-8b907d6da3f5/908db1a6-8c16-4ec7-b1cc-5d68b8eb28f8"
-					(reference "U23")
+					(reference "U18")
 					(unit 1)
 				)
@@
 		(in_pos_files yes)
 		(dnp no)
-		(property "Reference" "#3V014"
+		(property "Reference" "#3V020"
 			(at 204.47 81.28 0)
 			(hide yes)
@@
 			(project "cfc-sensor-card"
 				(path "/8c53300c-27d6-4efc-b05b-8b907d6da3f5/908db1a6-8c16-4ec7-b1cc-5d68b8eb28f8"
-					(reference "#3V014")
+					(reference "#3V020")
 					(unit 1)
 				)
@@
 		(in_pos_files yes)
 		(dnp no)
-		(property "Reference" "U22"
+		(property "Reference" "U19"
 			(at 209.55 179.07 0)
 			(show_name no)
@@
 			(project "cfc-sensor-card"
 				(path "/8c53300c-27d6-4efc-b05b-8b907d6da3f5/908db1a6-8c16-4ec7-b1cc-5d68b8eb28f8"
-					(reference "U22")
+					(reference "U19")
 					(unit 1)
 				)
@@
 		(in_pos_files yes)
 		(dnp no)
-		(property "Reference" "C65"
+		(property "Reference" "C46"
 			(at 181.356 99.06 0)
 			(show_name no)
@@
 			(project "cfc-sensor-card"
 				(path "/8c53300c-27d6-4efc-b05b-8b907d6da3f5/908db1a6-8c16-4ec7-b1cc-5d68b8eb28f8"
-					(reference "C65")
+					(reference "C46")
 					(unit 1)
 				)
@@
 		(in_pos_files yes)
 		(dnp no)
-		(property "Reference" "#3V011"
+		(property "Reference" "#3V019"
 			(at 200.66 101.6 0)
 			(hide yes)
@@
 			(project "cfc-sensor-card"
 				(path "/8c53300c-27d6-4efc-b05b-8b907d6da3f5/908db1a6-8c16-4ec7-b1cc-5d68b8eb28f8"
-					(reference "#3V011")
+					(reference "#3V019")
 					(unit 1)
 				)
@@
 		(in_pos_files yes)
 		(dnp no)
-		(property "Reference" "#GND0119"
+		(property "Reference" "#GND087"
 			(at 193.04 96.52 0)
 			(hide yes)
@@
 			(project "cfc-sensor-card"
 				(path "/8c53300c-27d6-4efc-b05b-8b907d6da3f5/908db1a6-8c16-4ec7-b1cc-5d68b8eb28f8"
-					(reference "#GND0119")
+					(reference "#GND087")
 					(unit 1)
 				)
@@
 		(in_pos_files yes)
 		(dnp no)
-		(property "Reference" "#GND0115"
+		(property "Reference" "#GND084"
 			(at 120.65 153.67 0)
 			(hide yes)
@@
 			(project "cfc-sensor-card"
 				(path "/8c53300c-27d6-4efc-b05b-8b907d6da3f5/908db1a6-8c16-4ec7-b1cc-5d68b8eb28f8"
-					(reference "#GND0115")
+					(reference "#GND084")
 					(unit 1)
 				)
@@
 		(dnp no)
 		(fields_autoplaced yes)
-		(property "Reference" "#GND0113"
+		(property "Reference" "#GND083"
 			(at 106.68 137.16 0)
 			(hide yes)
@@
 			(project "cfc-sensor-card"
 				(path "/8c53300c-27d6-4efc-b05b-8b907d6da3f5/908db1a6-8c16-4ec7-b1cc-5d68b8eb28f8"
-					(reference "#GND0113")
-					(unit 1)
-				)
+					(reference "#GND083")
+					(unit 1)
+				)
