File: cfc-sensor-card-v2/cfc-sensor-card.kicad_pcb (KiCad board)
At the start: 4 copper layers, 99.8 x 94.6 mm, 190 parts, among them J1 TFM-120-01-L-D-RA, J2 J-SAMTEC-TFM-110-X1-XXX-D-RA, Q1 DMP2240UDM, Q2 PMV45EN, Q3 DMP3050LVT-7, Q4 DMP3050LVT-7, Q5 PMV45EN, U1 MIC842LYC5, U10 LT3042IMSE, U11 LT3042IMSE, U12 AD5593RBCPZ-RL7, U13 SN74LVC1G86DBVR, U14 SN74LVC1G08DCKR, U15 MP2410A, U16 DRV8212DSGR, U17 INA186A1IDCKR, U18 XO_ISM95-XXXXXX, U19 U-PIRT-PIRT1280A1-12, U2 MIC842LYC5, U3 MAX7310ATE+, U4 MAX4211FETE, U5 LP2985-3.3, U6 TLC3704IPWR, U7 LT3042IMSE, U8 LT3042IMSE, U9 LT3042IMSE

Commit message: Update
Updated OPD to align with proto card. Made changes from DR with Greenberg. Moved around polygon pours, led indicators, silkscreen issue date, etc. Ready for fab.
Routing:
- net Net-(U6-1OUT): track 134.7 -> 79.1 mm, vias 6 -> 4
- net Net-(U10-EN/UV): track 120.3 -> 70.5 mm
- net 3.3V: track 72.2 -> 35.2 mm
- net /OPD/ON/~{OFF}: track 152.1 -> 126.5 mm
- net Net-(U16-VM): track 3.15 -> 0.00 mm, vias 7 -> 6
Changed lines of the file:
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@@
 	)
 	(segment
-		(start 221.501626 173.8786)
-		(end 217.8284 170.205374)
-		(width 0.2032)
-		(layer "F.Cu")
-		(net "3.3V")
-	)
-	(segment
-		(start 217.8284 170.205374)
-		(end 217.8284 167.624348)
-		(width 0.2032)
-		(layer "F.Cu")
-		(net "3.3V")
-	)
-	(segment
 		(start 221.007642 205.62814)
 		(end 216.409142 205.62814)
@@
 	)
 	(segment
-		(start 199.8706 165.6744)
-		(end 192.5 173.045)
-		(width 0.2032)
-		(layer "F.Cu")
-		(net "3.3V")
-	)
-	(segment
 		(start 227.357642 188.89064)
 		(end 228.627642 190.16064)
@@
 	)
 	(segment
-		(start 215.878452 165.6744)
-		(end 199.8706 165.6744)
-		(width 0.2032)
-		(layer "F.Cu")
-		(net "3.3V")
-	)
-	(segment
 		(start 226.595642 194.83314)
 		(end 226.595642 203.85014)
@@
 	)
 	(segment
-		(start 217.8284 167.624348)
-		(end 215.878452 165.6744)
-		(width 0.2032)
-		(layer "F.Cu")
-		(net "3.3V")
-	)
-	(segment
 		(start 182.005 93.9349)
 		(end 181.9641 93.894)
@@
 	)
 	(segment
-		(start 218.1586 167.487574)
-		(end 216.015226 165.3442)
-		(width 0.2032)
-		(layer "F.Cu")
-		(net "Net-(U10-EN{slash}UV)")
-	)
-	(segment
-		(start 218.1586 170.0686)
-		(end 218.1586 167.487574)
-		(width 0.2032)
-		(layer "F.Cu")
-		(net "Net-(U10-EN{slash}UV)")
-	)
-	(segment
 		(start 180.37 156.495974)
 		(end 180.37 116.913)
@@
 	)
 	(segment
-		(start 216.015226 165.3442)
-		(end 189.218226 165.3442)
-		(width 0.2032)
-		(layer "F.Cu")
-		(net "Net-(U10-EN{slash}UV)")
-	)
-	(segment
 		(start 173.861 110.404)
 		(end 173.861 108.499)
@@
 	)
 	(segment
-		(start 189.218226 165.3442)
-		(end 180.37 156.495974)
-		(width 0.2032)
-		(layer "F.Cu")
-		(net "Net-(U10-EN{slash}UV)")
-	)
-	(segment
 		(start 219.333142 201.07964)
 		(end 219.333142 201.69114)
@@
 	)
 	(segment
-		(start 221.6384 173.5484)
-		(end 218.1586 170.0686)
-		(width 0.2032)
-		(layer "F.Cu")
-		(net "Net-(U10-EN{slash}UV)")
-	)
-	(segment
 		(start 217.520142 202.22914)
 		(end 216.44583 202.22914)
@@
 	)
 	(segment
-		(start 213.04 166.43)
-		(end 213.4654 166.0046)
-		(width 0.2032)
-		(layer "F.Cu")
-		(net "/OPD/ON{slash}~{OFF}")
-	)
-	(segment
 		(start 243.412 96.135)
 		(end 243.076 95.799)
@@
 	)
 	(segment
-		(start 213.4654 166.0046)
-		(end 215.741678 166.0046)
-		(width 0.2032)
-		(layer "F.Cu")
-		(net "/OPD/ON{slash}~{OFF}")
-	)
-	(segment
 		(start 229.106242 192.999383)
 		(end 229.106242 188.32674)
@@
 	)
 	(segment
-		(start 264.8906 152.5386)
-		(end 258.87 146.518)
-		(width 0.2032)
-		(layer "F.Cu")
-		(net "/OPD/ON{slash}~{OFF}")
-	)
-	(segment
 		(start 236.472 94.603672)
 		(end 236.472 96.307)
@@
 	)
 	(segment
-		(start 217.4982 167.761122)
-		(end 217.4982 170.342147)
-		(width 0.2032)
-		(layer "F.Cu")
-		(net "/OPD/ON{slash}~{OFF}")
-	)
-	(segment
 		(start 242.568 95.799)
 		(end 240.8905 95.799)
@@
 	)
 	(segment
-		(start 215.741678 166.0046)
-		(end 217.4982 167.761122)
-		(width 0.2032)
-		(layer "F.Cu")
-		(net "/OPD/ON{slash}~{OFF}")
-	)
-	(segment
 		(start 227.074242 195.031383)
 		(end 229.106242 192.999383)
@@
 	)
 	(segment
-		(start 217.4982 170.342147)
-		(end 221.364852 174.2088)
-		(width 0.2032)
-		(layer "F.Cu")
-		(net "/OPD/ON{slash}~{OFF}")
-	)
-	(segment
 		(start 220.996016 206.10674)
 		(end 225.015884 206.10674)
@@
 	)
 	(segment
-		(start 213.04 170.029)
-		(end 213.04 166.43)
-		(width 0.2032)
-		(layer "F.Cu")
-		(net "/OPD/ON{slash}~{OFF}")
-	)
-	(segment
 		(start 235.5595 94.275)
 		(end 236.143328 94.275)
@@
 		(net "/SPI_MOSI")
 	)
-	(segment
-		(start 215.39 169.8165)
-		(end 215.39 166.665)
-		(width 0.2032)
-		(layer "F.Cu")
-		(net "Net-(U16-VM)")
-	)
 	(via
 		(at 234.948 148.885)
@@
 	)
 	(via
-		(at 215.39 166.665)
-		(size 0.4572)
-		(drill 0.254)
-		(layers "F.Cu" "B.Cu")
-		(capping no)
-		(covering
-			(front no)
-			(back no)
-		)
-		(plugging
-			(front no)
-			(back no)
-		)
-		(filling no)
-		(net "Net-(U16-VM)")
-	)
-	(via
 		(at 234.948 150.409)
 		(size 0.4572)
@@
 	)
 	(segment
-		(start 180.82 156.479)
-		(end 189.355 165.014)
-		(width 0.2032)
-		(layer "F.Cu")
-		(net "Net-(U6-1OUT)")
-	)
-	(segment
 		(start 223.039642 202.45314)
 		(end 222.889142 202.30264)
@@
 	)
 	(segment
-		(start 214.22 170.029)
-		(end 214.22 166.82)
-		(width 0.2032)
-		(layer "F.Cu")
-		(net "Net-(U6-1OUT)")
-	)
-	(segment
-		(start 214.24 165.014)
-		(end 210.945 165.014)
-		(width 0.2032)
-		(layer "F.Cu")
-		(net "Net-(U6-1OUT)")
-	)
-	(segment
-		(start 216.152 165.014)
-		(end 214.24 165.014)
-		(width 0.2032)
-		(layer "F.Cu")
-		(net "Net-(U6-1OUT)")
-	)
-	(segment
-		(start 189.355 165.014)
-		(end 210.945 165.014)
-		(width 0.2032)
-		(layer "F.Cu")
-		(net "Net-(U6-1OUT)")
-	)
-	(segment
 		(start 221.601207 202.39474)
 		(end 221.874242 202.121705)
@@
 	)
 	(segment
-		(start 218.4888 167.3508)
-		(end 216.152 165.014)
-		(width 0.2032)
-		(layer "F.Cu")
-		(net "Net-(U6-1OUT)")
-	)
-	(segment
-		(start 221.775174 173.2182)
-		(end 218.4888 169.931826)
-		(width 0.2032)
-		(layer "F.Cu")
-		(net "Net-(U6-1OUT)")
-	)
-	(segment
-		(start 214.22 164.46)
-		(end 214.22 164.994)
-		(width 0.2032)
-		(layer "F.Cu")
-		(net "Net-(U6-1OUT)")
-	)
-	(segment
 		(start 217.520142 202.87914)
 		(end 218.295642 202.87914)
@@
 		(net "Net-(U6-1OUT)")
 	)
-	(segment
-		(start 214.22 164.994)
-		(end 214.24 165.014)
-		(width 0.2032)
-		(layer "F.Cu")
-		(net "Net-(U6-1OUT)")
-	)
-	(segment
-		(start 218.4888 169.931826)
-		(end 218.4888 167.3508)
-		(width 0.2032)
-		(layer "F.Cu")
-		(net "Net-(U6-1OUT)")
-	)
 	(via
 		(at 177.036 110.912)
@@
 		(net "Net-(U6-1OUT)")
 	)
-	(via
-		(at 214.22 164.46)
-		(size 0.4572)
-		(drill 0.254)
-		(layers "F.Cu" "B.Cu")
-		(net "Net-(U6-1OUT)")
-	)
-	(via
-		(at 214.22 166.82)
-		(size 0.4572)
-		(drill 0.254)
-		(layers "F.Cu" "B.Cu")
-		(net "Net-(U6-1OUT)")
-	)
-	(segment
-		(start 214.22 166.82)
-		(end 214.22 164.46)
-		(width 0.2032)
-		(layer "B.Cu")
-		(net "Net-(U6-1OUT)")
-	)

Commit message: Updated OPD on sensor card
updated OPD on sensor card to match protocard. Finished placement on PCB.
Parts:
- D1: value AMBER -> AMB
- Q2, Q5: value PMV45EN -> DMN2050LQ-7
- Q4: value DMP3050LVT-7 -> DMPH2040UVTQ-7
- R11: value 10 -> 100
- moved C31 75.8 mm to (209.4, 170.5), turned to 180 degrees
- moved C32 73.9 mm to (211.7, 170.5)
- moved R53 71.2 mm to (176.8, 161.7), turned to 180 degrees
- moved R52 71.1 mm to (176.8, 160.2), turned to 180 degrees
- moved TP11 67.5 mm to (166.6, 168.8)
- moved TP13 67.5 mm to (166.6, 170.6)
- moved TP14 67.5 mm to (166.6, 174.2)
- moved TP15 67.5 mm to (166.6, 172.4)
- moved TP16 67.5 mm to (166.6, 177.7)
- moved TP17 67.5 mm to (166.6, 175.9)
- moved C34 66.1 mm to (214.8, 168.8)
- moved R61 66.1 mm to (214.8, 166.5)
- moved U12 66.1 mm to (210.5, 167.4)
- moved R59 64.4 mm to (209.1, 164.8)
- moved C11 61.0 mm to (174.7, 150.4)
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Connections:
- C38 pad 2: /PIRT/TEC- -> Net-(C38-Pad2)
- R63 pad 2: /PIRT/TEC- -> Net-(C38-Pad2)
- R64 pad 1: /PIRT/TEC- -> Net-(C38-Pad2)
Routing:
- net /SENSOR_ENABLE: track 145.3 -> 25.1 mm, vias 2 -> 0
- net /SPI_MOSI: track 119.5 -> 27.2 mm
- net /SPI_CLK: track 114.8 -> 25.5 mm
- net /SPI_MISO: track 116.6 -> 29.1 mm
- net VPH-3.3V: track 140.0 -> 75.1 mm
- net /OPD/ON/~{OFF}: track 126.5 -> 62.3 mm, vias 3 -> 2
- net VPL-1.6V: track 131.7 -> 67.8 mm
- net VPOUT-0.9V: track 108.8 -> 45.4 mm
- net Net-(U6-1OUT): track 79.1 -> 25.0 mm, vias 4 -> 2
- net Net-(U10-EN/UV): track 70.5 -> 20.4 mm, vias 2 -> 0
- net VPOS-3.3V: track 56.9 -> 7.17 mm, vias 1 -> 0
- net /I2C1_SDA: track 69.0 -> 26.5 mm
- net VDETCOM-2.9V: track 53.1 -> 20.4 mm, vias 1 -> 0
- net 3.3V: track 35.2 -> 3.54 mm
- net Net-(U6-1IN+): track 21.0 -> 0.00 mm, vias 1 -> 0
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
Commit message: Update
Finished sensor board routing. Ready for DR.
Parts:
- moved TP10 125.9 mm to (248.7, 88.0)
- moved TP23 66.2 mm to (224.4, 158.6), turned to 90 degrees
- moved TP27 65.8 mm to (173.8, 111.9), turned to -90 degrees
- moved TP25 63.5 mm to (173.8, 113.3), turned to -90 degrees
- moved TP24 61.4 mm to (173.8, 114.8), turned to -90 degrees
- moved TP26 58.1 mm to (213.5, 158.6), turned to 90 degrees
- moved TP11 29.6 mm to (194.0, 157.4), turned to -90 degrees
- moved TP15 28.8 mm to (193.0, 160.8)
- moved TP14 28.8 mm to (193.0, 162.6)
- moved TP13 28.3 mm to (191.6, 157.4), turned to -90 degrees
- moved TP16 19.4 mm to (178.7, 162.6)
- moved TP17 19.4 mm to (178.7, 160.8)
- moved TP12 19.2 mm to (176.7, 160.4), turned to 90 degrees
- moved R59 15.7 mm to (221.7, 174.2), turned to 180 degrees
- moved C31 12.2 mm to (221.4, 168.4), turned to 0 degrees
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Routing:
- net /PIRT/CLK_EN: track 0.00 -> 159.7 mm, vias 0 -> 2
- net Net-(U6-1OUT): track 25.0 -> 161.3 mm, vias 2 -> 7
- net /I2C1_CLK: track 1.27 -> 108.5 mm, vias 0 -> 1
- net /SPI_MOSI: track 27.2 -> 120.0 mm
- net /PIRT/THERM+: track 4.86 -> 94.7 mm
- net /SPI_CLK: track 25.5 -> 114.8 mm
- net /SPI_MISO: track 29.1 -> 116.0 mm
- net /I2C1_SDA: track 26.5 -> 107.0 mm, vias 0 -> 1
- net /OPD/ON/~{OFF}: track 62.3 -> 125.0 mm, vias 2 -> 3
- net /SENSOR_ENABLE: track 25.1 -> 86.6 mm, vias 0 -> 1
- net VBUSP: track 7.88 -> 68.0 mm, vias 35 -> 52
- net Net-(U10-EN/UV): track 20.4 -> 77.7 mm, vias 0 -> 2
- net /TEC Control/CURRENT_SET: track 0.00 -> 48.5 mm, vias 0 -> 2
- net /TEC Control/BRIDGE_EN: track 10.0 -> 50.5 mm, vias 0 -> 3
- net /TEC Control/BRIDGE_DIR: track 6.52 -> 45.6 mm
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- added copper zone on F.Cu, net /PIRT/TEC+
- added copper zone on In2.Cu, net /PIRT/TEC-
- added copper zone on F.Cu, net 3.3V
- added copper zone on In2.Cu, net 3.3V
- added copper zone on F.Cu, net Net-(U15-SW)
- added copper zone on F.Cu, net Net-(U16-OUT2)
- added copper zone on F.Cu, net Net-(U16-VM)
- added copper zone on In2.Cu, net Net-(U16-VM)
- removed copper zone on B.Cu, net Net-(C38-Pad2)
- removed copper zone on B.Cu, net Net-(U16-VM)
