File: cfc-sensor-card-v2/cfc-sensor-card.kicad_pcb (KiCad board)
At the start: 4 copper layers, 99.8 x 94.6 mm, 190 parts, among them J1 TFM-120-01-L-D-RA, J2 J-SAMTEC-TFM-110-X1-XXX-D-RA, Q1 DMP2240UDM, Q2 DMN2050LQ-7, Q3 DMP3050LVT-7, Q4 DMPH2040UVTQ-7, Q5 DMN2050LQ-7, U1 MIC842LYC5, U10 LT3042IMSE, U11 LT3042IMSE, U12 AD5593RBCPZ-RL7, U13 SN74LVC1G86DBVR, U14 SN74LVC1G08DCKR, U15 MP2410A, U16 DRV8212DSGR, U17 INA186A1IDCKR, U18 XO_ISM95-XXXXXX, U19 U-PIRT-PIRT1280A1-12, U2 MIC842LYC5, U3 MAX7310ATE+, U4 MAX4211FETE, U5 LP2985-3.3, U6 TLC3704IPWR, U7 LT3042IMSE, U8 LT3042IMSE, U9 LT3042IMSE

Commit message: Update
Fixed all DRC errors and warnings.
Parts:
- J2: value J-SAMTEC-TFM-110-X1-XXX-D-RA -> Val**
- R12, R13, R16, R17, R20, R3, R32, R33, R5, R6, R7: footprint Resistor_SMD:R_0603_1608Metric_Pad0.98x0.95mm_HandSolder -> oresat-passives:0603-C-NOSILK
- moved G*** 70.5 mm to (205.9, 170.2)
- moved D4 1.41 mm to (257.5, 170.2)
- moved D5 1.13 mm to (259.0, 170.2)
- moved D2 0.85 mm to (260.5, 170.2)
- moved C44 0.77 mm to (263.9, 115.8)
- moved U18 0.77 mm to (263.8, 113.5)
- moved D1 0.57 mm to (261.9, 170.2)
- moved C6 0.30 mm to (243.3, 89.7)
- moved D3 0.29 mm to (263.4, 170.2)
- moved C35 0.22 mm to (261.6, 163.7)
- moved Q4 0.19 mm to (250.1, 92.0)
- moved C40 0.19 mm to (250.0, 163.3)
- moved C41 0.19 mm to (248.5, 163.1)
- moved Q3 0.12 mm to (240.7, 92.0)
- moved C33 0.09 mm to (256.4, 162.8)
Routing:
- net /OPD/OPD_SCL: track 36.1 -> 39.8 mm, vias 0 -> 2
- net /CAN1_H: track 4.57 -> 1.27 mm
- net /CAN1_L: track 4.56 -> 1.27 mm
- net Net-(Q1B-G): track 14.2 -> 17.0 mm, vias 0 -> 2
- net /OPD/OPD_SDA: track 34.3 -> 36.7 mm, vias 0 -> 2
- net VPD: track 83.4 -> 81.7 mm
- net Net-(U1-OUT): track 5.63 -> 4.13 mm
- net /OPD/PEN-SDA-FILT: track 34.9 -> 35.8 mm
- net GND: track 37.7 -> 36.8 mm
- net Net-(U18-CLK): track 36.6 -> 35.8 mm
- net Net-(D2-A): track 1.77 -> 2.42 mm
- net Net-(D4-A): track 2.06 -> 2.65 mm
- net Net-(D1-A): track 1.77 -> 2.31 mm
- net VBUSP: vias 52 -> 50
- net /OPD/CB_CTRL: vias 3 -> 2
Other:
- board text added: "${ISSUE_DATE}"
- board text added: "COOL"
- board text added: "HEAT"
- board text added: "SENSOR EN"
- board text removed: "3.3V"
- board text removed: "Oliver Rew et al ${ISSUE_DATE}"
- board text removed: "SENSOR ENABLE"
- board text removed: "VDETCOM-2.9V"
- board text removed: "VPH-3.3V"
- board text removed: "VPL-1.6V"
- board text removed: "VPOS-3.3V"
- board text removed: "VPOUT-0.9V"

Commit message: Update
Minor changes to silkscreen. Added extra grounding vias with minor routing changes.
Routing:
- net Net-(U6-1OUT): track 161.3 -> 162.9 mm
- net GND: vias 169 -> 208
