File: cfc-processor-card-v2/cfc-processor-sch-sip-b.kicad_sch (KiCad schematic)
At the start: 19 parts, among them U10 RCLAMP0504FB, U7 OSD3358-1G-ISM, Y1 ECS-240-12-30BQ-AEN-TR, Y2 ABS07-32.768KHZ-T

Commit message: Processor board routing
Completed rework and routing of processor board. No drc errors or warnings. Ready for design review on processor board. Minor changes to schematic for easier routing on pull down resistors connected to the octavo SIP. Reannotated sensor schematic component designators.
Parts:
- removed TP23: TEST-POINT3X4, oresat-misc:TestPoint_Pad_D1.0mm, symbol oresat-misc:Test-Point-1mm-round
Connections:
- net at R64.3 (33): now also U7.C8 (AIN5); no longer U7.A8 (AIN0)
- net at R64.4 (44): now also U7.C7 (AIN4)
- net at R64.6 (66): now also U7.C6 (AIN3); no longer U7.C7 (AIN4)
- net at R64.7 (77): now also U7.B6 (AIN2); no longer U7.C6 (AIN3)
- net at R64.8 (88): no longer U7.B6 (AIN2)
- net at R64.9 (99): now also U7.A8 (AIN0); no longer U7.C8 (AIN5)
