File: cfc-processor-card-v2/cfc-processor-sch-sip-b.kicad_sch (KiCad schematic)
At the start: 18 parts, among them U10 RCLAMP0504FB, U7 OSD3358-1G-ISM, Y1 ECS-240-12-30BQ-AEN-TR, Y2 ABS07-32.768KHZ-T

Commit message: Update
Updated BOM, couple of fixes on OPD. Minor routing and layout changes. Removed logic gates from sensor card.
Parts:
- C16, C17: DPN 399-6840-1-ND -> 399-16015-1-ND; MPN C0603C100J5GACAUTO -> C0603C100J1GACAUTO
- C18, C19: DPN 399-C0603C180F5GACAUTOCT-ND -> 399-15781-1-ND; MPN C0603C180F5GACAUTO -> C0603C180J1GACAUTO
- C20, C21: DPN 587-3472-1-ND -> 399-6856-1-ND; MFR Taiyo Yuden -> KEMET; MPN TMK107BJ104KAHT -> C0603C104K5RACAUTO
Changed lines of the file:
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@@
 			)
 		)
-		(property "Description" "Unpolarized capacitor, small symbol"
+		(property "Description" "10 pF ±5% 100V Ceramic Capacitor C0G, NP0 0603 (1608 Metric)"
 			(at 125.73 87.63 0)
 			(hide yes)
@@
 			)
 		)
-		(property "DPN" "399-6840-1-ND"
+		(property "DPN" "399-16015-1-ND"
 			(at 125.73 87.63 90)
 			(hide yes)
@@
 			)
 		)
-		(property "MPN" "C0603C100J5GACAUTO"
+		(property "MPN" "C0603C100J1GACAUTO"
 			(at 125.73 87.63 90)
 			(hide yes)
@@
 			)
 		)
-		(property "Description" "Unpolarized capacitor, small symbol"
+		(property "Description" "0.1 µF ±10% 50V Ceramic Capacitor X7R 0603 (1608 Metric)"
 			(at 139.7 209.55 0)
 			(hide yes)
@@
 			)
 		)
-		(property "DPN" "587-3472-1-ND"
+		(property "DPN" "399-6856-1-ND"
 			(at 139.7 209.55 0)
 			(hide yes)
@@
 			)
 		)
-		(property "MFR" "Taiyo Yuden"
+		(property "MFR" "KEMET"
 			(at 139.7 209.55 0)
 			(hide yes)
@@
 			)
 		)
-		(property "MPN" "TMK107BJ104KAHT"
+		(property "MPN" "C0603C104K5RACAUTO"
 			(at 139.7 209.55 0)
 			(hide yes)
@@
 			)
 		)
-		(property "Description" "Unpolarized capacitor, small symbol"
+		(property "Description" "18 pF ±5% 100V Ceramic Capacitor C0G, NP0 0603 (1608 Metric)"
 			(at 133.35 118.11 0)
 			(hide yes)
@@
 			)
 		)
-		(property "DPN" "399-C0603C180F5GACAUTOCT-ND"
+		(property "DPN" "399-15781-1-ND"
 			(at 133.35 118.11 90)
 			(hide yes)
@@
 			)
 		)
-		(property "MPN" "C0603C180F5GACAUTO"
+		(property "MPN" "C0603C180J1GACAUTO"
 			(at 133.35 118.11 90)
 			(hide yes)
@@
 			)
 		)
-		(property "Description" "Unpolarized capacitor, small symbol"
+		(property "Description" "18 pF ±5% 100V Ceramic Capacitor C0G, NP0 0603 (1608 Metric)"
 			(at 133.35 102.87 0)
 			(hide yes)
@@
 			)
 		)
-		(property "DPN" "399-C0603C180F5GACAUTOCT-ND"
+		(property "DPN" "399-15781-1-ND"
 			(at 133.35 102.87 90)
 			(hide yes)
@@
 			)
 		)
-		(property "MPN" "C0603C180F5GACAUTO"
+		(property "MPN" "C0603C180J1GACAUTO"
 			(at 133.35 102.87 90)
 			(hide yes)
@@
 			)
 		)
-		(property "Description" "Unpolarized capacitor, small symbol"
+		(property "Description" "0.1 µF ±10% 50V Ceramic Capacitor X7R 0603 (1608 Metric)"
 			(at 247.65 87.63 0)
 			(hide yes)
@@
 			)
 		)
-		(property "DPN" "587-3472-1-ND"
+		(property "DPN" "399-6856-1-ND"
 			(at 247.65 87.63 0)
 			(hide yes)
@@
 			)
 		)
-		(property "MFR" "Taiyo Yuden"
+		(property "MFR" "KEMET"
 			(at 247.65 87.63 0)
 			(hide yes)
@@
 			)
 		)
-		(property "MPN" "TMK107BJ104KAHT"
+		(property "MPN" "C0603C104K5RACAUTO"
 			(at 247.65 87.63 0)
 			(hide yes)
@@
 			)
 		)
-		(property "Description" "Unpolarized capacitor, small symbol"
+		(property "Description" "10 pF ±5% 100V Ceramic Capacitor C0G, NP0 0603 (1608 Metric)"
 			(at 125.73 72.39 0)
 			(hide yes)
@@
 			)
 		)
-		(property "DPN" "399-6840-1-ND"
+		(property "DPN" "399-16015-1-ND"
 			(at 125.73 72.39 90)
 			(hide yes)
@@
 			)
 		)
-		(property "MPN" "C0603C100J5GACAUTO"
+		(property "MPN" "C0603C100J1GACAUTO"
 			(at 125.73 72.39 90)
 			(hide yes)

Commit message: Small update
Fixed minor issue with voltage clamp on usb line. Added nreset clamp and changed VBUS pin to USB voltage bus
Connections:
- net 3.3V: no longer C20.1, U10.5 (VCC)
- net USB_CLI_VBUS: now also C20.1, U10.5 (VCC); no longer U10.4 (I3)
- new net nRESET_CLAMP: U10.4 (I3)
Changed lines of the file:
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@@
 	(text "ESD Protection for USB lines"
 		(exclude_from_sim no)
-		(at 113.03 188.468 0)
+		(at 133.858 194.564 0)
 		(effects
 			(font
@@
 	)
 	(junction
-		(at 90.17 170.18)
-		(diameter 0)
-		(color 0 0 0 0)
-	)
-	(junction
 		(at 127 222.25)
 		(diameter 0)
@@
 	)
 	(junction
+		(at 127 170.18)
+		(diameter 0)
+		(color 0 0 0 0)
+	)
+	(junction
 		(at 153.67 87.63)
 		(diameter 0)
@@
 	(wire
 		(pts
+			(xy 127 170.18) (xy 127 196.85)
+		)
+		(stroke
+			(width 0.1524)
+			(type solid)
+		)
+	)
+	(wire
+		(pts
 			(xy 143.51 161.29) (xy 184.15 161.29)
 		)
@@
 	(wire
 		(pts
-			(xy 127 170.18) (xy 90.17 170.18)
-		)
-		(stroke
-			(width 0.1524)
-			(type solid)
-		)
-	)
-	(wire
-		(pts
 			(xy 130.81 72.39) (xy 138.43 72.39)
 		)
@@
 	(wire
 		(pts
-			(xy 90.17 212.09) (xy 90.17 170.18)
-		)
-		(stroke
-			(width 0)
-			(type default)
-		)
-	)
-	(wire
-		(pts
 			(xy 153.67 87.63) (xy 184.15 87.63)
 		)
@@
 	(wire
 		(pts
-			(xy 127 196.85) (xy 127 194.31)
-		)
-		(stroke
-			(width 0.1524)
-			(type solid)
-		)
-	)
-	(wire
-		(pts
 			(xy 128.27 102.87) (xy 130.81 102.87)
 		)
@@
 	(wire
 		(pts
-			(xy 90.17 170.18) (xy 86.36 170.18)
+			(xy 86.36 170.18) (xy 127 170.18)
 		)
 		(stroke
@@
 		(shape bidirectional)
 		(at 83.82 170.18 180)
+		(effects
+			(font
+				(size 1.27 1.27)
+			)
+			(justify right)
+		)
+	)
+	(hierarchical_label "nRESET_CLAMP"
+		(shape input)
+		(at 90.17 212.09 180)
 		(effects
 			(font
@@
 					(unit 1)
 				)
-			)
-		)
-	)
-	(symbol
-		(lib_id "cfc-card-eagle-import:3.3V")
-		(at 127 191.77 0)
-		(unit 1)
-		(body_style 1)
-		(exclude_from_sim no)
-		(in_bom yes)
-		(on_board yes)
-		(in_pos_files yes)
-		(dnp no)
-		(property "Reference" "#3V-014"
-			(at 127 191.77 0)
-			(hide yes)
-			(show_name no)
-			(do_not_autoplace no)
-			(effects
-				(font
-					(size 1.27 1.27)
-				)
-			)
-		)
-		(property "Value" "3.3V"
-			(at 124.46 190.5 0)
-			(show_name no)
-			(do_not_autoplace no)
-			(effects
-				(font
-					(size 1.778 1.5113)
-				)
-				(justify left bottom)
-			)
-		)
-		(property "Footprint" ""
-			(at 127 191.77 0)
-			(hide yes)
-			(show_name no)
-			(do_not_autoplace no)
-			(effects
-				(font
-					(size 1.27 1.27)
-				)
-			)
-		)
-		(property "Datasheet" ""
-			(at 127 191.77 0)
-			(hide yes)
-			(show_name no)
-			(do_not_autoplace no)
-			(effects
-				(font
-					(size 1.27 1.27)
-				)
-			)
-		)
-		(property "Description" ""
-			(at 127 191.77 0)
-			(hide yes)
-			(show_name no)
-			(do_not_autoplace no)
-			(effects
-				(font
-					(size 1.27 1.27)
-				)
-			)
-		)
-		(pin "1"
-		)
-		(instances
-			(project "cfc-processor"
-				(path "/07ac832f-8d98-4777-b655-1877592dfd88/fb0d8cda-da67-4375-9bc6-6081ff32bfc0"
-					(reference "#3V-014")
-					(unit 1)
-				)
