File: cfc-processor-card-v2/cfc-processor.kicad_pcb (KiCad board)
At the start: 4 copper layers, 99.8 x 94.6 mm, 291 parts, among them J1 2-1734592-0, J1 TFM-120-01-L-D-RA, J2 2-1734592-0, J2 J-SAMTEC-TFM-110-X1-XXX-D-RA, J3 J-SAMTEC-TFM-110-X1-XXX-D-RA, J4 Conn_01x04, J4 TFM-120-01-L-D-RA, J5 Conn_01x04, J5 DM3BT-DSF-PEJS, J6 Conn_01x02, Q1 DMP2240UDM, Q2 PMV45EN, Q3 DMP3050LVT-7, Q4 DMP3050LVT-7, Q5 PMV45EN, Q6 MMBT2907, U1 MAX7310ATE+, U1 RCLAMP0504FB, U10 RCLAMP0504FB, U11 TCAN330, U12 SFEM016GB1EA1TO-I-GE-121-STD, U13 DS90CR218AMTD/NOPB, U2 DS90CR218AMTD/NOPB, U2 MIC842LYC5, U3 MIC842LYC5, U4 TS5A21366, U5 MAX4211FETE, U6 TPS62112, U7 OSD3358-1G-ISM, U8 SN74AUC1G07DCKR, U9 TLVH431, Y1 ECS-240-12-30BQ-AEN-TR, Y2 ABS07-32.768KHZ-T

Commit message: Processor board routing
Completed rework and routing of processor board. No drc errors or warnings. Ready for design review on processor board. Minor changes to schematic for easier routing on pull down resistors connected to the octavo SIP. Reannotated sensor schematic component designators.
Parts:
- removed the C1 at (118.9, 73.3)
- removed the C16 at (124.4, 73.3)
- removed the C17 at (121.9, 73.3)
- removed the C20 at (128.4, 83.3)
- removed the C21 at (118.9, 72.3)
- removed the C23 at (128.9, 72.3)
- removed the C24 at (124.4, 72.3)
- removed the C25 at (121.9, 72.3)
- removed the C26 at (128.4, 84.3)
- removed the C27 at (124.4, 84.3)
- removed the C28 at (124.4, 83.3)
- removed the C4 at (156.4, 134.0)
- removed the C42 at (118.9, 71.3)
- removed the C43 at (128.9, 71.3)
- removed the C45 at (124.4, 71.3)
- removed the C46 at (121.9, 71.3)
- removed the C47 at (124.3, 85.3)
- removed the C48 at (128.4, 85.3)
- removed the C49 at (124.3, 86.9)
- removed the C51 at (151.6, 98.8)
- removed the C7 at (128.9, 73.3)
- removed the J1 at (153.1, 142.3)
- removed the J2 at (120.5, 64.4)
- removed the J4 at (148.5, 64.4)
- removed the J5 at (114.2, 114.2)
- removed JP1: JUMPER-SMT_2_NC_TRACE_SILK, cfc-card:SMT-JUMPER_2_NC_TRACE_SILK
- removed the R21 at (152.8, 98.8)
- removed the R29 at (125.3, 79.7)
- removed the R30 at (123.4, 79.7)
- removed the R6 at (122.4, 83.3)
- removed the R7 at (126.4, 83.3)
- removed the TP1 at (113.1, 96.3)
- removed the TP10 at (144.8, 123.8)
- removed TP102, TP11, TP12, TP121, TP129, TP130, TP132, TP133, TP136, TP138, TP139, TP140, TP141, TP144, TP154, TP156, TP160, TP161, TP163, TP164, TP165, TP166, TP167, TP168, TP35, TP36, TP4, TP40, TP5: TEST-POINT3X4, cfc-card:PAD.03X.04
- removed the TP13 at (158.1, 95.8)
- removed the TP14 at (143.4, 123.9)
- removed the TP15 at (162.6, 111.8)
- removed the TP16 at (164.1, 111.8)
- removed the TP17 at (165.6, 111.8)
- removed the TP18 at (109.1, 96.3)
- removed the TP22 at (177.2, 115.8)
- removed TP23: TEST-POINT3X4, oresat-misc:TestPoint_Pad_D1.0mm
- removed the TP31 at (121.4, 145.7)
- removed TP32, TP41, TP42, TP43, TP44, TP72, TP74, TP75, TP77, TP78: TEST-POINT, cfc-card:2MM-TEST-POINT
- removed the TP37 at (128.1, 99.3)
- removed the TP38 at (126.6, 99.3)
- removed the TP6 at (122.1, 99.3)
- removed the TP7 at (126.6, 102.8)
- removed the TP8 at (125.1, 102.8)
- removed the TP9 at (142.1, 123.8)
- removed the U1 at (155.9, 135.8)
- removed the U2 at (124.4, 78.3)
- J3: value J-SAMTEC-TFM-110-X1-XXX-D-RA -> Val**
- PCB1: value ORESAT-CARD-V1.3-GENERIC-0RF -> (none)
- moved J4 111.3 mm to (114.2, 114.2)
- moved C38 107.9 mm to (118.8, 73.2)
- moved TP83 107.5 mm to (128.5, 145.7)
- moved C44 107.1 mm to (121.8, 72.3)
- moved C46 106.7 mm to (121.8, 71.4)
- moved C42 106.3 mm to (124.3, 70.1), turned to 180 degrees
- moved C43 105.8 mm to (121.8, 73.2)
- moved C35 105.8 mm to (118.8, 72.3)
- moved C33 104.7 mm to (118.8, 71.4)
- moved R59 104.4 mm to (122.3, 83.3), turned to 180 degrees
- moved R60 102.9 mm to (122.6, 89.4), turned to 180 degrees
- moved C41 102.8 mm to (124.3, 73.2), turned to 180 degrees
- moved R62 102.4 mm to (126.3, 83.3)
- moved C36 102.1 mm to (124.3, 71.4), turned to 180 degrees
- moved C39 101.6 mm to (124.3, 72.3), turned to 180 degrees
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Connections:
- net Net-(U13-RXIN1+) renamed /Deserializer/RXIN1_P
- net Net-(U13-RXIN1-) renamed /Deserializer/RXIN1_N
- net Net-(U13-RXIN2+) renamed /Deserializer/RXIN2_P
- net Net-(U13-RXIN2-) renamed /Deserializer/RXIN2_N
- R64 pad 4: unconnected-(R64-44-Pad4) -> Net-(R64-44)
- R64 pad 8: Net-(R64-88) -> unconnected-(R64-88-Pad8)
- U7 pad A8: Net-(R64-33) -> Net-(R64-99)
- U7 pad B6: Net-(R64-88) -> Net-(R64-77)
- U7 pad C6: Net-(R64-77) -> Net-(R64-66)
- U7 pad C7: Net-(R64-66) -> Net-(R64-44)
- U7 pad C8: Net-(R64-99) -> Net-(R64-33)
Routing:
- net (no net): track 386.7 -> 0.00 mm
- net UART0_TX: track 156.3 -> 0.00 mm, vias 4 -> 0
- net UART0_RX: track 147.2 -> 0.00 mm, vias 4 -> 0
- net /OSD3358: SIP C/UART-RX: track 0.00 -> 110.6 mm, vias 0 -> 2
- net /OSD3358: SIP C/UART-TX: track 0.00 -> 107.1 mm, vias 0 -> 4
- net /I2C1_SDA: track 0.00 -> 98.4 mm, vias 0 -> 3
- net SPI1_MOSI: track 92.2 -> 0.00 mm
- net /I2C1_CLK: track 0.00 -> 92.1 mm, vias 0 -> 3
- net /SPI1_MOSI: track 0.00 -> 89.8 mm
- net SPI1_MISO: track 84.5 -> 0.00 mm
- net /SPI1_MISO: track 0.00 -> 83.4 mm
- net SPI1_CLK: track 75.2 -> 0.00 mm, vias 2 -> 0
- net SENSOR_ENABLE: track 74.6 -> 0.00 mm, vias 2 -> 0
- net /SENSOR_ENABLE: track 0.00 -> 74.6 mm, vias 0 -> 2
- net /SPI1_CLK: track 0.00 -> 73.0 mm, vias 0 -> 2
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- added copper zone on B.Cu, net /OSD3358: SIP B/USB_CLI_VBUS
- removed copper zone on In2.Cu, net /OSD3358: SIP B/USB_CLI_VBUS
Other:
- board text added: "VUSB"
- board text removed: "GND"
- board text removed: "SPI_MISO"
- board text removed: "SPI_MOSI"
- board text removed: "UART0_RX"
- board text removed: "UART0_TX"

Commit message: Update
Updated OPD to align with proto card. Made changes from DR with Greenberg. Moved around polygon pours, led indicators, silkscreen issue date, etc. Ready for fab.
Parts:
- removed FID4, FID5, FID6: Fiducial, Fiducial:Fiducial_1mm_Mask2mm
- removed TP16, TP17, TP19: TEST-POINT, oresat-misc:TestPoint-0.75mm-th
- J3: value Val** -> J-SAMTEC-TFM-110-X1-XXX-D-RA
- J4: value Conn_01x04 -> GRPB041VWVN-RC; footprint Connector_PinHeader_2.54mm:PinHeader_1x04_P2.54mm_Vertical -> Connector_PinHeader_1.27mm:PinHeader_1x04_P1.27mm_Vertical
- Q2, Q5: value PMV45EN -> DMN2050LQ-7
- Q3, Q4: value DMP3050LVT-7 -> DMPH2040UVTQ-7
- R1: value 10 -> 100
- R11, R13, R3: value 100 -> 1k
- R24: value 10k -> 1k
- R28: value 2.7k -> 4.7k
- R39, R41: value 2.7k -> 10k
- R43: value 1k -> 10k
- moved D3 66.4 mm to (186.3, 136.5), turned to 90 degrees
- moved D4 66.3 mm to (191.2, 136.6), turned to 90 degrees
- moved D2 66.3 mm to (188.7, 136.6), turned to 90 degrees
- moved D1 66.2 mm to (183.8, 136.5), turned to 90 degrees
- moved R41 58.5 mm to (186.3, 132.5), turned to 90 degrees
- moved R43 58.3 mm to (191.2, 132.6), turned to -90 degrees
- moved R39 58.3 mm to (188.7, 132.6), turned to 90 degrees
- moved R28 58.2 mm to (183.8, 132.5), turned to 90 degrees
- moved J4 1.14 mm to (114.2, 115.4)
Routing:
- net VBUSP: track 15.1 -> 68.6 mm, vias 0 -> 1
- net VPD: track 80.5 -> 36.9 mm
- net /Power (OPD)/ON/~{OFF}: track 76.1 -> 116.8 mm, vias 4 -> 3
- net Net-(U5-CIN1+): track 22.8 -> 5.27 mm
- net Net-(U5-CIN1-): track 21.1 -> 4.88 mm, vias 1 -> 0
- net 3.3V: track 57.4 -> 62.6 mm
- net /EEPROM_WP: track 28.7 -> 28.1 mm
- net 5V: track 11.3 -> 11.5 mm, vias 16 -> 17
- net GND: vias 297 -> 291
- net /Power (OPD)/CB-RESET: vias 1 -> 2
Other:
- board text removed: "OLIVER REW et al"
