File: cfc-processor-card-v2/cfc-processor-sch-Deserializer.kicad_sch (KiCad schematic)
At the start: 24 parts, among them U13 DS90CR218AMTD/NOPB

Commit message: Processor board routing
Completed rework and routing of processor board. No drc errors or warnings. Ready for design review on processor board. Minor changes to schematic for easier routing on pull down resistors connected to the octavo SIP. Reannotated sensor schematic component designators.
Connections:
- net RXIN1_N: now reaches R60.2, U13.10 (RXIN1-)
- net RXIN1_P: now reaches R60.1, U13.11 (RXIN1+)
- net RXIN2_N: now reaches R61.2, U13.14 (RXIN2-)
- net RXIN2_P: now reaches R61.1, U13.15 (RXIN2+)
Changed lines of the file:
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@@
+		)
+	)
+	(label "RXIN2_N"
+		(at 229.87 171.45 0)
+		(effects
+			(font
+				(size 0.889 0.889)
+			)
+			(justify left bottom)
+		)
+	)
+	(label "RXIN1_N"
+		(at 229.87 163.83 0)
+		(effects
+			(font
+				(size 0.889 0.889)
+			)
+			(justify left bottom)
 		)
 	)
@@
 		)
 	)
+	(label "RXIN2_P"
+		(at 229.87 173.99 0)
+		(effects
+			(font
+				(size 0.889 0.889)
+			)
+			(justify left bottom)
+		)
+	)
 	(label "PRU_BUS.PRU0_6"
 		(at 179.07 163.83 180)
@@
 		)
 	)
+	(label "RXIN1_P"
+		(at 229.87 166.37 0)
+		(effects
+			(font
+				(size 0.889 0.889)
+			)
+			(justify left bottom)
+		)
+	)

Commit message: Update
Updated BOM, couple of fixes on OPD. Minor routing and layout changes. Removed logic gates from sensor card.
Parts:
- C35, C37, C39, C44, C47, C50: DIS DigiKey -> Mouser; DPN 399-C0402C100F5GACAUTOCT-ND -> 81-GXT155R71E103KE1D; MFR KEMET -> Murata Electronics; MPN C0402C100F5GACAUTO -> GXT155R71E103KE01D
- C42: DPN 490-GRT21BC71E106KE13LCT-ND -> 490-GRT21BC71E106KE13KCT-ND; MPN GRT21BC71E106KE13L -> GRT21BC71E106KE13K
Changed lines of the file:
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@@
 			)
 		)
-		(property "Datasheet" "https://search.kemet.com/download/datasheet/C0402C100F5GACAUTO"
+		(property "Datasheet" ""
 			(at 177.8 107.95 0)
 			(hide yes)
@@
 			)
 		)
-		(property "Description" "Unpolarized capacitor, small symbol"
+		(property "Description" "0.01uF 10% 25VDC Multilayer Ceramic Capacitors MLCC - SMD/SMT 0402 X7R AEC-Q200"
 			(at 177.8 107.95 0)
 			(hide yes)
@@
 			)
 		)
-		(property "DIS" "DigiKey"
+		(property "DIS" "Mouser"
 			(at 177.8 107.95 0)
 			(hide yes)
@@
 			)
 		)
-		(property "DPN" "399-C0402C100F5GACAUTOCT-ND"
+		(property "DPN" "81-GXT155R71E103KE1D"
 			(at 177.8 107.95 0)
 			(hide yes)
@@
 			)
 		)
-		(property "MFR" "KEMET"
+		(property "MFR" "Murata Electronics"
 			(at 177.8 107.95 0)
 			(hide yes)
@@
 			)
 		)
-		(property "MPN" "C0402C100F5GACAUTO"
+		(property "MPN" "GXT155R71E103KE01D"
 			(at 177.8 107.95 0)
 			(hide yes)
@@
 			)
 		)
-		(property "Description" "Unpolarized capacitor, small symbol"
+		(property "Description" "1000 pF ±5% 25V Ceramic Capacitor C0G, NP0 0402 (1005 Metric)"
 			(at 177.8 125.73 0)
 			(hide yes)
@@
 			)
 		)
-		(property "Datasheet" "https://search.kemet.com/download/datasheet/C0402C100F5GACAUTO"
+		(property "Datasheet" ""
 			(at 231.14 109.22 0)
 			(hide yes)
@@
 			)
 		)
-		(property "Description" "Unpolarized capacitor, small symbol"
+		(property "Description" "0.01uF 10% 25VDC Multilayer Ceramic Capacitors MLCC - SMD/SMT 0402 X7R AEC-Q200"
 			(at 231.14 109.22 0)
 			(hide yes)
@@
 			)
 		)
-		(property "DIS" "DigiKey"
+		(property "DIS" "Mouser"
 			(at 231.14 109.22 0)
 			(hide yes)
@@
 			)
 		)
-		(property "DPN" "399-C0402C100F5GACAUTOCT-ND"
+		(property "DPN" "81-GXT155R71E103KE1D"
 			(at 231.14 109.22 0)
 			(hide yes)
@@
 			)
 		)
-		(property "MFR" "KEMET"
+		(property "MFR" "Murata Electronics"
 			(at 231.14 109.22 0)
 			(hide yes)
@@
 			)
 		)
-		(property "MPN" "C0402C100F5GACAUTO"
+		(property "MPN" "GXT155R71E103KE01D"
 			(at 231.14 109.22 0)
 			(hide yes)
@@
 			)
 		)
-		(property "Description" "Unpolarized capacitor, small symbol"
+		(property "Description" "8.8 pF ±0.1pF 50V Ceramic Capacitor C0G, NP0 0603 (1608 Metric)"
 			(at 231.14 91.44 0)
 			(hide yes)
@@
 			)
 		)
-		(property "Description" "Unpolarized capacitor, small symbol"
+		(property "Description" "1000 pF ±5% 25V Ceramic Capacitor C0G, NP0 0402 (1005 Metric)"
 			(at 193.04 90.17 0)
 			(hide yes)
@@
 			)
 		)
-		(property "Datasheet" "https://search.kemet.com/download/datasheet/C0402C100F5GACAUTO"
+		(property "Datasheet" ""
 			(at 185.42 90.17 0)
 			(hide yes)
@@
 			)
 		)
-		(property "Description" "Unpolarized capacitor, small symbol"
+		(property "Description" "0.01uF 10% 25VDC Multilayer Ceramic Capacitors MLCC - SMD/SMT 0402 X7R AEC-Q200"
 			(at 185.42 90.17 0)
 			(hide yes)
@@
 			)
 		)
-		(property "DIS" "DigiKey"
+		(property "DIS" "Mouser"
 			(at 185.42 90.17 0)
 			(hide yes)
@@
 			)
 		)
-		(property "DPN" "399-C0402C100F5GACAUTOCT-ND"
+		(property "DPN" "81-GXT155R71E103KE1D"
 			(at 185.42 90.17 0)
 			(hide yes)
@@
 			)
 		)
-		(property "MFR" "KEMET"
+		(property "MFR" "Murata Electronics"
 			(at 185.42 90.17 0)
 			(hide yes)
@@
 			)
 		)
-		(property "MPN" "C0402C100F5GACAUTO"
+		(property "MPN" "GXT155R71E103KE01D"
 			(at 185.42 90.17 0)
 			(hide yes)
@@
 			)
 		)
-		(property "Datasheet" "https://search.kemet.com/download/datasheet/C0402C100F5GACAUTO"
+		(property "Datasheet" ""
 			(at 170.18 125.73 0)
 			(hide yes)
@@
 			)
 		)
-		(property "Description" "Unpolarized capacitor, small symbol"
+		(property "Description" "0.01uF 10% 25VDC Multilayer Ceramic Capacitors MLCC - SMD/SMT 0402 X7R AEC-Q200"
 			(at 170.18 125.73 0)
 			(hide yes)
@@
 			)
 		)
-		(property "DIS" "DigiKey"
+		(property "DIS" "Mouser"
 			(at 170.18 125.73 0)
 			(hide yes)
@@
 			)
 		)
-		(property "DPN" "399-C0402C100F5GACAUTOCT-ND"
+		(property "DPN" "81-GXT155R71E103KE1D"
 			(at 170.18 125.73 0)
 			(hide yes)
@@
 			)
 		)
-		(property "MFR" "KEMET"
+		(property "MFR" "Murata Electronics"
 			(at 170.18 125.73 0)
 			(hide yes)
@@
 			)
 		)
-		(property "MPN" "C0402C100F5GACAUTO"
+		(property "MPN" "GXT155R71E103KE01D"
 			(at 170.18 125.73 0)
 			(hide yes)
@@
 			)
 		)
-		(property "Description" "Unpolarized capacitor, small symbol"
+		(property "Description" "1000 pF ±5% 25V Ceramic Capacitor C0G, NP0 0402 (1005 Metric)"
 			(at 185.42 107.95 0)
 			(hide yes)
@@
 			)
 		)
-		(property "Datasheet" "https://search.kemet.com/download/datasheet/C0402C100F5GACAUTO"
+		(property "Datasheet" ""
 			(at 223.52 91.44 0)
 			(hide yes)
@@
 			)
 		)
-		(property "Description" "Unpolarized capacitor, small symbol"
+		(property "Description" "0.01uF 10% 25VDC Multilayer Ceramic Capacitors MLCC - SMD/SMT 0402 X7R AEC-Q200"
 			(at 223.52 91.44 0)
 			(hide yes)
@@
 			)
 		)
-		(property "DIS" "DigiKey"
+		(property "DIS" "Mouser"
 			(at 223.52 91.44 0)
 			(hide yes)
@@
 			)
 		)
-		(property "DPN" "399-C0402C100F5GACAUTOCT-ND"
+		(property "DPN" "81-GXT155R71E103KE1D"
 			(at 223.52 91.44 0)
 			(hide yes)
@@
 			)
 		)
-		(property "MFR" "KEMET"
+		(property "MFR" "Murata Electronics"
 			(at 223.52 91.44 0)
 			(hide yes)
@@
 			)
 		)
-		(property "MPN" "C0402C100F5GACAUTO"
+		(property "MPN" "GXT155R71E103KE01D"
 			(at 223.52 91.44 0)
 			(hide yes)
@@
 			)
 		)
-		(property "Description" "Unpolarized capacitor, small symbol"
+		(property "Description" "1000 pF ±5% 25V Ceramic Capacitor C0G, NP0 0402 (1005 Metric)"
 			(at 215.9 91.44 0)
 			(hide yes)
@@
 			)
 		)
-		(property "Description" "Unpolarized capacitor, small symbol"
+		(property "Description" "8.8 pF ±0.1pF 50V Ceramic Capacitor C0G, NP0 0603 (1608 Metric)"
 			(at 170.18 107.95 0)
 			(hide yes)
@@
 			)
 		)
-		(property "Description" "Unpolarized capacitor, small symbol"
+		(property "Description" "10 µF ±10% 25V Ceramic Capacitor X7S 0805 (2012 Metric)"
 			(at 205.74 72.39 0)
 			(hide yes)
@@
 			)
 		)
-		(property "DPN" "490-GRT21BC71E106KE13LCT-ND"
+		(property "DPN" "490-GRT21BC71E106KE13KCT-ND"
 			(at 205.74 72.39 0)
 			(hide yes)
@@
 			)
 		)
-		(property "MPN" "GRT21BC71E106KE13L"
+		(property "MPN" "GRT21BC71E106KE13K"
 			(at 205.74 72.39 0)
 			(hide yes)
@@
 			)
 		)
-		(property "Datasheet" "https://search.kemet.com/download/datasheet/C0402C100F5GACAUTO"
+		(property "Datasheet" ""
 			(at 238.76 127 0)
 			(hide yes)
@@
 			)
 		)
-		(property "Description" "Unpolarized capacitor, small symbol"
+		(property "Description" "0.01uF 10% 25VDC Multilayer Ceramic Capacitors MLCC - SMD/SMT 0402 X7R AEC-Q200"
 			(at 238.76 127 0)
 			(hide yes)
@@
 			)
 		)
-		(property "DIS" "DigiKey"
+		(property "DIS" "Mouser"
 			(at 238.76 127 0)
 			(hide yes)
@@
 			)
 		)
-		(property "DPN" "399-C0402C100F5GACAUTOCT-ND"
+		(property "DPN" "81-GXT155R71E103KE1D"
 			(at 238.76 127 0)
 			(hide yes)
@@
 			)
 		)
-		(property "MFR" "KEMET"
+		(property "MFR" "Murata Electronics"
 			(at 238.76 127 0)
 			(hide yes)
@@
 			)
 		)
-		(property "MPN" "C0402C100F5GACAUTO"
+		(property "MPN" "GXT155R71E103KE01D"
 			(at 238.76 127 0)
 			(hide yes)
@@
 			)
 		)
-		(property "Description" "Unpolarized capacitor, small symbol"
+		(property "Description" "8.8 pF ±0.1pF 50V Ceramic Capacitor C0G, NP0 0603 (1608 Metric)"
 			(at 238.76 109.22 0)
 			(hide yes)
@@
 			)
 		)
-		(property "Description" "Unpolarized capacitor, small symbol"
+		(property "Description" "8.8 pF ±0.1pF 50V Ceramic Capacitor C0G, NP0 0603 (1608 Metric)"
 			(at 246.38 127 0)
 			(hide yes)
@@
 			)
 		)
-		(property "Description" "Unpolarized capacitor, small symbol"
+		(property "Description" "1000 pF ±5% 25V Ceramic Capacitor C0G, NP0 0402 (1005 Metric)"
 			(at 231.14 127 0)
 			(hide yes)
@@
 			)
 		)
-		(property "Description" "Unpolarized capacitor, small symbol"
+		(property "Description" "8.8 pF ±0.1pF 50V Ceramic Capacitor C0G, NP0 0603 (1608 Metric)"
 			(at 177.8 90.17 0)
 			(hide yes)
@@
 			)
 		)
-		(property "Description" "Unpolarized capacitor, small symbol"
+		(property "Description" "1000 pF ±5% 25V Ceramic Capacitor C0G, NP0 0402 (1005 Metric)"
 			(at 223.52 109.22 0)
 			(hide yes)
@@
 			)
 		)
-		(property "Description" "Unpolarized capacitor, small symbol"
+		(property "Description" "8.8 pF ±0.1pF 50V Ceramic Capacitor C0G, NP0 0603 (1608 Metric)"
 			(at 162.56 125.73 0)
 			(hide yes)
