File: cfc-processor-card-v2/cfc-processor.kicad_sch (KiCad schematic)
At the start: 11 parts, among them J1 TFM-120-01-L-D-RA, J2 2-1734592-0, J3 J-SAMTEC-TFM-110-X1-XXX-D-RA, J4 Conn_01x04

Commit message: Update
Updated OPD to align with proto card. Made changes from DR with Greenberg. Moved around polygon pours, led indicators, silkscreen issue date, etc. Ready for fab.
Parts:
- removed FID4, FID5, FID6: Fiducial, Fiducial:Fiducial_1mm_Mask2mm, symbol Mechanical:Fiducial
- J4: value Conn_01x04 -> GRPB041VWVN-RC; footprint Connector_PinHeader_2.54mm:PinHeader_1x04_P2.54mm_Vertical -> Connector_PinHeader_1.27mm:PinHeader_1x04_P1.27mm_Vertical; DIS (none) -> DigiKey; DPN (none) -> S9014E-04-ND; MFR (none) -> Sullins Connector Solutions; MPN (none) -> GRPB041VWVN-RC
Other:
- moved on the sheet: FID1, FID2, FID3

Commit message: Small update
Fixed minor issue with voltage clamp on usb line. Added nreset clamp and changed VBUS pin to USB voltage bus
Other:
- sheet OSD3358: SIP A (PWR) ports: added nRESET_CLAMP; removed none
- sheet OSD3358: SIP B ports: added nRESET_CLAMP; removed none
Changed lines of the file:
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@@
+	(wire
+		(pts
+			(xy 240.03 228.6) (xy 240.03 210.82)
+		)
+		(stroke
+			(width 0)
+			(type default)
+		)
+	)
 	(wire
 		(pts
@@
 	(wire
 		(pts
+			(xy 228.6 228.6) (xy 240.03 228.6)
+		)
+		(stroke
+			(width 0)
+			(type default)
+		)
+	)
+	(wire
+		(pts
 			(xy 242.57 95.25) (xy 267.97 95.25)
 		)
@@
 			(width 0.1524)
 			(type solid)
+		)
+	)
+	(wire
+		(pts
+			(xy 240.03 210.82) (xy 228.6 210.82)
+		)
+		(stroke
+			(width 0)
+			(type default)
 		)
 	)
@@
 			)
 		)
+		(pin "nRESET_CLAMP" output
+			(at 228.6 228.6 0)
+			(effects
+				(font
+					(size 1.27 1.27)
+				)
+				(justify right)
+			)
+		)
 		(instances
 			(project "cfc-processor"
@@
 			(effects
 				(font
+					(size 1.27 1.27)
+				)
+				(justify right)
+			)
+		)
+		(pin "nRESET_CLAMP" input
+			(at 228.6 210.82 0)
+			(effects
+				(font
